File: latentred/boards/linecard/latentred-linecard/phys.sch (KiCad schematic (older format))
At the start: 396 parts, among them J2 STEWART_SS_74500_024, Q1 SSM6N58NU, Q2 SSM6N58NU, Q3 SSM6N58NU, Q4 SSM6N58NU, Q5 SSM6N58NU, Q6 SSM6N58NU, Q7 SSM6N58NU, Q8 SSM6N58NU, U10 DP83867, U11 DP83867, U12 DP83867, U13 DP83867, U14 DP83867, U15 DP83867, U16 DSC6101CI2A-025.0000, U17 5PB1108CMG, U8 DP83867, U9 DP83867

Commit message: Completely rerouted magnetics for much cleaner, though slightly wider, "clamshell" layout
Parts:
- added C238, C239: TBD, azonenberg_pcb:EIA_1206_CAP_NOSILK, symbol device:C
- added unit 9 of J2
- added R157, R158: TBD, azonenberg_pcb:EIA_1206_CAP_NOSILK, symbol device:R
Connections:
- net GND: now also C238.2, C239.2, R157.2, R158.2; no longer C126.1, C127.1, C128.1, C229.1, C230.1, C231.1, C232.1, C50.1
- new net SHIELD: C126.1, C127.1, C128.1, C229.1, C230.1, C231.1, C232.1, C238.1, C239.1, C50.1, J2.SHLD (SHIELD), R157.1, R158.1
Other:
- note added: "TODO: R/C between shield and ground"
- note removed: "TODO: Add connections for RJ45 shield"
Changed lines of the file:
@@
 Sheet 3 3
 Title "LATENTRED 8-port 10/100/1000 Base-T Line Card"
-Date "2018-04-21"
+Date "2018-04-23"
 Rev "0.1"
 Comp "Andrew D. Zonenberg"
@@
 	10650 2300 10650 2400
 Text Label 11350 2300 0    50   ~ 0
-GND
+SHIELD
 Wire Wire Line
 	11350 2300 11150 2300
@@
 	10650 7050 10650 7150
 Text Label 11350 7050 0    50   ~ 0
-GND
+SHIELD
 Wire Wire Line
 	11350 7050 11150 7050
@@
 	10700 11750 10700 11850
 Text Label 11400 11750 0    50   ~ 0
-GND
+SHIELD
 Wire Wire Line
 	11400 11750 11200 11750
@@
 	10700 16500 10700 16600
 Text Label 11400 16500 0    50   ~ 0
-GND
+SHIELD
 Wire Wire Line
 	11400 16500 11200 16500
@@
 	22500 2300 22500 2400
 Text Label 23200 2300 0    50   ~ 0
-GND
+SHIELD
 Wire Wire Line
 	23200 2300 23000 2300
@@
 	22500 7050 22500 7150
 Text Label 23200 7050 0    50   ~ 0
-GND
+SHIELD
 Wire Wire Line
 	23200 7050 23000 7050
@@
 	22550 11750 22550 11850
 Text Label 23250 11750 0    50   ~ 0
-GND
+SHIELD
 Wire Wire Line
 	23250 11750 23050 11750
@@
 	22550 16500 22550 16600
 Text Label 23250 16500 0    50   ~ 0
-GND
+SHIELD
 Wire Wire Line
 	23250 16500 23050 16500
@@
 Wire Wire Line
 	29200 4250 29000 4250
-Text Notes 30900 750  0    50   ~ 0
-TODO: Add connections for RJ45 shield
+Text Notes 30750 7550 0    50   ~ 0
+TODO: R/C between shield and ground
 Wire Wire Line
 	17000 16650 17200 16650
@@
 Text Label 10850 3700 2    50   ~ 0
 ETH0_DM_N
+$Comp
+L special-azonenberg:STEWART_SS_74500_024 J2
+U 9 1 6893DE21
+P 30700 9000
+F 0 "J2" H 31377 9701 50  0000 L CNN
+F 1 "STEWART_SS_74500_024" H 31377 9610 50  0000 L CNN
+F 2 "azonenberg_pcb:CONN_STEWART_SS_74500_024" H 30700 9000 50  0001 C CNN
+F 3 "" H 30700 9000 50  0001 C CNN
+	9    30700 9000
+	1    0    0    -1
+$EndComp
+Text Label 30500 8950 2    50   ~ 0
+SHIELD
+Wire Wire Line
+	30500 8950 30600 8950
+$Comp
+L device:C C238
+U 1 1 68E3168F
+P 30500 9400
+F 0 "C238" H 30615 9446 50  0000 L CNN
+F 1 "TBD" H 30615 9355 50  0000 L CNN
+F 2 "azonenberg_pcb:EIA_1206_CAP_NOSILK" H 30538 9250 50  0001 C CNN
+F 3 "" H 30500 9400 50  0001 C CNN
+	1    30500 9400
+	1    0    0    -1
+$EndComp
+Text Label 30500 9250 2    50   ~ 0
+SHIELD
+Text Label 30500 9550 2    50   ~ 0
+GND
+$Comp
+L device:C C239
+U 1 1 68E32774
+P 30900 9400
+F 0 "C239" H 31015 9446 50  0000 L CNN
+F 1 "TBD" H 31015 9355 50  0000 L CNN
+F 2 "azonenberg_pcb:EIA_1206_CAP_NOSILK" H 30938 9250 50  0001 C CNN
+F 3 "" H 30900 9400 50  0001 C CNN
+	1    30900 9400
+	1    0    0    -1
+$EndComp
+$Comp
+L device:R R157
+U 1 1 68E32FEB
+P 31300 9400
+F 0 "R157" H 31370 9446 50  0000 L CNN
+F 1 "TBD" H 31370 9355 50  0000 L CNN
+F 2 "azonenberg_pcb:EIA_1206_CAP_NOSILK" V 31230 9400 50  0001 C CNN
+F 3 "" H 31300 9400 50  0001 C CNN
+	1    31300 9400
+	1    0    0    -1
+$EndComp
+$Comp
+L device:R R158
+U 1 1 68E34123
+P 31650 9400
+F 0 "R158" H 31720 9446 50  0000 L CNN
+F 1 "TBD" H 31720 9355 50  0000 L CNN
+F 2 "azonenberg_pcb:EIA_1206_CAP_NOSILK" V 31580 9400 50  0001 C CNN
+F 3 "" H 31650 9400 50  0001 C CNN
+	1    31650 9400
+	1    0    0    -1
+$EndComp
+Wire Wire Line
+	31650 9250 31300 9250
+Wire Wire Line
+	31300 9250 30900 9250
+Connection ~ 31300 9250
+Wire Wire Line
+	30900 9250 30500 9250
+Connection ~ 30900 9250
+Wire Wire Line
+	30500 9550 30900 9550
+Wire Wire Line
+	30900 9550 31300 9550
+Connection ~ 30900 9550
+Wire Wire Line
+	31300 9550 31650 9550
+Connection ~ 31300 9550
 $EndSCHEMATC

Commit message: Continued PHY layout
Parts:
- removed C146, C148, C154, C155, C156: 4.7 uF, azonenberg_pcb:EIA_0603_CAP_NOSILK, symbol device:C
- removed L20, L22, L26, L27, L28: 600R, azonenberg_pcb:EIA_0402_RES_NOSILK, symbol passive-azonenberg:INDUCTOR_PWROUT
Connections:
- net A1V0_4 is gone; now on net A1V0_5: C167.1, C187.1, C203.1, C217.1, C225.1, U12.24 (1V0), U12.31 (1V0), U12.42 (1V0), U12.6 (1V0)
- net A1V0_6 is gone; now on net A1V0_7: C173.1, C193.1, C209.1, C219.1, C227.1, U14.24 (1V0), U14.31 (1V0), U14.42 (1V0), U14.6 (1V0)
- net A1V8_6 is gone; now on net A1V8_7: C172.1, C192.1, C208.1, U14.13 (A1V8), U14.48 (A1V8)
- net A2V5_4 is gone; now on net A2V5_5: C165.1, C185.1, C201.1, U12.3 (A2V5), U12.9 (A2V5)
- net A2V5_6 is gone; now on net A2V5_7: C171.1, C191.1, C207.1, U14.3 (A2V5), U14.9 (A2V5)
- net ETH4_A_N: now also L32.11 (D_P); no longer L32.12 (D_N)
- net ETH4_A_P: now also L32.12 (D_N); no longer L32.11 (D_P)
- net ETH4_B_N: now also L32.8 (C_P); no longer L32.9 (C_N)
- net ETH4_B_P: now also L32.9 (C_N); no longer L32.8 (C_P)
- net ETH4_C_N: now also L32.5 (B_P); no longer L32.6 (B_N)
- net ETH4_C_P: now also L32.6 (B_N); no longer L32.5 (B_P)
- net ETH4_D_N: now also L32.2 (A_P); no longer L32.3 (A_N)
- net ETH4_D_P: now also L32.3 (A_N); no longer L32.2 (A_P)
- net ETH5_A_N: now also L33.11 (D_P); no longer L33.12 (D_N)
- net ETH5_A_P: now also L33.12 (D_N); no longer L33.11 (D_P)
- net ETH5_B_N: now also L33.8 (C_P); no longer L33.9 (C_N)
- net ETH5_B_P: now also L33.9 (C_N); no longer L33.8 (C_P)
- net ETH5_C_N: now also L33.5 (B_P); no longer L33.6 (B_N)
- net ETH5_C_P: now also L33.6 (B_N); no longer L33.5 (B_P)
- net ETH5_D_N: now also L33.2 (A_P); no longer L33.3 (A_N)
- net ETH5_D_P: now also L33.3 (A_N); no longer L33.2 (A_P)
- net ETH6_A_N: now also L34.11 (D_P); no longer L34.12 (D_N)
- net ETH6_A_P: now also L34.12 (D_N); no longer L34.11 (D_P)
- net ETH6_B_N: now also L34.8 (C_P); no longer L34.9 (C_N)
- net ETH6_B_P: now also L34.9 (C_N); no longer L34.8 (C_P)
- net ETH6_C_N: now also L34.5 (B_P); no longer L34.6 (B_N)
- net ETH6_C_P: now also L34.6 (B_N); no longer L34.5 (B_P)
- net ETH6_D_N: now also L34.2 (A_P); no longer L34.3 (A_N)
- net ETH6_D_P: now also L34.3 (A_N); no longer L34.2 (A_P)
- net ETH7_A_N: now also L35.11 (D_P); no longer L35.12 (D_N)
- net ETH7_A_P: now also L35.12 (D_N); no longer L35.11 (D_P)
- net ETH7_B_N: now also L35.8 (C_P); no longer L35.9 (C_N)
- net ETH7_B_P: now also L35.9 (C_N); no longer L35.8 (C_P)
- net ETH7_C_N: now also L35.5 (B_P); no longer L35.6 (B_N)
- net ETH7_C_P: now also L35.6 (B_N); no longer L35.5 (B_P)
- net ETH7_D_N: now also L35.2 (A_P); no longer L35.3 (A_N)
- net ETH7_D_P: now also L35.3 (A_N); no longer L35.2 (A_P)
- net SGMII6_TX_C_P: now reaches C137.1, U14.27 (TX_D1/SGMII_TX_P)
- net SGMII6_TX_C_N: now reaches C138.1, U14.28 (TX_D0/SGMII_TX_N)
- net SGMII7_TX_C_P: now reaches C141.1, U15.27 (TX_D1/SGMII_TX_P)
- net SGMII7_TX_C_N: now reaches C142.1, U15.28 (TX_D0/SGMII_TX_N)
- net RX_D2_6 renamed SGMII6_RX_C_P
- net RX_D2_7 renamed SGMII7_RX_C_P
- net RX_D3_6 renamed SGMII6_RX_C_N
- net RX_D3_7 renamed SGMII7_RX_C_N
Other:
- note added: "Sharing analog rail with sandwiched PHY"
- note added: "Swap P/N pairs for easier layout. PHY auto-corrects."

Commit message: Laid out second pair of PHYs
Parts:
- removed C147: 4.7 uF, azonenberg_pcb:EIA_0603_CAP_NOSILK, symbol device:C
- removed L21: 600R, azonenberg_pcb:EIA_0402_RES_NOSILK, symbol passive-azonenberg:INDUCTOR_PWROUT
Connections:
- net A1V8_4 is gone; now on net A1V8_5: C166.1, C186.1, C202.1, U12.13 (A1V8), U12.48 (A1V8)
- net SGMII4_TX_C_P: now reaches C129.1, U12.27 (TX_D1/SGMII_TX_P)
- net SGMII4_TX_C_N: now reaches C130.1, U12.28 (TX_D0/SGMII_TX_N)
- net SGMII5_TX_C_P: now reaches C133.1, U13.27 (TX_D1/SGMII_TX_P)
- net SGMII5_TX_C_N: now reaches C134.1, U13.28 (TX_D0/SGMII_TX_N)
- net RX_D2_4 renamed SGMII4_RX_C_P
- net RX_D2_5 renamed SGMII5_RX_C_P
- net RX_D3_4 renamed SGMII4_RX_C_N
- net RX_D3_5 renamed SGMII5_RX_C_N
Changed lines of the file:
@@
 Sheet 3 3
 Title "LATENTRED 8-port 10/100/1000 Base-T Line Card"
-Date "2018-04-24"
+Date "2018-04-25"
 Rev "0.1"
 Comp "Andrew D. Zonenberg"
@@
 Text Label 5350 17850 0    50   ~ 0
 JTAG_TCK
-Text HLabel 17200 5450 0    50   Input ~ 0
-1V8
 Text HLabel 14450 4100 0    50   Input ~ 0
 SGMII4_TX_P
@@
 A1V0_5
 Text Label 15100 3050 2    50   ~ 0
-A1V8_4
-$Comp
-L passive-azonenberg:INDUCTOR_PWROUT L21
-U 1 1 5BB3FA23
-P 17900 5450
-F 0 "L21" V 17850 5200 40  0000 C CNN
-F 1 "600R" V 17850 5700 40  0000 C CNN
-F 2 "azonenberg_pcb:EIA_0402_RES_NOSILK" H 17900 5450 60  0001 C CNN
-F 3 "" H 17900 5450 60  0000 C CNN
-	1    17900 5450
-	0    1    1    0
-$EndComp
+A1V8_5
 Text Label 15100 3250 2    50   ~ 0
 1V8
@@
 	18850 5250 19400 5250
 Connection ~ 18850 5250
-$Comp
-L device:C C147
-U 1 1 5BB3FAA9
-P 17300 5600
-F 0 "C147" H 17415 5646 50  0000 L CNN
-F 1 "4.7 uF" H 17415 5555 50  0000 L CNN
-F 2 "azonenberg_pcb:EIA_0603_CAP_NOSILK" H 17338 5450 50  0001 C CNN
-F 3 "" H 17300 5600 50  0001 C CNN
-	1    17300 5600
-	1    0    0    -1
-$EndComp
-Wire Wire Line
-	17600 5450 17300 5450
-Wire Wire Line
-	17300 5450 17200 5450
-Connection ~ 17300 5450
-Text Label 17200 5750 2    50   ~ 0
+Text Label 19400 5750 0    50   ~ 0
 GND
-Wire Wire Line
-	17200 5750 17300 5750
 $Comp
 L device:C C166
@@
 Connection ~ 19400 4950
 Text Label 19400 5450 0    50   ~ 0
-A1V8_4
+A1V8_5
 Wire Wire Line
 	19400 5450 18850 5450
-Wire Wire Line
-	18350 5450 18200 5450
-Connection ~ 18350 5450
 $Comp
 L device:C C186
@@
 $EndComp
 Wire Wire Line
-	17300 5750 18350 5750
-Connection ~ 17300 5750
-Wire Wire Line
 	18350 5750 18850 5750
-Connection ~ 18350 5750
 Wire Wire Line
 	18850 5750 19400 5750
@@
 	16950 3750 17150 3750
 Text Label 15150 4850 2    50   ~ 0
-RX_D2_4
+SGMII4_RX_C_P
 Text Label 15150 4950 2    50   ~ 0
-RX_D3_4
+SGMII4_RX_C_N
 Text Label 20800 5250 0    50   ~ 0
-RX_D2_4
+SGMII4_RX_C_P
 Text Label 20800 5450 0    50   ~ 0
-RX_D3_4
+SGMII4_RX_C_N
 $Comp
 L device:R R83
@@
 Connection ~ 20500 14850
 Text Label 20800 10200 0    50   ~ 0
-RX_D2_5
+SGMII5_RX_C_P
 Text Label 20800 10400 0    50   ~ 0
-RX_D3_5
+SGMII5_RX_C_N
 $Comp
 L device:R R87
@@
 Text Label 15200 14400 2    50   ~ 0
 SGMII6_RX_C_N
-Text Label 15150 9600 2    50   ~ 0
-RX_D2_5
-Text Label 15150 9700 2    50   ~ 0
-RX_D3_5
+Text Label 15100 9600 2    50   ~ 0
+SGMII5_RX_C_P
+Text Label 15100 9700 2    50   ~ 0
+SGMII5_RX_C_N
 $Comp
 L osc-azonenberg:OSC U16
@@
 Text Label 15250 13700 2    50   ~ 0
 SGMII6_TX_C_N
+Text Label 15150 8900 2    50   ~ 0
+SGMII5_TX_C_P
+Text Label 15150 9000 2    50   ~ 0
+SGMII5_TX_C_N
+Text Label 15100 4150 2    50   ~ 0
+SGMII4_TX_C_P
+Text Label 15100 4250 2    50   ~ 0
+SGMII4_TX_C_N
 $EndSCHEMATC
