File: latentred/boards/linecard/latentred-linecard/phys.sch (KiCad schematic (older format))
At the start: 388 parts, among them J2 STEWART_SS_74500_024, Q1 SSM6N58NU, Q2 SSM6N58NU, Q3 SSM6N58NU, Q4 SSM6N58NU, Q5 SSM6N58NU, Q6 SSM6N58NU, Q7 SSM6N58NU, Q8 SSM6N58NU, U10 DP83867, U11 DP83867, U12 DP83867, U13 DP83867, U14 DP83867, U15 DP83867, U16 DSC6101CI2A-025.0000, U17 5PB1108CMG, U8 DP83867, U9 DP83867

Commit message: Initial layout on ports 2/3
Parts:
- removed C68, C69, C70: 4.7 uF, azonenberg_pcb:EIA_0603_CAP_NOSILK, symbol device:C
- removed L11, L12, L13: 600R, azonenberg_pcb:EIA_0402_RES_NOSILK, symbol passive-azonenberg:INDUCTOR_PWROUT
Connections:
- net A1V0_2 is gone; now on net A1V0_3: C110.1, C118.1, C124.1, C83.1, C98.1, U10.24 (1V0), U10.31 (1V0), U10.42 (1V0), U10.6 (1V0)
- net A1V8_2 is gone; now on net A1V8_3: C109.1, C82.1, C97.1, U10.13 (A1V8), U10.48 (A1V8)
- net A2V5_2 is gone; now on net A2V5_3: C108.1, C81.1, C96.1, U10.3 (A2V5), U10.9 (A2V5)
- net ETH2_A_N: now also L18.11 (DM_P); no longer L18.12 (DM_N)
- net ETH2_A_P: now also L18.12 (DM_N); no longer L18.11 (DM_P)
- net ETH2_B_N: now also L18.8 (CM_P); no longer L18.9 (CM_N)
- net ETH2_B_P: now also L18.9 (CM_N); no longer L18.8 (CM_P)
- net ETH2_C_N: now also L18.5 (BM_P); no longer L18.6 (BM_N)
- net ETH2_C_P: now also L18.6 (BM_N); no longer L18.5 (BM_P)
- net ETH2_D_N: now also L18.2 (AM_P); no longer L18.3 (AM_N)
- net ETH2_D_P: now also L18.3 (AM_N); no longer L18.2 (AM_P)
- net ETH3_A_N: now also L19.11 (DM_P); no longer L19.12 (DM_N)
- net ETH3_A_P: now also L19.12 (DM_N); no longer L19.11 (DM_P)
- net ETH3_B_N: now also L19.8 (CM_P); no longer L19.9 (CM_N)
- net ETH3_B_P: now also L19.9 (CM_N); no longer L19.8 (CM_P)
- net ETH3_C_N: now also L19.5 (BM_P); no longer L19.6 (BM_N)
- net ETH3_C_P: now also L19.6 (BM_N); no longer L19.5 (BM_P)
- net ETH3_D_N: now also L19.2 (AM_P); no longer L19.3 (AM_N)
- net ETH3_D_P: now also L19.3 (AM_N); no longer L19.2 (AM_P)
- net SGMII2_TX_C_P: now reaches C55.1, U10.27 (TX_D1/SGMII_TX_P)
- net SGMII2_TX_C_N: now reaches C56.1, U10.28 (TX_D0/SGMII_TX_N)
- net SGMII2_RX_C_P: now reaches C57.1, U10.35 (RX_D2/SGMII_RX_P)
- net SGMII2_RX_C_N: now reaches C58.1, U10.36 (RX_D3/SGMII_RX_N)
- net SGMII3_TX_C_P: now reaches C59.1, U11.27 (TX_D1/SGMII_TX_P)
- net SGMII3_TX_C_N: now reaches C60.1, U11.28 (TX_D0/SGMII_TX_N)
- net SGMII3_RX_C_P: now reaches C61.1, U11.35 (RX_D2/SGMII_RX_P)
- net SGMII3_RX_C_N: now reaches C62.1, U11.36 (RX_D3/SGMII_RX_N)
Changed lines of the file:
@@
 Sheet 3 3
 Title "LATENTRED 8-port 10/100/1000 Base-T Line Card"
-Date "2018-04-25"
+Date "2018-04-26"
 Rev "0.1"
 Comp "Andrew D. Zonenberg"
@@
 Text Notes 3450 11050 0    50   ~ 0
 PHY_ADDR = 5'h1
-Text HLabel 5400 14700 0    50   Input ~ 0
-GND
-Text HLabel 5400 15350 0    50   Input ~ 0
-1V0
-Text HLabel 5400 14900 0    50   Input ~ 0
-1V8
-Text HLabel 5400 14400 0    50   Input ~ 0
-2V5
 Text HLabel 2650 13550 0    50   Input ~ 0
 SGMII2_TX_P
@@
 Wire Wire Line
 	3300 12500 3400 12500
-$Comp
-L passive-azonenberg:INDUCTOR_PWROUT L11
-U 1 1 5B5CE678
-P 6100 14400
-F 0 "L11" V 6050 14150 40  0000 C CNN
-F 1 "600R" V 6050 14650 40  0000 C CNN
-F 2 "azonenberg_pcb:EIA_0402_RES_NOSILK" H 6100 14400 60  0001 C CNN
-F 3 "" H 6100 14400 60  0000 C CNN
-	1    6100 14400
-	0    1    1    0
-$EndComp
 Text Label 3300 12100 2    50   ~ 0
-A1V0_2
+A1V0_3
 Text Label 3300 12500 2    50   ~ 0
-A1V8_2
-$Comp
-L passive-azonenberg:INDUCTOR_PWROUT L13
-U 1 1 5B5CE680
-P 6100 15350
-F 0 "L13" V 6050 15100 40  0000 C CNN
-F 1 "600R" V 6050 15600 40  0000 C CNN
-F 2 "azonenberg_pcb:EIA_0402_RES_NOSILK" H 6100 15350 60  0001 C CNN
-F 3 "" H 6100 15350 60  0000 C CNN
-	1    6100 15350
-	0    1    1    0
-$EndComp
-$Comp
-L passive-azonenberg:INDUCTOR_PWROUT L12
-U 1 1 5B5CE686
-P 6100 14900
-F 0 "L12" V 6050 14650 40  0000 C CNN
-F 1 "600R" V 6050 15150 40  0000 C CNN
-F 2 "azonenberg_pcb:EIA_0402_RES_NOSILK" H 6100 14900 60  0001 C CNN
-F 3 "" H 6100 14900 60  0000 C CNN
-	1    6100 14900
-	0    1    1    0
-$EndComp
+A1V8_3
 Text Label 3300 12700 2    50   ~ 0
 1V8
@@
 Wire Wire Line
 	2650 14450 2850 14450
-$Comp
-L device:C C68
-U 1 1 5B5CE6E0
-P 5500 14550
-F 0 "C68" H 5615 14596 50  0000 L CNN
-F 1 "4.7 uF" H 5615 14505 50  0000 L CNN
-F 2 "azonenberg_pcb:EIA_0603_CAP_NOSILK" H 5538 14400 50  0001 C CNN
-F 3 "" H 5500 14550 50  0001 C CNN
-	1    5500 14550
-	1    0    0    -1
-$EndComp
 Text Label 3300 11900 2    50   ~ 0
-A2V5_2
+A2V5_3
 $Comp
 L device:C C81
@@
 $EndComp
 Wire Wire Line
-	5400 14400 5500 14400
-Wire Wire Line
-	5500 14400 5800 14400
-Connection ~ 5500 14400
-Wire Wire Line
-	6400 14400 6550 14400
-Wire Wire Line
 	6550 14400 7050 14400
-Connection ~ 6550 14400
 Wire Wire Line
 	7050 14400 7600 14400
@@
 	3300 13000 3400 13000
 Wire Wire Line
-	5400 14700 5500 14700
-Wire Wire Line
-	5500 14700 6550 14700
-Connection ~ 5500 14700
-Wire Wire Line
 	7050 14700 6550 14700
-Connection ~ 6550 14700
 Wire Wire Line
 	7050 14700 7600 14700
 Connection ~ 7050 14700
 $Comp
-L device:C C69
-U 1 1 5B5CE70A
-P 5500 15050
-F 0 "C69" H 5615 15096 50  0000 L CNN
-F 1 "4.7 uF" H 5615 15005 50  0000 L CNN
-F 2 "azonenberg_pcb:EIA_0603_CAP_NOSILK" H 5538 14900 50  0001 C CNN
-F 3 "" H 5500 15050 50  0001 C CNN
-	1    5500 15050
-	1    0    0    -1
-$EndComp
-Wire Wire Line
-	5800 14900 5500 14900
-Wire Wire Line
-	5500 14900 5400 14900
-Connection ~ 5500 14900
-Text Label 5400 15200 2    50   ~ 0
-GND
-Wire Wire Line
-	5400 15200 5500 15200
-$Comp
 L device:C C82
 U 1 1 5B5CE715
@@
 $EndComp
 Text Label 7700 14400 0    50   ~ 0
-A2V5_2
+A2V5_3
 Wire Wire Line
 	7700 14400 7600 14400
 Connection ~ 7600 14400
 Text Label 7600 14900 0    50   ~ 0
-A1V8_2
+A1V8_3
 Wire Wire Line
 	7600 14900 7050 14900
-Wire Wire Line
-	6550 14900 6400 14900
-Connection ~ 6550 14900
 $Comp
 L device:C C97
@@
 $EndComp
 Wire Wire Line
-	5500 15200 6550 15200
-Connection ~ 5500 15200
-Wire Wire Line
 	6550 15200 7050 15200
-Connection ~ 6550 15200
 Wire Wire Line
 	7050 15200 7600 15200
 Connection ~ 7050 15200
 $Comp
-L device:C C70
-U 1 1 5B5CE736
-P 5500 15500
-F 0 "C70" H 5615 15546 50  0000 L CNN
-F 1 "4.7 uF" H 5615 15455 50  0000 L CNN
-F 2 "azonenberg_pcb:EIA_0603_CAP_NOSILK" H 5538 15350 50  0001 C CNN
-F 3 "" H 5500 15500 50  0001 C CNN
-	1    5500 15500
-	1    0    0    -1
-$EndComp
-Wire Wire Line
-	5800 15350 5500 15350
-Wire Wire Line
-	5400 15350 5500 15350
-Connection ~ 5500 15350
-$Comp
 L device:C C83
 U 1 1 5B5CE73F
@@
 Wire Wire Line
 	8700 15350 8150 15350
-Wire Wire Line
-	6400 15350 6550 15350
 Connection ~ 8150 15350
-Connection ~ 6550 15350
 Wire Wire Line
 	6550 15350 7050 15350
@@
 	7600 15350 8150 15350
 Wire Wire Line
-	5500 15650 6550 15650
-Connection ~ 6550 15650
-Wire Wire Line
 	6550 15650 7050 15650
 Connection ~ 7050 15650
@@
 	8150 15650 8700 15650
 Text Label 8800 15350 0    50   ~ 0
-A1V0_2
+A1V0_3
 Wire Wire Line
 	8800 15350 8700 15350
@@
 Text Label 5400 13950 2    50   ~ 0
 1V8
-Text Label 5400 15650 2    50   ~ 0
-GND
-Wire Wire Line
-	5400 15650 5500 15650
-Connection ~ 5500 15650
 Text Label 5400 14250 2    50   ~ 0
 GND
@@
 Text Label 21450 7850 0    50   ~ 0
 ETH5_DM_N
-Text Label 8650 17800 2    50   ~ 0
-ETH3_A_P
 Text Label 8650 17900 2    50   ~ 0
+ETH3_A_P
+Text Label 8650 17800 2    50   ~ 0
 ETH3_A_N
-Text Label 8650 17600 2    50   ~ 0
-ETH3_B_P
 Text Label 8650 17700 2    50   ~ 0
+ETH3_B_P
+Text Label 8650 17600 2    50   ~ 0
 ETH3_B_N
-Text Label 8650 17400 2    50   ~ 0
-ETH3_C_P
 Text Label 8650 17500 2    50   ~ 0
+ETH3_C_P
+Text Label 8650 17400 2    50   ~ 0
 ETH3_C_N
-Text Label 8650 17200 2    50   ~ 0
-ETH3_D_P
 Text Label 8650 17300 2    50   ~ 0
+ETH3_D_P
+Text Label 8650 17200 2    50   ~ 0
 ETH3_D_N
 Text Label 9650 17800 0    50   ~ 0
@@
 Text Label 9650 12550 0    50   ~ 0
 ETH2_DM_N
-Text Label 8650 13050 2    50   ~ 0
-ETH2_A_P
 Text Label 8650 13150 2    50   ~ 0
+ETH2_A_P
+Text Label 8650 13050 2    50   ~ 0
 ETH2_A_N
-Text Label 8650 12850 2    50   ~ 0
-ETH2_B_P
 Text Label 8650 12950 2    50   ~ 0
+ETH2_B_P
+Text Label 8650 12850 2    50   ~ 0
 ETH2_B_N
-Text Label 8650 12650 2    50   ~ 0
-ETH2_C_P
 Text Label 8650 12750 2    50   ~ 0
+ETH2_C_P
+Text Label 8650 12650 2    50   ~ 0
 ETH2_C_N
-Text Label 8650 12450 2    50   ~ 0
-ETH2_D_P
 Text Label 8650 12550 2    50   ~ 0
+ETH2_D_P
+Text Label 8650 12450 2    50   ~ 0
 ETH2_D_N
 Text Label 8600 3600 2    50   ~ 0
@@
 Text Label 15100 4250 2    50   ~ 0
 SGMII4_TX_C_N
+Text Label 7600 14700 0    50   ~ 0
+GND
+Text Label 7600 15200 0    50   ~ 0
+GND
+Text Label 8700 15650 0    50   ~ 0
+GND
+Text Label 3300 18350 2    50   ~ 0
+SGMII3_TX_C_P
+Text Label 3300 18450 2    50   ~ 0
+SGMII3_TX_C_N
+Text Label 3300 13600 2    50   ~ 0
+SGMII2_TX_C_P
+Text Label 3300 13700 2    50   ~ 0
+SGMII2_TX_C_N
+Text Label 3300 14300 2    50   ~ 0
+SGMII2_RX_C_P
+Text Label 3300 14400 2    50   ~ 0
+SGMII2_RX_C_N
+Text Label 3300 19050 2    50   ~ 0
+SGMII3_RX_C_P
+Text Label 3300 19150 2    50   ~ 0
+SGMII3_RX_C_N
+Text Notes 8300 18050 0    50   ~ 0
+Swap P/N pairs for easier layout. PHY auto-corrects.
+Text Notes 8300 13300 0    50   ~ 0
+Swap P/N pairs for easier layout. PHY auto-corrects.
 $EndSCHEMATC
