File: latentred/boards/linecard/latentred-linecard/phys.sch (KiCad schematic (older format))
At the start: 376 parts, among them J2 STEWART_SS_74500_024, Q1 SSM6N58NU, Q2 SSM6N58NU, Q3 SSM6N58NU, Q4 SSM6N58NU, Q5 SSM6N58NU, Q6 SSM6N58NU, Q7 SSM6N58NU, Q8 SSM6N58NU, U10 DP83867, U11 DP83867, U12 DP83867, U13 DP83867, U14 DP83867, U15 DP83867, U16 DSC6101CI2A-025.0000, U17 5PB1108CMG, U8 DP83867, U9 DP83867

Commit message: Continued initial line card layout
Connections:
- net ETH0_AM_N: now also L7.3 (AM_N); no longer L7.13 (D_N)
- net ETH0_AM_P: now also L7.2 (AM_P); no longer L7.14 (D_P)
- net ETH0_A_N: now also L7.22 (A_N); no longer L7.11 (DM_P)
- net ETH0_A_P: now also L7.23 (A_P); no longer L7.12 (DM_N)
- net ETH0_BM_N: now also L7.5 (BM_P); no longer L7.16 (C_N)
- net ETH0_BM_P: now also L7.6 (BM_N); no longer L7.17 (C_P)
- net ETH0_B_N: now also L7.19 (B_N); no longer L7.8 (CM_P)
- net ETH0_B_P: now also L7.20 (B_P); no longer L7.9 (CM_N)
- net ETH0_CM_N: now also L7.9 (CM_N); no longer L7.19 (B_N)
- net ETH0_CM_P: now also L7.8 (CM_P); no longer L7.20 (B_P)
- net ETH0_C_N: now also L7.16 (C_N); no longer L7.5 (BM_P)
- net ETH0_C_P: now also L7.17 (C_P); no longer L7.6 (BM_N)
- net ETH0_DM_N: now also L7.11 (DM_P); no longer L7.22 (A_N)
- net ETH0_DM_P: now also L7.12 (DM_N); no longer L7.23 (A_P)
- net ETH0_D_N: now also L7.13 (D_N); no longer L7.2 (AM_P)
- net ETH0_D_P: now also L7.14 (D_P); no longer L7.3 (AM_N)
- net ETH1_AM_N: now also L17.3 (AM_N); no longer L17.13 (D_N)
- net ETH1_AM_P: now also L17.2 (AM_P); no longer L17.14 (D_P)
- net ETH1_A_N: now also L17.22 (A_N); no longer L17.11 (DM_P)
- net ETH1_A_P: now also L17.23 (A_P); no longer L17.12 (DM_N)
- net ETH1_BM_N: now also L17.5 (BM_P); no longer L17.16 (C_N)
- net ETH1_BM_P: now also L17.6 (BM_N); no longer L17.17 (C_P)
- net ETH1_B_N: now also L17.19 (B_N); no longer L17.8 (CM_P)
- net ETH1_B_P: now also L17.20 (B_P); no longer L17.9 (CM_N)
- net ETH1_CM_N: now also L17.9 (CM_N); no longer L17.19 (B_N)
- net ETH1_CM_P: now also L17.8 (CM_P); no longer L17.20 (B_P)
- net ETH1_C_N: now also L17.16 (C_N); no longer L17.5 (BM_P)
- net ETH1_C_P: now also L17.17 (C_P); no longer L17.6 (BM_N)
- net ETH1_DM_N: now also L17.11 (DM_P); no longer L17.22 (A_N)
- net ETH1_DM_P: now also L17.12 (DM_N); no longer L17.23 (A_P)
- net ETH1_D_N: now also L17.13 (D_N); no longer L17.2 (AM_P)
- net ETH1_D_P: now also L17.14 (D_P); no longer L17.3 (AM_N)
- net ETH2_AM_N: now also L18.3 (AM_N); no longer L18.13 (D_N)
- net ETH2_AM_P: now also L18.2 (AM_P); no longer L18.14 (D_P)
- net ETH2_A_N: now also L18.22 (A_N); no longer L18.11 (DM_P)
- net ETH2_A_P: now also L18.23 (A_P); no longer L18.12 (DM_N)
- net ETH2_BM_N: now also L18.5 (BM_P); no longer L18.16 (C_N)
- net ETH2_BM_P: now also L18.6 (BM_N); no longer L18.17 (C_P)
- net ETH2_B_N: now also L18.19 (B_N); no longer L18.8 (CM_P)
- net ETH2_B_P: now also L18.20 (B_P); no longer L18.9 (CM_N)
- net ETH2_CM_N: now also L18.9 (CM_N); no longer L18.19 (B_N)
- net ETH2_CM_P: now also L18.8 (CM_P); no longer L18.20 (B_P)
- net ETH2_C_N: now also L18.16 (C_N); no longer L18.5 (BM_P)
- net ETH2_C_P: now also L18.17 (C_P); no longer L18.6 (BM_N)
- net ETH2_DM_N: now also L18.11 (DM_P); no longer L18.22 (A_N)
- net ETH2_DM_P: now also L18.12 (DM_N); no longer L18.23 (A_P)
- net ETH2_D_N: now also L18.13 (D_N); no longer L18.2 (AM_P)
- net ETH2_D_P: now also L18.14 (D_P); no longer L18.3 (AM_N)
- net ETH3_AM_N: now also L19.3 (AM_N); no longer L19.13 (D_N)
- net ETH3_AM_P: now also L19.2 (AM_P); no longer L19.14 (D_P)
- net ETH3_A_N: now also L19.22 (A_N); no longer L19.11 (DM_P)
- net ETH3_A_P: now also L19.23 (A_P); no longer L19.12 (DM_N)
- net ETH3_BM_N: now also L19.5 (BM_P); no longer L19.16 (C_N)
- net ETH3_BM_P: now also L19.6 (BM_N); no longer L19.17 (C_P)
- net ETH3_B_N: now also L19.19 (B_N); no longer L19.8 (CM_P)
- net ETH3_B_P: now also L19.20 (B_P); no longer L19.9 (CM_N)
- net ETH3_CM_N: now also L19.9 (CM_N); no longer L19.19 (B_N)
- net ETH3_CM_P: now also L19.8 (CM_P); no longer L19.20 (B_P)
- net ETH3_C_N: now also L19.16 (C_N); no longer L19.5 (BM_P)
- net ETH3_C_P: now also L19.17 (C_P); no longer L19.6 (BM_N)
- net ETH3_DM_N: now also L19.11 (DM_P); no longer L19.22 (A_N)
- net ETH3_DM_P: now also L19.12 (DM_N); no longer L19.23 (A_P)
- net ETH3_D_N: now also L19.13 (D_N); no longer L19.2 (AM_P)
- net ETH3_D_P: now also L19.14 (D_P); no longer L19.3 (AM_N)
- net ETH4_AM_N: now also L32.3 (AM_N); no longer L32.13 (D_N)
- net ETH4_AM_P: now also L32.2 (AM_P); no longer L32.14 (D_P)
- net ETH4_A_N: now also L32.22 (A_N); no longer L32.11 (DM_P)
- net ETH4_A_P: now also L32.23 (A_P); no longer L32.12 (DM_N)
- net ETH4_BM_N: now also L32.5 (BM_P); no longer L32.16 (C_N)
- net ETH4_BM_P: now also L32.6 (BM_N); no longer L32.17 (C_P)
- net ETH4_B_N: now also L32.19 (B_N); no longer L32.8 (CM_P)
- net ETH4_B_P: now also L32.20 (B_P); no longer L32.9 (CM_N)
- net ETH4_CM_N: now also L32.9 (CM_N); no longer L32.19 (B_N)
- net ETH4_CM_P: now also L32.8 (CM_P); no longer L32.20 (B_P)
- net ETH4_C_N: now also L32.16 (C_N); no longer L32.5 (BM_P)
- net ETH4_C_P: now also L32.17 (C_P); no longer L32.6 (BM_N)
- net ETH4_DM_N: now also L32.11 (DM_P); no longer L32.22 (A_N)
- net ETH4_DM_P: now also L32.12 (DM_N); no longer L32.23 (A_P)
- net ETH4_D_N: now also L32.13 (D_N); no longer L32.2 (AM_P)
- net ETH4_D_P: now also L32.14 (D_P); no longer L32.3 (AM_N)
- net ETH5_AM_N: now also L33.2 (AM_P); no longer L33.13 (D_N)
- net ETH5_AM_P: now also L33.3 (AM_N); no longer L33.14 (D_P)
- net ETH5_A_N: now also L33.22 (A_N); no longer L33.11 (DM_P)
- net ETH5_A_P: now also L33.23 (A_P); no longer L33.12 (DM_N)
- net ETH5_BM_N: now also L33.5 (BM_P); no longer L33.16 (C_N)
- net ETH5_BM_P: now also L33.6 (BM_N); no longer L33.17 (C_P)
- net ETH5_B_N: now also L33.19 (B_N); no longer L33.8 (CM_P)
- net ETH5_B_P: now also L33.20 (B_P); no longer L33.9 (CM_N)
- net ETH5_CM_N: now also L33.9 (CM_N); no longer L33.19 (B_N)
- net ETH5_CM_P: now also L33.8 (CM_P); no longer L33.20 (B_P)
- net ETH5_C_N: now also L33.16 (C_N); no longer L33.5 (BM_P)
- net ETH5_C_P: now also L33.17 (C_P); no longer L33.6 (BM_N)
- net ETH5_DM_N: now also L33.11 (DM_P); no longer L33.22 (A_N)
- net ETH5_DM_P: now also L33.12 (DM_N); no longer L33.23 (A_P)
- net ETH5_D_N: now also L33.13 (D_N); no longer L33.2 (AM_P)
- net ETH5_D_P: now also L33.14 (D_P); no longer L33.3 (AM_N)
- net ETH6_AM_N: now also L34.3 (AM_N); no longer L34.13 (D_N)
- net ETH6_AM_P: now also L34.2 (AM_P); no longer L34.14 (D_P)
- net ETH6_A_N: now also L34.22 (A_N); no longer L34.11 (DM_P)
- net ETH6_A_P: now also L34.23 (A_P); no longer L34.12 (DM_N)
- net ETH6_BM_N: now also L34.6 (BM_N); no longer L34.16 (C_N)
- net ETH6_BM_P: now also L34.5 (BM_P); no longer L34.17 (C_P)
- net ETH6_B_N: now also L34.19 (B_N); no longer L34.8 (CM_P)
- net ETH6_B_P: now also L34.20 (B_P); no longer L34.9 (CM_N)
- net ETH6_CM_N: now also L34.9 (CM_N); no longer L34.19 (B_N)
- net ETH6_CM_P: now also L34.8 (CM_P); no longer L34.20 (B_P)
- net ETH6_C_N: now also L34.16 (C_N); no longer L34.5 (BM_P)
- net ETH6_C_P: now also L34.17 (C_P); no longer L34.6 (BM_N)
- net ETH6_DM_N: now also L34.11 (DM_P); no longer L34.22 (A_N)
- net ETH6_DM_P: now also L34.12 (DM_N); no longer L34.23 (A_P)
- net ETH6_D_N: now also L34.13 (D_N); no longer L34.2 (AM_P)
- net ETH6_D_P: now also L34.14 (D_P); no longer L34.3 (AM_N)
- net ETH7_AM_N: now also L35.2 (AM_P); no longer L35.13 (D_N)
- net ETH7_AM_P: now also L35.3 (AM_N); no longer L35.14 (D_P)
- net ETH7_A_N: now also L35.22 (A_N); no longer L35.11 (DM_P)
- net ETH7_A_P: now also L35.23 (A_P); no longer L35.12 (DM_N)
- net ETH7_BM_N: now also L35.6 (BM_N); no longer L35.16 (C_N)
- net ETH7_BM_P: now also L35.5 (BM_P); no longer L35.17 (C_P)
- net ETH7_B_N: now also L35.19 (B_N); no longer L35.8 (CM_P)
- net ETH7_B_P: now also L35.20 (B_P); no longer L35.9 (CM_N)
- net ETH7_CM_N: now also L35.8 (CM_P); no longer L35.19 (B_N)
- net ETH7_CM_P: now also L35.9 (CM_N); no longer L35.20 (B_P)
- net ETH7_C_N: now also L35.16 (C_N); no longer L35.5 (BM_P)
- net ETH7_C_P: now also L35.17 (C_P); no longer L35.6 (BM_N)
- net ETH7_DM_N: now also L35.11 (DM_P); no longer L35.22 (A_N)
- net ETH7_DM_P: now also L35.12 (DM_N); no longer L35.23 (A_P)
- net ETH7_D_N: now also L35.13 (D_N); no longer L35.2 (AM_P)
- net ETH7_D_P: now also L35.14 (D_P); no longer L35.3 (AM_N)
- net at L7.1 (AM_CT): now also R29.2; no longer C49.2
- net at L7.10 (DM_CT): now also R32.2; no longer C46.2
- net at L7.15 (D_CT): now also C46.2; no longer R32.2
- net at L7.18 (C_CT): now also C47.2; no longer R31.2
- net at L7.21 (B_CT): now also C48.2; no longer R30.2
- net at L7.24 (A_CT): now also C49.2; no longer R29.2
- net at L7.4 (BM_CT): now also R30.2; no longer C48.2
- net at L7.7 (CM_CT): now also R31.2; no longer C47.2
- net at L17.1 (AM_CT): now also R50.2; no longer C120.2
- net at L17.10 (DM_CT): now also R62.2; no longer C90.2
- net at L17.15 (D_CT): now also C90.2; no longer R62.2
- net at L17.18 (C_CT): now also C102.2; no longer R56.2
- net at L17.21 (B_CT): now also C114.2; no longer R53.2
- net at L17.24 (A_CT): now also C120.2; no longer R50.2
- net at L17.4 (BM_CT): now also R53.2; no longer C114.2
- net at L17.7 (CM_CT): now also R56.2; no longer C102.2
- net at L18.1 (AM_CT): now also R51.2; no longer C121.2
- net at L18.10 (DM_CT): now also R63.2; no longer C91.2
- net at L18.15 (D_CT): now also C91.2; no longer R63.2
- net at L18.18 (C_CT): now also C103.2; no longer R58.2
- net at L18.21 (B_CT): now also C115.2; no longer R54.2
- net at L18.24 (A_CT): now also C121.2; no longer R51.2
- net at L18.4 (BM_CT): now also R54.2; no longer C115.2
- net at L18.7 (CM_CT): now also R58.2; no longer C103.2
- net at L19.1 (AM_CT): now also R52.2; no longer C122.2
- net at L19.10 (DM_CT): now also R64.2; no longer C92.2
- net at L19.15 (D_CT): now also C92.2; no longer R64.2
- net at L19.18 (C_CT): now also C104.2; no longer R60.2
- net at L19.21 (B_CT): now also C116.2; no longer R55.2
- net at L19.24 (A_CT): now also C122.2; no longer R52.2
- net at L19.4 (BM_CT): now also R55.2; no longer C116.2
- net at L19.7 (CM_CT): now also R60.2; no longer C104.2
- net at L32.1 (AM_CT): now also R111.2; no longer C221.2
- net at L32.10 (DM_CT): now also R127.2; no longer C181.2
- net at L32.15 (D_CT): now also C181.2; no longer R127.2
- net at L32.18 (C_CT): now also C197.2; no longer R119.2
- net at L32.21 (B_CT): now also C213.2; no longer R115.2
- net at L32.24 (A_CT): now also C221.2; no longer R111.2
- net at L32.4 (BM_CT): now also R115.2; no longer C213.2
- net at L32.7 (CM_CT): now also R119.2; no longer C197.2
- net at L33.1 (AM_CT): now also R112.2; no longer C222.2
- net at L33.10 (DM_CT): now also R128.2; no longer C182.2
- net at L33.15 (D_CT): now also C182.2; no longer R128.2
- net at L33.18 (C_CT): now also C198.2; no longer R121.2
- net at L33.21 (B_CT): now also C214.2; no longer R116.2
- net at L33.24 (A_CT): now also C222.2; no longer R112.2
- net at L33.4 (BM_CT): now also R116.2; no longer C214.2
- net at L33.7 (CM_CT): now also R121.2; no longer C198.2
- net at L34.1 (AM_CT): now also R113.2; no longer C223.2
- net at L34.10 (DM_CT): now also R129.2; no longer C183.2
- net at L34.15 (D_CT): now also C183.2; no longer R129.2
- net at L34.18 (C_CT): now also C199.2; no longer R123.2
- net at L34.21 (B_CT): now also C215.2; no longer R117.2
- net at L34.24 (A_CT): now also C223.2; no longer R113.2
- net at L34.4 (BM_CT): now also R117.2; no longer C215.2
- net at L34.7 (CM_CT): now also R123.2; no longer C199.2
- net at L35.1 (AM_CT): now also R114.2; no longer C224.2
- net at L35.10 (DM_CT): now also R130.2; no longer C184.2
- net at L35.15 (D_CT): now also C184.2; no longer R130.2
- net at L35.18 (C_CT): now also C200.2; no longer R125.2
- net at L35.21 (B_CT): now also C216.2; no longer R118.2
- net at L35.24 (A_CT): now also C224.2; no longer R114.2
- net at L35.4 (BM_CT): now also R118.2; no longer C216.2
- net at L35.7 (CM_CT): now also R125.2; no longer C200.2
Other:
- note removed: "TODO: R/C between shield and ground"
