File: latentred/boards/linecard/latentred-linecard/psu.sch (KiCad schematic (older format))
At the start: 40 parts, among them U1 MCP1703T-3302E, U2 LTC3374-QFN, U3 SI7050, U4 LTC2451, U5 INA226, U6 INA226, U7 INA226

Commit message: Continued work on line card design. Now have PSU and all PHYs, still working on clock distribution.
Parts:
- added C33, C34, C36, C38, C39, C42, C44, C45: 47 uF, symbol device:C
- added C35, C37, C43: 4.7 uF, symbol device:C
- added C40, C41: 0.47 uF, symbol device:C
Connections:
- net 3V3: now also C37.1, C40.1
- net 5V0: now also C33.1, C35.1, C36.1, C38.1, C41.1, C43.1
- net GND: now also C33.2, C34.2, C35.2, C36.2, C37.2, C38.2, C39.2, C40.2, C41.2, C42.2, C43.2, C44.2, C45.2
- net 1V0_DECOUPLE: now reaches L1.2, R7.4 (Vi)
- net 1V0_DECOUPLE: now also C44.1, C45.1
- net 2V5_DECOUPLE: now reaches L2.2, R8.4 (Vi)
- net 2V5_DECOUPLE: now also C39.1, C42.1
- net 1V8_DECOUPLE: now reaches L3.2, R9.4 (Vi)
- net 1V8_DECOUPLE: now also C34.1
Other:
- note added: "0805 size"
- note added: "1210 size"
- note added: "SMPS input caps"
- note added: "SMPS output caps"

Commit message: Finished initial version of LATENTRED line card schematic. Not yet reviewed.
Parts:
- added R152, R153, R154: 10K, symbol device:R
Connections:
- net 1V0_DECOUPLE: now also L1.1; no longer L1.2
- net 1V0_EN: now also R152.2
- net 1V0_SW: now also L1.2; no longer L1.1
- net 1V8_DECOUPLE: now also L3.1; no longer L3.2
- net 1V8_EN: now also R153.2
- net 1V8_SW: now also L3.2; no longer L3.1
- net 2V5_DECOUPLE: now also L2.1; no longer L2.2
- net 2V5_EN: now also R154.2
- net 2V5_SW: now also L2.2; no longer L2.1
- net GND: now also R152.1, R153.1, R154.1
Other:
- note removed: "TODO: Input caps\n10 uF input, 22 uF output (per channel)\n\n2ch: 22 / 47 uF\nProbably also should get a cap at Vcc"
- moved on the sheet: L1, L2, L3
Changed lines of the file:
@@
 U 1 1 5AD4397D
 P 5750 2700
-F 0 "L1" V 5595 2700 40  0000 C CNN
-F 1 "NR6028T2R2N" V 5671 2700 40  0000 C CNN
+F 0 "L1" V 5900 2900 40  0000 C CNN
+F 1 "NR6028T2R2N" V 5850 2700 40  0000 C CNN
 F 2 "" H 5750 2700 60  0000 C CNN
 F 3 "" H 5750 2700 60  0000 C CNN
 	1    5750 2700
-	0    1    1    0
+	0    -1   -1   0
 $EndComp
 Text Label 6550 2500 2    50   ~ 0
@@
 Wire Wire Line
 	6550 6700 6650 6700
-Text Notes 7350 1100 0    50   ~ 0
-TODO: Input caps\n10 uF input, 22 uF output (per channel)\n\n2ch: 22 / 47 uF\nProbably also should get a cap at Vcc
 Text HLabel 9700 1900 2    50   Output ~ 0
 PGOOD
@@
 U 1 1 5AD494EC
 P 5750 4500
-F 0 "L2" V 5595 4500 40  0000 C CNN
-F 1 "NR6028T2R2N" V 5671 4500 40  0000 C CNN
+F 0 "L2" V 5950 4600 40  0000 C CNN
+F 1 "NR6028T2R2N" V 5850 4500 40  0000 C CNN
 F 2 "" H 5750 4500 60  0000 C CNN
 F 3 "" H 5750 4500 60  0000 C CNN
 	1    5750 4500
-	0    1    1    0
+	0    -1   -1   0
 $EndComp
 $Comp
@@
 U 1 1 5AD49C68
 P 5750 6300
-F 0 "L3" V 5595 6300 40  0000 C CNN
-F 1 "NR6028T2R2N" V 5671 6300 40  0000 C CNN
+F 0 "L3" V 5950 6450 40  0000 C CNN
+F 1 "NR6028T2R2N" V 5850 6300 40  0000 C CNN
 F 2 "" H 5750 6300 60  0000 C CNN
 F 3 "" H 5750 6300 60  0000 C CNN
 	1    5750 6300
-	0    1    1    0
+	0    -1   -1   0
 $EndComp
 $Comp
@@
 Text Notes 1200 1250 0    50   ~ 0
 0805 size
+Text Label 11050 2300 2    50   ~ 0
+1V0_EN
+$Comp
+L device:R R152
+U 1 1 68FFFDEA
+P 11300 2300
+F 0 "R152" V 11250 2550 50  0000 C CNN
+F 1 "10K" V 11300 2300 50  0000 C CNN
+F 2 "" V 11230 2300 50  0001 C CNN
+F 3 "" H 11300 2300 50  0001 C CNN
+	1    11300 2300
+	0    1    1    0
+$EndComp
+Text Label 11050 2550 2    50   ~ 0
+1V8_EN
+$Comp
+L device:R R153
+U 1 1 69002ADA
+P 11300 2550
+F 0 "R153" V 11250 2800 50  0000 C CNN
+F 1 "10K" V 11300 2550 50  0000 C CNN
+F 2 "" V 11230 2550 50  0001 C CNN
+F 3 "" H 11300 2550 50  0001 C CNN
+	1    11300 2550
+	0    1    1    0
+$EndComp
+$Comp
+L device:R R154
+U 1 1 69002B6E
+P 11300 2800
+F 0 "R154" V 11250 3050 50  0000 C CNN
+F 1 "10K" V 11300 2800 50  0000 C CNN
+F 2 "" V 11230 2800 50  0001 C CNN
+F 3 "" H 11300 2800 50  0001 C CNN
+	1    11300 2800
+	0    1    1    0
+$EndComp
+Text Label 11050 2800 2    50   ~ 0
+2V5_EN
+Wire Wire Line
+	11050 2800 11150 2800
+Wire Wire Line
+	11050 2550 11150 2550
+Wire Wire Line
+	11050 2300 11150 2300
+Text Label 11650 2300 0    50   ~ 0
+GND
+Wire Wire Line
+	11650 2300 11450 2300
+Text Label 11650 2550 0    50   ~ 0
+GND
+Wire Wire Line
+	11650 2550 11450 2550
+Text Label 11650 2800 0    50   ~ 0
+GND
+Wire Wire Line
+	11650 2800 11450 2800
 $EndSCHEMATC

Commit message: Finished initial footprint creation, ready to begin layout
Parts:
- C1, C10, C11, C40, C41, C5, C6, C7: footprint (none) -> azonenberg_pcb:EIA_0402_CAP_NOSILK
- C2, C3: value C -> 0.47 uF; footprint (none) -> azonenberg_pcb:EIA_0402_CAP_NOSILK
- C33, C36, C38, C39, C42: footprint (none) -> azonenberg_pcb:EIA_1210_CAP_NOSILK
- C34, C44, C45: footprint (none) -> azonenberg_pcb:EIA_0805_CAP_NOSILK
- C35, C37, C4, C43, C8, C9: footprint (none) -> azonenberg_pcb:EIA_0603_CAP_NOSILK
- L1, L2, L3: footprint (none) -> azonenberg_pcb:INDUCTOR_YUDEN_NR6028
- R1, R10, R11, R12, R13, R14, R15, R152, R153, R154, R16, R17, R18, R19, R2, R3, R4, R5, R6: footprint (none) -> azonenberg_pcb:EIA_0402_RES_NOSILK
- R7, R8, R9: footprint (none) -> azonenberg_pcb:OHMITE_LVK12
- U1: footprint (none) -> azonenberg_pcb:DFN_8_0.5MM_3x3MM
- U2: footprint (none) -> azonenberg_pcb:QFN_38_0.5MM_5x7MM
- U3: footprint (none) -> azonenberg_pcb:DFN_6_1MM_3x3MM
- U4: footprint (none) -> azonenberg_pcb:DFN_8_0.5MM_2x3MM
- U5, U6, U7: footprint (none) -> azonenberg_pcb:SOP_10_0.5MM_3MM
