File: latentred/boards/testing/magnetic-crosstalk/magnetic-crosstalk/magnetic-crosstalk.sch (KiCad schematic (older format))
At the start: 41 parts, among them J1 STEWART_SS_74500_024, J2 SMA, J3 SMA, J4 SMA, J5 SMA, J6 SMA, J7 SMA, J8 SMA, J9 SMA

Commit message: Finished initial version of crosstalk characterization board
Parts:
- added unit 4 of J1
- added unit 3 of J1
- added unit 6 of J1
- added unit 5 of J1
- added R15, R16, R17, R18, R19, R20, R21, R22: 953, azonenberg_pcb:EIA_0402_RES_NOSILK, symbol device:R
- added R23, R24, R25, R26, R27, R28, R29, R30, R31, R32, R33, R34, R35, R36, R37, R38, R47, R48, R49, R50, R51, R52, R53, R54, R55, R56, R57, R58, R59, R60, R61, R62: 34.8, azonenberg_pcb:EIA_0402_RES_NOSILK, symbol device:R
- added R39, R40, R41, R42, R43, R44, R45, R46: 36.5, azonenberg_pcb:EIA_0402_RES_NOSILK, symbol device:R
Connections:
- net A_N: now also R16.1; no longer J3.1 (In)
- net A_P: now also R15.1; no longer J2.1 (In)
- net B_N: now also R18.1; no longer J5.1 (In)
- net B_P: now also R17.1; no longer J4.1 (In)
- net C_N: now also R20.1; no longer J7.1 (In)
- net C_P: now also R19.1; no longer J6.1 (In)
- net D_N: now also R22.1; no longer J9.1 (In)
- net D_P: now also R21.1; no longer J8.1 (In)
- new net: J2.1 (In), R15.2
- new net: J3.1 (In), R16.2
- new net: J4.1 (In), R17.2
- new net: J5.1 (In), R18.2
- new net: J6.1 (In), R19.2
- new net: J7.1 (In), R20.2
- new net: J8.1 (In), R21.2
- new net: J9.1 (In), R22.2
- new net A1X_A_N: J1.D2 (A_N), R48.1
- new net A1X_A_P: J1.D1 (A_P), R47.1
- new net A1X_B_N: J1.D4 (B_N), R50.1
- new net A1X_B_P: J1.D3 (B_P), R49.1
- new net A1X_C_N: J1.D6 (C_N), R52.1
- new net A1X_C_P: J1.D5 (C_P), R51.1
- new net A1X_D_N: J1.D8 (D_N), R54.1
- new net A1X_D_P: J1.D7 (D_P), R53.1
- new net A1Y_A_N: R24.1, R39.1, R48.2
- new net A1Y_A_P: R23.1, R39.2, R47.2
- new net A1Y_B_N: R26.1, R40.1, R50.2
- new net A1Y_B_P: R25.1, R40.2, R49.2
- new net A1Y_C_N: R28.1, R41.1, R52.2
- new net A1Y_C_P: R27.1, R41.2, R51.2
- new net A1Y_D_N: R30.1, R42.1, R54.2
- new net A1Y_D_P: R29.1, R42.2, R53.2
- new net A1_A_N: J1.E2 (A_N), R24.2
- new net A1_A_P: J1.E1 (A_P), R23.2
- new net A1_B_N: J1.E4 (B_N), R26.2
- new net A1_B_P: J1.E3 (B_P), R25.2
- new net A1_C_N: J1.E6 (C_N), R28.2
- new net A1_C_P: J1.E5 (C_P), R27.2
- new net A1_D_N: J1.E8 (D_N), R30.2
- new net A1_D_P: J1.E7 (D_P), R29.2
- new net A2X_A_N: J1.F2 (A_N), R56.1
- new net A2X_A_P: J1.F1 (A_P), R55.1
- new net A2X_B_N: J1.F4 (B_N), R58.1
- new net A2X_B_P: J1.F3 (B_P), R57.1
- new net A2X_C_N: J1.F6 (C_N), R60.1
- new net A2X_C_P: J1.F5 (C_P), R59.1
- new net A2X_D_N: J1.F8 (D_N), R62.1
- new net A2X_D_P: J1.F7 (D_P), R61.1
- new net A2Y_A_N: R32.1, R43.1, R56.2
- new net A2Y_A_P: R31.1, R43.2, R55.2
- new net A2Y_B_N: R34.1, R44.1, R58.2
- new net A2Y_B_P: R33.1, R44.2, R57.2
- new net A2Y_C_N: R36.1, R45.1, R60.2
- new net A2Y_C_P: R35.1, R45.2, R59.2
- new net A2Y_D_N: R38.1, R46.1, R62.2
- new net A2Y_D_P: R37.1, R46.2, R61.2
- new net A2_A_N: J1.C2 (A_N), R32.2
- new net A2_A_P: J1.C1 (A_P), R31.2
- new net A2_B_N: J1.C4 (B_N), R34.2
- new net A2_B_P: J1.C3 (B_P), R33.2
- new net A2_C_N: J1.C6 (C_N), R36.2
- new net A2_C_P: J1.C5 (C_P), R35.2
- new net A2_D_N: J1.C8 (D_N), R38.2
- new net A2_D_P: J1.C7 (D_P), R37.2
- no-connect marks 12 -> 28
Other:
- note added: "15 dB attenuators for victim signal"
- note added: "SMA test points for victim port"
- note added: "Shield and mechanical"
- moved on the sheet: C2, C3, C4, C5, C6, C7, C8, J1B, J1I, J2, J3, J4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

Commit message: Began updating magnetic-crosstalk board for v0.2
Connections:
- net AGG_A_N: now also L1.3 (AM_N); no longer L1.22 (A_N)
- net AGG_A_P: now also L1.2 (AM_P); no longer L1.23 (A_P)
- net AGG_B_N: now also L1.6 (BM_N); no longer L1.19 (B_N)
- net AGG_B_P: now also L1.5 (BM_P); no longer L1.20 (B_P)
- net AGG_C_N: now also L1.9 (CM_N); no longer L1.16 (C_N)
- net AGG_C_P: now also L1.8 (CM_P); no longer L1.17 (C_P)
- net AGG_D_N: now also L1.11 (DM_P); no longer L1.14 (D_P)
- net AGG_D_P: now also L1.12 (DM_N); no longer L1.13 (D_N)
- net A_N: now also L2.22 (A_N); no longer L2.3 (AM_N)
- net A_P: now also L2.23 (A_P); no longer L2.2 (AM_P)
- net B_N: now also L2.19 (B_N); no longer L2.6 (BM_N)
- net B_P: now also L2.20 (B_P); no longer L2.5 (BM_P)
- net C_N: now also L2.16 (C_N); no longer L2.9 (CM_N)
- net C_P: now also L2.17 (C_P); no longer L2.8 (CM_P)
- net D_N: now also L2.14 (D_P); no longer L2.11 (DM_P)
- net D_P: now also L2.13 (D_N); no longer L2.12 (DM_N)
- net VIC_A_N: now also L2.3 (AM_N); no longer L2.22 (A_N)
- net VIC_A_P: now also L2.2 (AM_P); no longer L2.23 (A_P)
- net VIC_B_N: now also L2.6 (BM_N); no longer L2.19 (B_N)
- net VIC_B_P: now also L2.5 (BM_P); no longer L2.20 (B_P)
- net VIC_C_N: now also L2.9 (CM_N); no longer L2.16 (C_N)
- net VIC_C_P: now also L2.8 (CM_P); no longer L2.17 (C_P)
- net VIC_D_N: now also L2.11 (DM_P); no longer L2.14 (D_P)
- net VIC_D_P: now also L2.12 (DM_N); no longer L2.13 (D_N)
- net at L1.1 (AM_CT): now also R3.2; no longer C12.2
- net at L1.10 (DM_CT): now also R6.2; no longer C9.2
- net at R2.1: now also L1.14 (D_P); no longer L1.11 (DM_P)
- net at R2.2: now also L1.13 (D_N); no longer L1.12 (DM_N)
- net at L1.15 (D_CT): now also C9.2; no longer R6.2
- net at L1.18 (C_CT): now also C10.2; no longer R5.2
- net at L1.21 (B_CT): now also C11.2; no longer R4.2
- net at L1.24 (A_CT): now also C12.2; no longer R3.2
- net at L1.4 (BM_CT): now also R4.2; no longer C11.2
- net at L1.7 (CM_CT): now also R5.2; no longer C10.2
- net at R1.1: now also L1.17 (C_P); no longer L1.8 (CM_P)
- net at R1.2: now also L1.16 (C_N); no longer L1.9 (CM_N)
- net at L2.1 (AM_CT): now also R11.2; no longer C7.2
- net at L2.10 (DM_CT): now also R14.2; no longer C4.2
- net at L2.15 (D_CT): now also C4.2; no longer R14.2
- net at L2.18 (C_CT): now also C5.2; no longer R13.2
- net at L2.21 (B_CT): now also C6.2; no longer R12.2
- net at L2.24 (A_CT): now also C7.2; no longer R11.2
- net at L2.4 (BM_CT): now also R12.2; no longer C6.2
- net at L2.7 (CM_CT): now also R13.2; no longer C5.2
- new net: L1.19 (B_N), L1.22 (A_N)
- new net: L1.20 (B_P), L1.23 (A_P)
Changed lines of the file:
@@
 EESchema Schematic File Version 4
+LIBS:magnetic-crosstalk-cache
 EELAYER 26 0
 EELAYER END
@@
 Sheet 1 1
 Title "Ethernet Magnetic EMC Characterization Board"
-Date "2018-04-30"
-Rev "0.1"
+Date "2018-05-14"
+Rev "0.2"
 Comp "Andrew D. Zonenberg"
 Comment1 ""
@@
 L special-azonenberg:BOURNS_PT6120EL L1
 U 1 1 5AE6D5A4
-P 2300 2300
-F 0 "L1" H 2700 3875 50  0000 C CNN
-F 1 "BOURNS_PT6120EL" H 2700 3784 50  0000 C CNN
-F 2 "azonenberg_pcb:BOURNS_PT61020EL" H 2350 2250 50  0001 C CNN
-F 3 "" H 2350 2250 50  0001 C CNN
-	1    2300 2300
-	1    0    0    -1
+P 3100 2300
+F 0 "L1" H 3500 3875 50  0000 C CNN
+F 1 "BOURNS_PT6120EL" H 3500 3784 50  0000 C CNN
+F 2 "azonenberg_pcb:BOURNS_PT61020EL" H 3150 2250 50  0001 C CNN
+F 3 "" H 3150 2250 50  0001 C CNN
+	1    3100 2300
+	-1   0    0    -1
 $EndComp
 $Comp
@@
 L special-azonenberg:BOURNS_PT6120EL L2
 U 1 1 5AE6F7DC
-P 12700 2700
-F 0 "L2" H 13100 4275 50  0000 C CNN
-F 1 "BOURNS_PT6120EL" H 13100 4184 50  0000 C CNN
-F 2 "azonenberg_pcb:BOURNS_PT61020EL" H 12750 2650 50  0001 C CNN
-F 3 "" H 12750 2650 50  0001 C CNN
-	1    12700 2700
-	1    0    0    -1
+P 13500 2700
+F 0 "L2" H 13900 4275 50  0000 C CNN
+F 1 "BOURNS_PT6120EL" H 13900 4184 50  0000 C CNN
+F 2 "azonenberg_pcb:BOURNS_PT61020EL" H 13550 2650 50  0001 C CNN
+F 3 "" H 13550 2650 50  0001 C CNN
+	1    13500 2700
+	-1   0    0    -1
 $EndComp
 NoConn ~ 14450 2850
@@
 $EndComp
 Wire Wire Line
-	12600 1650 11150 1650
+	12600 1650 11800 1650
 Wire Wire Line
 	11150 1350 11150 1050
@@
 	11600 1050 12000 1050
 Wire Wire Line
-	11600 1550 12600 1550
+	11600 1550 11800 1550
 $Comp
 L device:R R7
@@
 $EndComp
 Wire Wire Line
-	2200 1250 750  1250
-Wire Wire Line
 	750  950  750  650
 Connection ~ 2000 650
@@
 Wire Wire Line
 	1200 650  1600 650
-Wire Wire Line
-	1200 1150 2200 1150
 Text Notes 12700 2950 0    50   ~ 0
 VICTIM port\nTerminations plus test points\nSwap A/B/C/D pairs for easier routing
@@
 NoConn ~ 1950 4500
 NoConn ~ 1950 6600
+Wire Wire Line
+	750  1250 2200 1250
+Wire Wire Line
+	1200 1150 2200 1150
+Connection ~ 11800 1650
+Wire Wire Line
+	11800 1650 11150 1650
+Connection ~ 11800 1550
+Wire Wire Line
+	11800 1550 12600 1550
 $EndSCHEMATC
