File: latentred/boards/switchengine/ram.sch (KiCad schematic (older format))
At the start: 0 parts

Commit message: Continued initial work on switch engine schematic and power budgeting
Parts:
- added U? (x4): CY7C2245KV18-450BZKI, symbol memory-azonenberg:QDRII+_SRAM_36BIT
- added U?: XC7KxT-FBG484, symbol xilinx-azonenberg:XC7KxT-FBG484
Connections:
- new net QDR_BWS0_N: U?.B7 (BWS_0_N)
- new net QDR_BWS1_N: U?.A7 (BWS_1_N)
- new net QDR_BWS2_N: U?.A5 (BWS_2_N)
- new net QDR_BWS3_N: U?.B5 (BWS_3_N)
- new net QDR_CLK_N: U?.T16 (IO_L20N_T3_13)
- new net QDR_CLK_P: U?.R16 (IO_L20P_T3_13)
- new net QDR_D0: U?.P10 (D0), U?.T21 (IO_L1P_T0_13)
- new net QDR_D1: U?.N11 (D1), U?.U21 (IO_L1N_T0_13)
- new net QDR_D2: U?.M11 (D2), U?.U22 (IO_L2P_T0_13)
- new net QDR_D3: U?.K10 (D3), U?.V22 (IO_L2N_T0_13)
- new net QDR_D4: U?.J11 (D4), U?.W21 (IO_L4P_T0_13)
- new net QDR_D5: U?.G11 (D5), U?.W22 (IO_L4N_T0_13)
- new net QDR_D6: U?.E10 (D6), U?.U17 (IO_L5P_T0_13)
- new net QDR_D7: U?.D11 (D7), U?.V18 (IO_L5N_T0_13)
- new net QDR_D8: U?.C11 (D8), U?.T20 (IO_L6P_T0_13)
- new net QDR_WPS_N: U?.A4 (WPS_N)
- no-connect marks 0 -> 3
Changed lines of the file:
@@
 EELAYER 30 0
 EELAYER END
-$Descr A4 11693 8268
+$Descr A3 16535 11693
 encoding utf-8
-Sheet 1 5
-Title ""
-Date ""
-Rev ""
-Comp ""
-Comment1 ""
-Comment2 ""
+Sheet 5 6
+Title "LATENTRED Switch Engine"
+Date "2019-09-09"
+Rev "0.1"
+Comp "Antikernel Labs"
+Comment1 "QDR-II+ SRAM"
+Comment2 "Andrew D. Zonenberg"
 Comment3 ""
 Comment4 ""
 $EndDescr
+$Comp
+L memory-azonenberg:QDRII+_SRAM_36BIT U?
+U 1 1 5D78F9C5
+P 4200 6300
+F 0 "U?" H 4200 6200 60  0000 L CNN
+F 1 "CY7C2245KV18-450BZKI" H 4200 6100 60  0000 L CNN
+F 2 "" H 4200 6300 60  0000 C CNN
+F 3 "" H 4200 6300 60  0000 C CNN
+	1    4200 6300
+	1    0    0    -1
+$EndComp
+$Comp
+L memory-azonenberg:QDRII+_SRAM_36BIT U?
+U 2 1 5D794EA0
+P 8850 6150
+F 0 "U?" H 8850 6050 60  0000 L CNN
+F 1 "CY7C2245KV18-450BZKI" H 8850 5950 60  0000 L CNN
+F 2 "" H 8850 6150 60  0000 C CNN
+F 3 "" H 8850 6150 60  0000 C CNN
+	2    8850 6150
+	1    0    0    -1
+$EndComp
+$Comp
+L memory-azonenberg:QDRII+_SRAM_36BIT U?
+U 3 1 5D79766A
+P 11400 6150
+F 0 "U?" H 11400 6050 60  0000 L CNN
+F 1 "CY7C2245KV18-450BZKI" H 11400 5950 60  0000 L CNN
+F 2 "" H 11400 6150 60  0000 C CNN
+F 3 "" H 11400 6150 60  0000 C CNN
+	3    11400 6150
+	1    0    0    -1
+$EndComp
+$Comp
+L memory-azonenberg:QDRII+_SRAM_36BIT U?
+U 4 1 5D79BC70
+P 14050 6150
+F 0 "U?" H 14050 6050 60  0000 L CNN
+F 1 "CY7C2245KV18-450BZKI" H 14050 5950 60  0000 L CNN
+F 2 "" H 14050 6150 60  0000 C CNN
+F 3 "" H 14050 6150 60  0000 C CNN
+	4    14050 6150
+	1    0    0    -1
+$EndComp
+$Comp
+L xilinx-azonenberg:XC7KxT-FBG484 U?
+U 3 1 5D7AACCB
+P 2450 7000
+F 0 "U?" H 2450 6900 60  0000 L CNN
+F 1 "XC7KxT-FBG484" H 2450 6800 60  0000 L CNN
+F 2 "" H 2450 6700 60  0000 C CNN
+F 3 "" H 2450 6700 60  0000 C CNN
+	3    2450 7000
+	-1   0    0    -1
+$EndComp
+Text Label 2650 2200 0    50   ~ 0
+QDR_D0
+Text Label 2650 2300 0    50   ~ 0
+QDR_D1
+Text Label 2650 2400 0    50   ~ 0
+QDR_D2
+Text Label 2650 2500 0    50   ~ 0
+QDR_D3
+Text Label 2650 2800 0    50   ~ 0
+QDR_D4
+Text Label 2650 2900 0    50   ~ 0
+QDR_D5
+Text Label 2650 3000 0    50   ~ 0
+QDR_D6
+Text Label 2650 3100 0    50   ~ 0
+QDR_D7
+Text Label 2650 3200 0    50   ~ 0
+QDR_D8
+NoConn ~ 2650 2700
+NoConn ~ 2650 2600
+Text Label 7000 2300 2    50   ~ 0
+QDR_WPS_N
+Text Label 4000 2100 2    50   ~ 0
+QDR_WPS_N
+NoConn ~ 2650 2100
+Text Label 2650 6000 0    50   ~ 0
+QDR_CLK_P
+Text Label 2650 6100 0    50   ~ 0
+QDR_CLK_N
+Text Label 4000 2800 2    50   ~ 0
+QDR_D0
+Text Label 4000 2900 2    50   ~ 0
+QDR_D1
+Text Label 4000 3000 2    50   ~ 0
+QDR_D2
+Text Label 4000 3100 2    50   ~ 0
+QDR_D3
+Text Label 4000 3200 2    50   ~ 0
+QDR_D4
+Text Label 4000 3300 2    50   ~ 0
+QDR_D5
+Text Label 4000 3400 2    50   ~ 0
+QDR_D6
+Text Label 4000 3500 2    50   ~ 0
+QDR_D7
+Text Label 4000 3600 2    50   ~ 0
+QDR_D8
+Text Label 4000 2300 2    50   ~ 0
+QDR_BWS0_N
+Text Label 4000 2400 2    50   ~ 0
+QDR_BWS1_N
+Text Label 4000 2500 2    50   ~ 0
+QDR_BWS2_N
+Text Label 4000 2600 2    50   ~ 0
+QDR_BWS3_N
+Text Label 7000 2400 2    50   ~ 0
+QDR_BWS0_N
+Text Label 7000 2500 2    50   ~ 0
+QDR_BWS1_N
+Text Label 7000 2600 2    50   ~ 0
+QDR_BWS2_N
+Text Label 7000 2700 2    50   ~ 0
+QDR_BWS3_N
 $EndSCHEMATC
