File: latentpink/pcb/sgmii.kicad_sch (KiCad schematic)
At the start: 62 parts, among them J22 BEL_FUSE_0845-2R1T-E4, U2 XC7K160T-2FBG484C, U5 DP83867, U6 DP83867, U7 TBD, U8 TBD

Commit message: Continued footprint assignment and miscellaneous missing tidbits of schematic
Parts:
- added C450, C451, C452, C453, C454, C455, C456, C457: 0.1 uF, azonenberg_pcb:EIA_0402_CAP_NOSILK, symbol device:C
- added D6, D7: GREEN, azonenberg_pcb:EIA_0603_LED, symbol device:LED
- added R137, R141: 5.76K, azonenberg_pcb:EIA_0402_RES_NOSILK, symbol device:R
- added R138, R140, R142, R144, R146, R148: 2.49K, azonenberg_pcb:EIA_0402_RES_NOSILK, symbol device:R
- added R139, R143, R145, R147: 10K, azonenberg_pcb:EIA_0402_RES_NOSILK, symbol device:R
- added R149, R150, R151, R152, R153, R154: 470, azonenberg_pcb:EIA_0402_RES_NOSILK, symbol device:R
- R117, R118: footprint (none) -> azonenberg_pcb:EIA_0402_RES_NOSILK
- TP21, TP22: footprint (none) -> azonenberg_pcb:TESTPOINT_SMT_0.5MM
- U7, U8: value TBD -> ECS-1612MV-250-CN-TR; footprint (none) -> azonenberg_pcb:OSCILLATOR_1.6x1.2
Connections:
- net 1V8: now also R137.2, R139.2, R141.2, R143.2, R145.2, R147.2
- net ETH12_RX_CTRL_STRAP: now also R137.1, R138.1
- net ETH13_RX_CTRL_STRAP: now also R141.1, R142.1
- net ETH13_SGMII_CLKOUT_AC_N: now also U2.Y9 (IO_L13N_T2_MRCC_33)
- net ETH13_SGMII_CLKOUT_AC_P: now also U2.W9 (IO_L13P_T2_MRCC_33)
- net ETH13_SGMII_CLKOUT_N: now also R147.1, R148.1
- net ETH13_SGMII_CLKOUT_P: now also R145.1, R146.1
- net ETH13_SGMII_RX_AC_N: now also U2.AA8 (IO_L5N_T0_33)
- net ETH13_SGMII_RX_AC_P: now also U2.AA9 (IO_L5P_T0_33)
- net ETH13_SGMII_TX_AC_N: now also U2.AB10 (IO_L4N_T0_33)
- net ETH13_SGMII_TX_AC_P: now also U2.AA10 (IO_L4P_T0_33)
- net GND: now also J22.27 (LED1_N), J22.29 (LED2_G_N), J22.31 (LED1_N), J22.33 (LED2_G_N), C450.2, C451.2, C452.2, C453.2, C454.2, C455.2, C456.2, C457.2, D6.1 (K), D7.1 (K), R138.2, R140.2, R142.2, R144.2, R146.2, R148.2
- net ETH13_B_TAP: now reaches J22.12 (BI_DB_TAP)
- net ETH13_B_TAP: now also C455.1
- net at J22.32 (LED1_P): now also R151.2
- net at J22.34 (LED2_G_P): now also R152.2
- net ETH13_C_TAP: now reaches J22.4 (BI_DC_TAP)
- net ETH13_C_TAP: now also C456.1
- net ETH13_A_TAP: now reaches J22.7 (BI_DA_TAP)
- net ETH13_A_TAP: now also C454.1
- net ETH13_D_TAP: now reaches J22.8 (BI_DD_TAP)
- net ETH13_D_TAP: now also C457.1
- net ETH12_GPIO_0: now reaches U6.39 (GPIO_0)
- net ETH12_GPIO_0: now also U2.T10 (IO_L16N_T2_33)
- net ETH12_GPIO_1: now reaches U6.40 (GPIO_1)
- net ETH12_GPIO_1: now also U2.U12 (IO_L17P_T2_33)
- net ETH12_LED2_1V8: now reaches U6.45 (LED_2)
- net ETH12_LED2_1V8: now also U2.Y6 (IO_L7N_T1_33)
- net ETH12_LED1_1V8: now reaches U6.46 (LED_1)
- net ETH12_LED1_1V8: now also U2.R7 (IO_L8P_T1_33)
- net ETH12_LED0_1V8: now reaches U6.47 (LED_0)
- net ETH12_LED0_1V8: now also U2.R6 (IO_L8N_T1_33)
- net ETH13_GPIO_0: now reaches U5.39 (GPIO_0)
- net ETH13_GPIO_0: now also U2.T9 (IO_L18P_T2_33)
- net ETH13_GPIO_1: now reaches U5.40 (GPIO_1)
- net ETH13_GPIO_1: now also U2.U11 (IO_L17N_T2_33)
- net ETH13_LED2_1V8: now reaches U5.45 (LED_2)
- net ETH13_LED2_1V8: now also U2.W11 (IO_L6P_T0_33)
- net ETH13_LED1_1V8: now reaches U5.46 (LED_1)
- net ETH13_LED1_1V8: now also U2.Y11 (IO_L6N_T0_VREF_33)
- net ETH13_LED0_1V8: now reaches U5.47 (LED_0)
- net ETH13_LED0_1V8: now also U2.W6 (IO_L7P_T1_33)
- net VSC_MDC_1V8: now reaches U2.T11 (IO_L16P_T2_33)
- net VSC_FAST_STATUS_1V8: now reaches U2.U10 (IO_L14P_T2_SRCC_33)
- net VSC_MDIO_1V8: now reaches U2.V10 (IO_L15P_T2_DQS_33)
- net VSC_MDINT_1V8: now reaches U2.V9 (IO_L14N_T2_SRCC_33)
- net VSC_MDIO_OE: now reaches U2.W10 (IO_L15N_T2_DQS_33)
- net ETH12_A_TAP: now reaches J22.14 (BI_DA_TAP)
- net ETH12_A_TAP: now also C450.1
- net ETH12_C_TAP: now reaches J22.17 (BI_DC_TAP)
- net ETH12_C_TAP: now also C452.1
- net ETH12_B_TAP: now reaches J22.22 (BI_DB_TAP)
- net ETH12_B_TAP: now also C451.1
- net ETH12_D_TAP: now reaches J22.25 (BI_DD_TAP)
- net ETH12_D_TAP: now also C453.1
- net at J22.28 (LED1_P): now also R149.2
- net at J22.30 (LED2_G_P): now also R150.2
- new net: D6.2 (A), R153.2
- new net: D7.2 (A), R154.2
- new net ETH12_LED0_3V3: R149.1
- new net ETH12_LED1_3V3: R150.1
- new net ETH12_LED2_3V3: R153.1
- new net ETH12_LED_0_1V8: R139.1, R140.1
- new net ETH13_LED0_3V3: R151.1
- new net ETH13_LED1_3V3: R152.1
- new net ETH13_LED2_3V3: R154.1
- new net ETH13_LED_0_1V8: R143.1, R144.1
- no-connect marks 12 -> 35
Other:
- note added: "Common strap configuration: * RX_D2 open: PHY_ADD[3:2] = 2'b00 * RX_CTRL: autonegotiation enabled * GPIO_0 open: RGMII clock skew RX[0] = 0 * GPIO_1 open: RGMII clock skew RX[2:1] = 0 * LED_2 open: RGMII clock skew TX[1:0] = 0 * LED_1 open: ANEG_SEL=0, RGMII clock skew TX[2] = 0 * LED_0: mirror disable, SGMII enable"
- note added: "RX_D0 mode 2: PHY_ADD[1:0] = 2'b01"
- note added: "RX_D0 open: PHY_ADD[1:0] = 2'b00"
- note removed: "TODO: PHYADDR straps"
