File: latentpink/pcb/sgmii.kicad_sch (KiCad schematic)
At the start: 97 parts, among them J22 BEL_FUSE_0845-2R1T-E4, U2 XC7K160T-2FBG484C, U5 DP83867, U6 DP83867, U7 ECS-1612MV-250-CN-TR, U8 ECS-1612MV-250-CN-TR

Commit message: Lots more layout of low speed stuff and power. Partial layout of 1.2V supply. Initial RGMII escape routing.
Connections:
- net ETH12_LED0_1V8: now also U2.AB13 (IO_L22P_T3_33); no longer U2.R6 (IO_L8N_T1_33)
- net ETH12_LED1_1V8: now also U2.AB11 (IO_L20N_T3_33); no longer U2.R7 (IO_L8P_T1_33)
- net ETH12_SGMII_RX_AC_N: now also U2.V10 (IO_L15P_T2_DQS_33); no longer U2.U6 (IO_L10N_T1_33)
- net ETH12_SGMII_RX_AC_P: now also U2.V9 (IO_L14N_T2_SRCC_33); no longer U2.U7 (IO_L10P_T1_33)
- net VSC_FAST_STATUS_1V8: now also U2.R7 (IO_L8P_T1_33); no longer U2.U10 (IO_L14P_T2_SRCC_33)
- net VSC_MDC_1V8: now also U2.U6 (IO_L10N_T1_33); no longer U2.T11 (IO_L16P_T2_33)
- net VSC_MDINT_1V8: now also U2.R6 (IO_L8N_T1_33); no longer U2.V9 (IO_L14N_T2_SRCC_33)
- net VSC_MDIO_1V8: now also U2.U10 (IO_L14P_T2_SRCC_33); no longer U2.V10 (IO_L15P_T2_DQS_33)
Changed lines of the file:
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@@
   (paper "A3")
   (title_block
-    (date "2023-05-31")
+    (date "2023-06-01")
     (rev "0.1")
     (company "Antikernel Labs")
@@
   (no_connect (at 44.45 123.19))
   (no_connect (at 158.75 181.61))
-  (no_connect (at 44.45 128.27))
   (no_connect (at 158.75 191.77))
   (no_connect (at 158.75 176.53))
+  (no_connect (at 44.45 105.41))
   (no_connect (at 203.2 176.53))
   (no_connect (at 44.45 120.65))
   (no_connect (at 44.45 138.43))
-  (no_connect (at 44.45 135.89))
   (no_connect (at 158.75 62.23))
   (no_connect (at 158.75 179.07))
@@
   (no_connect (at 44.45 133.35))
   (no_connect (at 44.45 118.11))
+  (no_connect (at 44.45 74.93))
   (no_connect (at 203.2 59.69))
   (no_connect (at 203.2 62.23))
@@
     (effects (font (size 1.27 1.27)) (justify right bottom))
   )
-  (label "ETH12_LED1_1V8" (at 44.45 64.77 180)
+  (label "ETH12_LED1_1V8" (at 44.45 128.27 180)
     (effects (font (size 1.27 1.27)) (justify right bottom))
   )
@@
     (effects (font (size 1.27 1.27)) (justify right bottom))
   )
-  (label "ETH12_SGMII_RX_AC_N" (at 44.45 77.47 180)
+  (label "ETH12_SGMII_RX_AC_N" (at 44.45 100.33 180)
     (effects (font (size 1.27 1.27)) (justify right bottom))
   )
@@
     (effects (font (size 1.27 1.27)) (justify right bottom))
   )
-  (label "ETH12_LED0_1V8" (at 44.45 67.31 180)
+  (label "ETH12_LED0_1V8" (at 44.45 135.89 180)
     (effects (font (size 1.27 1.27)) (justify right bottom))
   )
@@
     (effects (font (size 1.27 1.27)) (justify right bottom))
   )
-  (label "ETH12_SGMII_RX_AC_P" (at 44.45 74.93 180)
+  (label "ETH12_SGMII_RX_AC_P" (at 44.45 97.79 180)
     (effects (font (size 1.27 1.27)) (justify right bottom))
   )
@@
     (effects (font (size 1.27 1.27)) (justify right bottom))
   )
-  (hierarchical_label "VSC_MDC_1V8" (shape output) (at 44.45 105.41 180)
+  (hierarchical_label "VSC_MDC_1V8" (shape output) (at 44.45 77.47 180)
     (effects (font (size 1.27 1.27)) (justify right))
   )
@@
     (effects (font (size 1.27 1.27)) (justify right))
   )
-  (hierarchical_label "VSC_FAST_STATUS_1V8" (shape input) (at 44.45 95.25 180)
+  (hierarchical_label "VSC_FAST_STATUS_1V8" (shape input) (at 44.45 64.77 180)
     (effects (font (size 1.27 1.27)) (justify right))
   )
@@
     (effects (font (size 1.27 1.27)) (justify right))
   )
-  (hierarchical_label "VSC_MDINT_1V8" (shape input) (at 44.45 97.79 180)
+  (hierarchical_label "VSC_MDINT_1V8" (shape input) (at 44.45 67.31 180)
     (effects (font (size 1.27 1.27)) (justify right))
   )
@@
     (effects (font (size 1.27 1.27)) (justify right))
   )
-  (hierarchical_label "VSC_MDIO_1V8" (shape bidirectional) (at 44.45 100.33 180)
+  (hierarchical_label "VSC_MDIO_1V8" (shape bidirectional) (at 44.45 95.25 180)
     (effects (font (size 1.27 1.27)) (justify right))
   )

Commit message: Routing of northwest corner
Connections:
- net ETH12_GPIO_0: now also U2.AA13 (IO_L21N_T3_DQS_33); no longer U2.T10 (IO_L16N_T2_33)
- net ETH12_GPIO_1: now also U2.AB12 (IO_L22N_T3_33); no longer U2.U12 (IO_L17P_T2_33)
- net ETH12_LED0_1V8: now also U2.Y12 (IO_L19N_T3_VREF_33); no longer U2.AB13 (IO_L22P_T3_33)
- net ETH12_LED2_1V8: now also U2.AB5 (IO_L1N_T0_33); no longer U2.Y6 (IO_L7N_T1_33)
- net ETH12_SGMII_TX_AC_N: now also U2.Y6 (IO_L7N_T1_33); no longer U2.W7 (IO_L11N_T1_SRCC_33)
- net ETH12_SGMII_TX_AC_P: now also U2.W6 (IO_L7P_T1_33); no longer U2.V7 (IO_L11P_T1_SRCC_33)
- net ETH13_GPIO_0: now also U2.AA11 (IO_L20P_T3_33); no longer U2.T9 (IO_L18P_T2_33)
- net ETH13_GPIO_1: now also U2.AB13 (IO_L22P_T3_33); no longer U2.U11 (IO_L17N_T2_33)
- net ETH13_LED0_1V8: now also U2.W7 (IO_L11N_T1_SRCC_33); no longer U2.W6 (IO_L7P_T1_33)
- net ETH13_LED1_1V8: now also U2.AA8 (IO_L5N_T0_33); no longer U2.Y11 (IO_L6N_T0_VREF_33)
- net ETH13_LED2_1V8: now also U2.AA9 (IO_L5P_T0_33); no longer U2.W11 (IO_L6P_T0_33)
- net ETH13_RST_N: now also U2.AA10 (IO_L4P_T0_33); no longer U2.AB5 (IO_L1N_T0_33)
- net ETH13_SGMII_RX_AC_N: now also U2.Y11 (IO_L6N_T0_VREF_33); no longer U2.AA8 (IO_L5N_T0_33)
- net ETH13_SGMII_RX_AC_P: now also U2.W11 (IO_L6P_T0_33); no longer U2.AA9 (IO_L5P_T0_33)
- net ETH13_SGMII_TX_AC_N: now also U2.V8 (IO_L9N_T1_DQS_33); no longer U2.AB10 (IO_L4N_T0_33)
- net ETH13_SGMII_TX_AC_P: now also U2.U8 (IO_L9P_T1_DQS_33); no longer U2.AA10 (IO_L4P_T0_33)
- net VSC_MDC_1V8: now also U2.T8 (IO_L18N_T2_33); no longer U2.U6 (IO_L10N_T1_33)
- net VSC_MDIO_1V8: now also U2.U7 (IO_L10P_T1_33); no longer U2.U10 (IO_L14P_T2_SRCC_33)
- net VSC_MDIO_OE: now also U2.U6 (IO_L10N_T1_33); no longer U2.W10 (IO_L15N_T2_DQS_33)
Changed lines of the file:
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@@
   (junction (at 340.36 46.99) (diameter 0) (color 0 0 0 0)
   )
+  (no_connect (at 44.45 110.49))
   (no_connect (at 203.2 57.15))
   (no_connect (at 158.75 173.99))
   (no_connect (at 44.45 143.51))
   (no_connect (at 158.75 67.31))
+  (no_connect (at 44.45 95.25))
   (no_connect (at 158.75 59.69))
   (no_connect (at 203.2 171.45))
-  (no_connect (at 44.45 125.73))
+  (no_connect (at 44.45 115.57))
   (no_connect (at 44.45 146.05))
-  (no_connect (at 44.45 69.85))
+  (no_connect (at 44.45 102.87))
   (no_connect (at 203.2 179.07))
   (no_connect (at 158.75 64.77))
   (no_connect (at 203.2 173.99))
   (no_connect (at 203.2 64.77))
-  (no_connect (at 44.45 123.19))
   (no_connect (at 158.75 181.61))
   (no_connect (at 158.75 191.77))
+  (no_connect (at 44.45 80.01))
   (no_connect (at 158.75 176.53))
   (no_connect (at 44.45 105.41))
+  (no_connect (at 44.45 130.81))
   (no_connect (at 203.2 176.53))
   (no_connect (at 44.45 120.65))
-  (no_connect (at 44.45 138.43))
+  (no_connect (at 44.45 107.95))
   (no_connect (at 158.75 62.23))
   (no_connect (at 158.75 179.07))
-  (no_connect (at 44.45 130.81))
+  (no_connect (at 44.45 46.99))
+  (no_connect (at 44.45 113.03))
   (no_connect (at 44.45 148.59))
   (no_connect (at 158.75 232.41))
@@
   (no_connect (at 158.75 77.47))
   (no_connect (at 44.45 140.97))
-  (no_connect (at 44.45 133.35))
-  (no_connect (at 44.45 118.11))
-  (no_connect (at 44.45 74.93))
   (no_connect (at 203.2 59.69))
   (no_connect (at 203.2 62.23))
-  (no_connect (at 44.45 72.39))
   (wire (pts (xy 142.24 120.65) (xy 158.75 120.65))
     (stroke (width 0) (type default) (color 0 0 0 0))
@@
     (effects (font (size 1.27 1.27)) (justify left bottom))
   )
-  (label "ETH13_LED1_1V8" (at 44.45 57.15 180)
+  (label "ETH13_LED1_1V8" (at 44.45 52.07 180)
     (effects (font (size 1.27 1.27)) (justify right bottom))
   )
@@
     (effects (font (size 1.27 1.27)) (justify right bottom))
   )
-  (label "ETH13_LED2_1V8" (at 44.45 54.61 180)
+  (label "ETH13_LED2_1V8" (at 44.45 49.53 180)
     (effects (font (size 1.27 1.27)) (justify right bottom))
   )
@@
     (effects (font (size 1.27 1.27)) (justify right bottom))
   )
-  (label "ETH13_SGMII_TX_AC_P" (at 44.45 44.45 180)
+  (label "ETH13_SGMII_TX_AC_P" (at 44.45 69.85 180)
     (effects (font (size 1.27 1.27)) (justify right bottom))
   )
@@
     (effects (font (size 1.27 1.27)) (justify right bottom))
   )
-  (label "ETH13_GPIO_0" (at 44.45 115.57 180)
+  (label "ETH13_GPIO_0" (at 44.45 125.73 180)
     (effects (font (size 1.27 1.27)) (justify right bottom))
   )
@@
     (effects (font (size 1.27 1.27)) (justify right bottom))
   )
-  (label "ETH13_SGMII_RX_AC_P" (at 44.45 49.53 180)
+  (label "ETH13_SGMII_RX_AC_P" (at 44.45 54.61 180)
     (effects (font (size 1.27 1.27)) (justify right bottom))
   )
@@
     (effects (font (size 1.27 1.27)) (justify right bottom))
   )
-  (label "ETH13_RST_N" (at 44.45 31.75 180)
+  (label "ETH13_RST_N" (at 44.45 44.45 180)
     (effects (font (size 1.27 1.27)) (justify right bottom))
   )
@@
     (effects (font (size 1.27 1.27)) (justify left bottom))
   )
-  (label "ETH13_GPIO_1" (at 44.45 113.03 180)
+  (label "ETH13_GPIO_1" (at 44.45 135.89 180)
     (effects (font (size 1.27 1.27)) (justify right bottom))
   )
@@
     (effects (font (size 1.27 1.27)) (justify right bottom))
   )
-  (label "ETH12_SGMII_TX_AC_P" (at 44.45 80.01 180)
+  (label "ETH12_SGMII_TX_AC_P" (at 44.45 59.69 180)
     (effects (font (size 1.27 1.27)) (justify right bottom))
   )
@@
     (effects (font (size 1.27 1.27)) (justify right bottom))
   )
-  (label "ETH13_SGMII_RX_AC_N" (at 44.45 52.07 180)
+  (label "ETH13_SGMII_RX_AC_N" (at 44.45 57.15 180)
     (effects (font (size 1.27 1.27)) (justify right bottom))
   )
@@
     (effects (font (size 1.27 1.27)) (justify right bottom))
   )
-  (label "ETH12_GPIO_0" (at 44.45 107.95 180)
+  (label "ETH12_GPIO_0" (at 44.45 133.35 180)
     (effects (font (size 1.27 1.27)) (justify right bottom))
   )
@@
     (effects (font (size 1.27 1.27)) (justify right bottom))
   )
-  (label "ETH13_SGMII_TX_AC_N" (at 44.45 46.99 180)
+  (label "ETH13_SGMII_TX_AC_N" (at 44.45 72.39 180)
     (effects (font (size 1.27 1.27)) (justify right bottom))
   )
@@
     (effects (font (size 1.27 1.27)) (justify right bottom))
   )
-  (label "ETH12_LED0_1V8" (at 44.45 135.89 180)
+  (label "ETH12_LED0_1V8" (at 44.45 123.19 180)
     (effects (font (size 1.27 1.27)) (justify right bottom))
   )
@@
     (effects (font (size 1.27 1.27)) (justify right bottom))
   )
-  (label "ETH12_LED2_1V8" (at 44.45 62.23 180)
+  (label "ETH12_LED2_1V8" (at 44.45 31.75 180)
     (effects (font (size 1.27 1.27)) (justify right bottom))
   )
@@
     (effects (font (size 1.27 1.27)) (justify left bottom))
   )
-  (label "ETH12_SGMII_TX_AC_N" (at 44.45 82.55 180)
-    (effects (font (size 1.27 1.27)) (justify right bottom))
-  )
-  (label "ETH13_LED0_1V8" (at 44.45 59.69 180)
+  (label "ETH12_SGMII_TX_AC_N" (at 44.45 62.23 180)
+    (effects (font (size 1.27 1.27)) (justify right bottom))
+  )
+  (label "ETH13_LED0_1V8" (at 44.45 82.55 180)
     (effects (font (size 1.27 1.27)) (justify right bottom))
   )
@@
     (effects (font (size 1.27 1.27)) (justify right bottom))
   )
-  (label "ETH12_GPIO_1" (at 44.45 110.49 180)
+  (label "ETH12_GPIO_1" (at 44.45 138.43 180)
     (effects (font (size 1.27 1.27)) (justify right bottom))
   )
@@
     (effects (font (size 1.27 1.27)) (justify right bottom))
   )
-  (hierarchical_label "VSC_MDC_1V8" (shape output) (at 44.45 77.47 180)
+  (hierarchical_label "VSC_MDC_1V8" (shape output) (at 44.45 118.11 180)
     (effects (font (size 1.27 1.27)) (justify right))
   )
@@
     (effects (font (size 1.27 1.27)) (justify right))
   )
-  (hierarchical_label "VSC_MDIO_1V8" (shape bidirectional) (at 44.45 95.25 180)
+  (hierarchical_label "VSC_MDIO_1V8" (shape bidirectional) (at 44.45 74.93 180)
     (effects (font (size 1.27 1.27)) (justify right))
   )
@@
     (effects (font (size 1.27 1.27)) (justify right))
   )
-  (hierarchical_label "VSC_MDIO_OE" (shape output) (at 44.45 102.87 180)
-    (effects (font (size 1.27 1.27)) (justify right))
-  )
+  (hierarchical_label "VSC_MDIO_OE" (shape output) (at 44.45 77.47 180)
+    (effects (font (size 1.27 1.27)) (justify right))
+  )

Commit message: Continued routing of power and top parts
Connections:
- net ETH12_SGMII_CLKOUT_AC_N: now also U2.Y9 (IO_L13N_T2_MRCC_33); no longer U2.Y7 (IO_L12N_T1_MRCC_33)
- net ETH12_SGMII_CLKOUT_AC_P: now also U2.W9 (IO_L13P_T2_MRCC_33); no longer U2.Y8 (IO_L12P_T1_MRCC_33)
- net ETH12_SGMII_RX_AC_N: now also U2.V9 (IO_L14N_T2_SRCC_33); no longer U2.V10 (IO_L15P_T2_DQS_33)
- net ETH12_SGMII_RX_AC_P: now also U2.U10 (IO_L14P_T2_SRCC_33); no longer U2.V9 (IO_L14N_T2_SRCC_33)
- net ETH12_SGMII_TX_AC_N: now also U2.Y11 (IO_L6N_T0_VREF_33); no longer U2.Y6 (IO_L7N_T1_33)
- net ETH12_SGMII_TX_AC_P: now also U2.W11 (IO_L6P_T0_33); no longer U2.W6 (IO_L7P_T1_33)
- net ETH13_SGMII_CLKOUT_AC_N: now also U2.Y8 (IO_L12P_T1_MRCC_33); no longer U2.Y9 (IO_L13N_T2_MRCC_33)
- net ETH13_SGMII_CLKOUT_AC_P: now also U2.Y7 (IO_L12N_T1_MRCC_33); no longer U2.W9 (IO_L13P_T2_MRCC_33)
- net ETH13_SGMII_RX_AC_N: now also U2.U8 (IO_L9P_T1_DQS_33); no longer U2.Y11 (IO_L6N_T0_VREF_33)
- net ETH13_SGMII_RX_AC_P: now also U2.V8 (IO_L9N_T1_DQS_33); no longer U2.W11 (IO_L6P_T0_33)
- net ETH13_SGMII_TX_AC_N: now also U2.W6 (IO_L7P_T1_33); no longer U2.V8 (IO_L9N_T1_DQS_33)
- net ETH13_SGMII_TX_AC_P: now also U2.Y6 (IO_L7N_T1_33); no longer U2.U8 (IO_L9P_T1_DQS_33)
Other:
- note added: "Polarity swap"
Changed lines of the file:
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@@
   (no_connect (at 44.45 143.51))
   (no_connect (at 158.75 67.31))
-  (no_connect (at 44.45 95.25))
   (no_connect (at 158.75 59.69))
   (no_connect (at 203.2 171.45))
@@
   (no_connect (at 203.2 173.99))
   (no_connect (at 203.2 64.77))
+  (no_connect (at 44.45 100.33))
   (no_connect (at 158.75 181.61))
   (no_connect (at 158.75 191.77))
@@
     (stroke (width 0) (type default) (color 0 0 0 0))
   )
+  (text "Polarity swap" (at 87.63 62.23 0)
+    (effects (font (size 1.27 1.27)) (justify left bottom))
+  )
+  (text "Polarity swap" (at 87.63 85.09 0)
+    (effects (font (size 1.27 1.27)) (justify left bottom))
+  )
   (text "RX_D0 open: PHY_ADD[1:0] = 2'b00" (at 161.29 124.46 0)
     (effects (font (size 1.27 1.27)) (justify left bottom))
@@
     (effects (font (size 1.27 1.27)) (justify left bottom))
   )
+  (text "Polarity swap" (at 87.63 72.39 0)
+    (effects (font (size 1.27 1.27)) (justify left bottom))
+  )
   (text "UG471 figure 1-10\nExt ref resistor = 2x Z0" (at 49.53 25.4 0)
     (effects (font (size 1.27 1.27)) (justify left bottom))
@@
     (effects (font (size 1.27 1.27)) (justify right bottom))
   )
-  (label "ETH13_SGMII_TX_AC_P" (at 44.45 69.85 180)
+  (label "ETH13_SGMII_TX_AC_P" (at 44.45 62.23 180)
     (effects (font (size 1.27 1.27)) (justify right bottom))
   )
@@
     (effects (font (size 1.27 1.27)) (justify left bottom))
   )
-  (label "ETH13_SGMII_CLKOUT_AC_P" (at 44.45 90.17 180)
+  (label "ETH13_SGMII_CLKOUT_AC_P" (at 44.45 87.63 180)
     (effects (font (size 1.27 1.27)) (justify right bottom))
   )
@@
     (effects (font (size 1.27 1.27)) (justify right bottom))
   )
-  (label "ETH13_SGMII_RX_AC_P" (at 44.45 54.61 180)
+  (label "ETH13_SGMII_RX_AC_P" (at 44.45 72.39 180)
     (effects (font (size 1.27 1.27)) (justify right bottom))
   )
@@
     (effects (font (size 1.27 1.27)) (justify right bottom))
   )
-  (label "ETH12_SGMII_TX_AC_P" (at 44.45 59.69 180)
+  (label "ETH12_SGMII_TX_AC_P" (at 44.45 54.61 180)
     (effects (font (size 1.27 1.27)) (justify right bottom))
   )
@@
     (effects (font (size 1.27 1.27)) (justify right bottom))
   )
-  (label "ETH13_SGMII_RX_AC_N" (at 44.45 57.15 180)
+  (label "ETH13_SGMII_RX_AC_N" (at 44.45 69.85 180)
     (effects (font (size 1.27 1.27)) (justify right bottom))
   )
@@
     (effects (font (size 1.27 1.27)) (justify right bottom))
   )
-  (label "ETH12_SGMII_RX_AC_N" (at 44.45 100.33 180)
+  (label "ETH12_SGMII_RX_AC_N" (at 44.45 97.79 180)
     (effects (font (size 1.27 1.27)) (justify right bottom))
   )
@@
     (effects (font (size 1.27 1.27)) (justify right bottom))
   )
-  (label "ETH13_SGMII_CLKOUT_AC_N" (at 44.45 92.71 180)
+  (label "ETH13_SGMII_CLKOUT_AC_N" (at 44.45 85.09 180)
     (effects (font (size 1.27 1.27)) (justify right bottom))
   )
@@
     (effects (font (size 1.27 1.27)) (justify right bottom))
   )
-  (label "ETH13_SGMII_TX_AC_N" (at 44.45 72.39 180)
+  (label "ETH13_SGMII_TX_AC_N" (at 44.45 59.69 180)
     (effects (font (size 1.27 1.27)) (justify right bottom))
   )
@@
     (effects (font (size 1.27 1.27)) (justify left bottom))
   )
-  (label "ETH12_SGMII_CLKOUT_AC_P" (at 44.45 85.09 180)
+  (label "ETH12_SGMII_CLKOUT_AC_P" (at 44.45 90.17 180)
     (effects (font (size 1.27 1.27)) (justify right bottom))
   )
@@
     (effects (font (size 1.27 1.27)) (justify right bottom))
   )
-  (label "ETH12_SGMII_RX_AC_P" (at 44.45 97.79 180)
+  (label "ETH12_SGMII_RX_AC_P" (at 44.45 95.25 180)
     (effects (font (size 1.27 1.27)) (justify right bottom))
   )
@@
     (effects (font (size 1.27 1.27)) (justify left bottom))
   )
-  (label "ETH12_SGMII_TX_AC_N" (at 44.45 62.23 180)
+  (label "ETH12_SGMII_TX_AC_N" (at 44.45 57.15 180)
     (effects (font (size 1.27 1.27)) (justify right bottom))
   )
@@
     (effects (font (size 1.27 1.27)) (justify left bottom))
   )
-  (label "ETH12_SGMII_CLKOUT_AC_N" (at 44.45 87.63 180)
-    (effects (font (size 1.27 1.27)) (justify right bottom))
-  )
+  (label "ETH12_SGMII_CLKOUT_AC_N" (at 44.45 92.71 180)
+    (effects (font (size 1.27 1.27)) (justify right bottom))
+  )

Commit message: Continued initial QDR routing
Connections:
- net DP_MDC: now also U2.AB12 (IO_L22N_T3_33); no longer U2.AA6 (IO_L3P_T0_DQS_33)
- net DP_MDIO: now also U2.Y12 (IO_L19N_T3_VREF_33); no longer U2.AB6 (IO_L3N_T0_DQS_33)
- net ETH12_GPIO_0: now also U2.AB8 (IO_L2P_T0_33); no longer U2.AA13 (IO_L21N_T3_DQS_33)
- net ETH12_GPIO_1: now also U2.AA8 (IO_L5N_T0_33); no longer U2.AB12 (IO_L22N_T3_33)
- net ETH12_INT_N: now also U2.AA6 (IO_L3P_T0_DQS_33); no longer U2.AB8 (IO_L2P_T0_33)
- net ETH12_LED0_1V8: now also U2.AB5 (IO_L1N_T0_33); no longer U2.Y12 (IO_L19N_T3_VREF_33)
- net ETH12_LED1_1V8: now also U2.W7 (IO_L11N_T1_SRCC_33); no longer U2.AB11 (IO_L20N_T3_33)
- net ETH12_LED2_1V8: now also U2.AB6 (IO_L3N_T0_DQS_33); no longer U2.AB5 (IO_L1N_T0_33)
- net ETH13_GPIO_0: now also U2.AB13 (IO_L22P_T3_33); no longer U2.AA11 (IO_L20P_T3_33)
- net ETH13_GPIO_1: now also U2.AA13 (IO_L21N_T3_DQS_33); no longer U2.AB13 (IO_L22P_T3_33)
- net ETH13_INT_N: now also U2.AB10 (IO_L4N_T0_33); no longer U2.AA5 (IO_L1P_T0_33)
- net ETH13_LED0_1V8: now also U2.AA9 (IO_L5P_T0_33); no longer U2.W7 (IO_L11N_T1_SRCC_33)
- net ETH13_LED1_1V8: now also U2.AA10 (IO_L4P_T0_33); no longer U2.AA8 (IO_L5N_T0_33)
- net ETH13_LED2_1V8: now also U2.AA11 (IO_L20P_T3_33); no longer U2.AA9 (IO_L5P_T0_33)
- net ETH13_RST_N: now also U2.AB11 (IO_L20N_T3_33); no longer U2.AA10 (IO_L4P_T0_33)
Changed lines of the file:
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@@
   (paper "A3")
   (title_block
-    (date "2023-06-01")
+    (date "2023-06-03")
     (rev "0.1")
     (company "Antikernel Labs")
@@
   (no_connect (at 44.45 107.95))
   (no_connect (at 158.75 62.23))
+  (no_connect (at 44.45 29.21))
   (no_connect (at 158.75 179.07))
-  (no_connect (at 44.45 46.99))
   (no_connect (at 44.45 113.03))
   (no_connect (at 44.45 148.59))
@@
     (effects (font (size 1.27 1.27)) (justify left bottom))
   )
-  (label "ETH13_LED1_1V8" (at 44.45 52.07 180)
+  (label "ETH13_LED1_1V8" (at 44.45 44.45 180)
     (effects (font (size 1.27 1.27)) (justify right bottom))
   )
@@
     (effects (font (size 1.27 1.27)) (justify right bottom))
   )
-  (label "ETH13_LED2_1V8" (at 44.45 49.53 180)
+  (label "ETH13_LED2_1V8" (at 44.45 125.73 180)
     (effects (font (size 1.27 1.27)) (justify right bottom))
   )
@@
     (effects (font (size 1.27 1.27)) (justify right bottom))
   )
-  (label "ETH13_GPIO_0" (at 44.45 125.73 180)
+  (label "ETH13_GPIO_0" (at 44.45 135.89 180)
     (effects (font (size 1.27 1.27)) (justify right bottom))
   )
@@
     (effects (font (size 1.27 1.27)) (justify right bottom))
   )
-  (label "DP_MDIO" (at 44.45 41.91 180)
+  (label "DP_MDIO" (at 44.45 123.19 180)
     (effects (font (size 1.27 1.27)) (justify right bottom))
   )
@@
     (effects (font (size 1.27 1.27)) (justify right bottom))
   )
-  (label "ETH12_LED1_1V8" (at 44.45 128.27 180)
+  (label "ETH12_LED1_1V8" (at 44.45 82.55 180)
     (effects (font (size 1.27 1.27)) (justify right bottom))
   )
@@
     (effects (font (size 1.27 1.27)) (justify right bottom))
   )
-  (label "ETH13_RST_N" (at 44.45 44.45 180)
+  (label "ETH13_RST_N" (at 44.45 128.27 180)
     (effects (font (size 1.27 1.27)) (justify right bottom))
   )
@@
     (effects (font (size 1.27 1.27)) (justify left bottom))
   )
-  (label "ETH13_GPIO_1" (at 44.45 135.89 180)
+  (label "ETH13_GPIO_1" (at 44.45 133.35 180)
     (effects (font (size 1.27 1.27)) (justify right bottom))
   )
@@
     (effects (font (size 1.27 1.27)) (justify right bottom))
   )
-  (label "DP_MDC" (at 44.45 39.37 180)
+  (label "DP_MDC" (at 44.45 138.43 180)
     (effects (font (size 1.27 1.27)) (justify right bottom))
   )
@@
     (effects (font (size 1.27 1.27)) (justify left bottom))
   )
-  (label "ETH13_INT_N" (at 44.45 29.21 180)
+  (label "ETH13_INT_N" (at 44.45 46.99 180)
     (effects (font (size 1.27 1.27)) (justify right bottom))
   )
@@
     (effects (font (size 1.27 1.27)) (justify right bottom))
   )
-  (label "ETH12_GPIO_0" (at 44.45 133.35 180)
+  (label "ETH12_GPIO_0" (at 44.45 34.29 180)
     (effects (font (size 1.27 1.27)) (justify right bottom))
   )
@@
     (effects (font (size 1.27 1.27)) (justify right bottom))
   )
-  (label "ETH12_LED0_1V8" (at 44.45 123.19 180)
+  (label "ETH12_LED0_1V8" (at 44.45 31.75 180)
     (effects (font (size 1.27 1.27)) (justify right bottom))
   )
@@
     (effects (font (size 1.27 1.27)) (justify right bottom))
   )
-  (label "ETH12_LED2_1V8" (at 44.45 31.75 180)
+  (label "ETH12_LED2_1V8" (at 44.45 41.91 180)
     (effects (font (size 1.27 1.27)) (justify right bottom))
   )
@@
     (effects (font (size 1.27 1.27)) (justify left bottom))
   )
-  (label "ETH12_INT_N" (at 44.45 34.29 180)
+  (label "ETH12_INT_N" (at 44.45 39.37 180)
     (effects (font (size 1.27 1.27)) (justify right bottom))
   )
@@
     (effects (font (size 1.27 1.27)) (justify right bottom))
   )
-  (label "ETH13_LED0_1V8" (at 44.45 82.55 180)
+  (label "ETH13_LED0_1V8" (at 44.45 49.53 180)
     (effects (font (size 1.27 1.27)) (justify right bottom))
   )
@@
     (effects (font (size 1.27 1.27)) (justify right bottom))
   )
-  (label "ETH12_GPIO_1" (at 44.45 138.43 180)
-    (effects (font (size 1.27 1.27)) (justify right bottom))
-  )
+  (label "ETH12_GPIO_1" (at 44.45 52.07 180)
+    (effects (font (size 1.27 1.27)) (justify right bottom))
+  )
