File: latentpink/pcb/mgmt.kicad_sch (KiCad schematic)
At the start: 77 parts, among them J10 XILINX_JTAG, J11 FAN_01, J12 FAN_01, J15 CONN_01X03, J16 JUMPER_0402_SPDT, J17 JUMPER_0402_SPDT, J23 PMOD_HOST, J7 RJ45, U2 XC7K160T-2FBG484C, U20 AT24MAC402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

Commit message: Continued work on signoff review, added some more test points and SFP+ activity LEDs
Parts:
- added D16, D17: GREEN, azonenberg_pcb:EIA_0603_LED, symbol device:LED
- added R164, R165: 470, azonenberg_pcb:EIA_0402_RES_NOSILK, symbol device:R
- added TP28: U.FL, azonenberg_pcb:CONN_U.FL_TE_1909763-1, symbol conn:CONN_COAXIAL
Connections:
- net GND: now also TP28.2 (Ext)
- net MCU_VDDA: now also TP28.1 (In)
- net SFP_LED0: now reaches U2.E12 (IO_L10N_T1_16)
- net SFP_LED0: now also R164.1
- net SFP_LED1: now reaches U2.F11 (IO_L11P_T1_SRCC_16)
- net SFP_LED1: now also R165.1
- new net: D17.2 (A), R165.2
- new net: D16.1 (K), D17.1 (K)
- new net: D16.2 (A), R164.2
- no-connect marks 102 -> 100
Other:
- note added: "LEDs for SFP+ port TX/RX indicators Place near SFP (no light pipes on prototype)"
Changed lines of the file:
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@@
   (paper "A3")
   (title_block
-    (date "2023-05-20")
+    (date "2023-05-21")
     (rev "0.1")
     (company "Antikernel Labs")
@@
   (no_connect (at 165.1 109.22))
   (no_connect (at 214.63 109.22))
-  (no_connect (at 335.28 119.38))
   (no_connect (at 214.63 43.18))
   (no_connect (at 260.35 83.82))
@@
   (no_connect (at 214.63 86.36))
   (no_connect (at 303.53 48.26))
-  (no_connect (at 335.28 121.92))
   (no_connect (at 303.53 50.8))
   (no_connect (at 214.63 91.44))
@@
     (stroke (width 0) (type default) (color 0 0 0 0))
   )
+  (wire (pts (xy 200.66 273.05) (xy 193.04 273.05))
+    (stroke (width 0) (type default) (color 0 0 0 0))
+  )
   (wire (pts (xy 114.3 71.12) (xy 114.3 73.66))
     (stroke (width 0) (type default) (color 0 0 0 0))
@@
     (stroke (width 0) (type default) (color 0 0 0 0))
   )
+  (wire (pts (xy 200.66 264.16) (xy 200.66 273.05))
+    (stroke (width 0) (type default) (color 0 0 0 0))
+  )
   (wire (pts (xy 241.3 158.75) (xy 241.3 156.21))
     (stroke (width 0) (type default) (color 0 0 0 0))
@@
     (stroke (width 0) (type default) (color 0 0 0 0))
   )
+  (wire (pts (xy 193.04 264.16) (xy 200.66 264.16))
+    (stroke (width 0) (type default) (color 0 0 0 0))
+  )
   (wire (pts (xy 52.07 118.11) (xy 63.5 118.11))
     (stroke (width 0) (type default) (color 0 0 0 0))
@@
     (effects (font (size 1.27 1.27)) (justify left bottom))
   )
+  (text "LEDs for SFP+ port TX/RX indicators\nPlace near SFP (no light pipes on prototype)"
+    (at 177.8 278.13 0)
+    (effects (font (size 1.27 1.27)) (justify left bottom))
+  )
   (text "MCU VCAP decoupling" (at 35.56 167.64 0)
     (effects (font (size 1.27 1.27)) (justify left bottom))
@@
     (effects (font (size 1.27 1.27)) (justify left bottom))
   )
+  (label "MCU_VDDA" (at 74.93 77.47 180)
+    (effects (font (size 1.27 1.27)) (justify right bottom))
+  )
   (label "GND" (at 85.09 38.1 180)
     (effects (font (size 1.27 1.27)) (justify right bottom))
@@
     (effects (font (size 1.27 1.27)) (justify right bottom))
   )
+  (label "SFP_LED1" (at 335.28 121.92 180)
+    (effects (font (size 1.27 1.27)) (justify right bottom))
+  )
   (label "3V3" (at 224.79 133.35 0)
     (effects (font (size 1.27 1.27)) (justify left bottom))
@@
     (effects (font (size 1.27 1.27)) (justify right bottom))
   )
+  (label "SFP_LED0" (at 335.28 119.38 180)
+    (effects (font (size 1.27 1.27)) (justify right bottom))
+  )
   (label "FAN1_TACH" (at 27.94 260.35 180)
     (effects (font (size 1.27 1.27)) (justify right bottom))
@@
     (effects (font (size 1.27 1.27)) (justify right bottom))
   )
+  (label "SFP_LED0" (at 177.8 264.16 180)
+    (effects (font (size 1.27 1.27)) (justify right bottom))
+  )
   (label "MCU_QSPI_CS_N" (at 335.28 185.42 180)
     (effects (font (size 1.27 1.27)) (justify right bottom))
@@
     (effects (font (size 1.27 1.27)) (justify right bottom))
   )
+  (label "SFP_LED1" (at 177.8 273.05 180)
+    (effects (font (size 1.27 1.27)) (justify right bottom))
+  )
   (label "PMOD_DQ0" (at 363.22 44.45 180)
     (effects (font (size 1.27 1.27)) (justify right bottom))
@@
     (effects (font (size 1.27 1.27)) (justify right bottom))
   )
+  (label "GND" (at 78.74 82.55 0)
+    (effects (font (size 1.27 1.27)) (justify left bottom))
+  )
   (label "FPGA_LED0" (at 270.51 200.66 180)
     (effects (font (size 1.27 1.27)) (justify right bottom))
@@
     (pin "2")
   )
+  (symbol (lib_id "device:R") (at 181.61 273.05 90) (unit 1)
+    (in_bom yes) (on_board yes)
+    (property "Reference" "R165" (id 0) (at 181.61 270.51 90))
+    (property "Value" "470" (id 1) (at 181.61 273.05 90))
+    (property "Footprint" "azonenberg_pcb:EIA_0402_RES_NOSILK" (id 2) (at 181.61 274.828 90)
+      (effects (font (size 1.27 1.27)) hide)
+    )
+    (property "Datasheet" "" (id 3) (at 181.61 273.05 0)
+      (effects (font (size 1.27 1.27)) hide)
+    )
+    (pin "1")
+    (pin "2")
+  )
   (symbol (lib_id "device:C") (at 35.56 161.29 0) (unit 1)
     (in_bom yes) (on_board yes) (fields_autoplaced)
@@
     (pin "2")
   )
+  (symbol (lib_id "device:LED") (at 189.23 273.05 180) (unit 1)
+    (in_bom yes) (on_board yes) (fields_autoplaced)
+    (property "Reference" "D17" (id 0) (at 190.8302 267.1912 0))
+    (property "Value" "GREEN" (id 1) (at 190.8302 269.7281 0))
+    (property "Footprint" "azonenberg_pcb:EIA_0603_LED" (id 2) (at 189.23 273.05 0)
+      (effects (font (size 1.27 1.27)) hide)
+    )
+    (property "Datasheet" "" (id 3) (at 189.23 273.05 0)
+      (effects (font (size 1.27 1.27)) hide)
+    )
+    (pin "1")
+    (pin "2")
+  )
   (symbol (lib_id "special-azonenberg:JUMPER_0402_SPDT") (at 215.9 236.22 0) (mirror y) (unit 1)
     (in_bom yes) (on_board yes) (fields_autoplaced)
@@
     (pin "2")
   )
+  (symbol (lib_id "device:LED") (at 189.23 264.16 180) (unit 1)
+    (in_bom yes) (on_board yes) (fields_autoplaced)
+    (property "Reference" "D16" (id 0) (at 190.8302 258.3012 0))
+    (property "Value" "GREEN" (id 1) (at 190.8302 260.8381 0))
+    (property "Footprint" "azonenberg_pcb:EIA_0603_LED" (id 2) (at 189.23 264.16 0)
+      (effects (font (size 1.27 1.27)) hide)
+    )
+    (property "Datasheet" "" (id 3) (at 189.23 264.16 0)
+      (effects (font (size 1.27 1.27)) hide)
+    )
+    (pin "1")
+    (pin "2")
+  )
   (symbol (lib_id "conn:CONN_01X04") (at 33.02 259.08 0) (unit 1)
     (in_bom yes) (on_board yes) (fields_autoplaced)
@@
     (pin "8")
   )
+  (symbol (lib_id "device:R") (at 181.61 264.16 90) (unit 1)
+    (in_bom yes) (on_board yes)
+    (property "Reference" "R164" (id 0) (at 181.61 261.62 90))
+    (property "Value" "470" (id 1) (at 181.61 264.16 90))
+    (property "Footprint" "azonenberg_pcb:EIA_0402_RES_NOSILK" (id 2) (at 181.61 265.938 90)
+      (effects (font (size 1.27 1.27)) hide)
+    )
+    (property "Datasheet" "" (id 3) (at 181.61 264.16 0)
+      (effects (font (size 1.27 1.27)) hide)
+    )
+    (pin "1")
+    (pin "2")
+  )
   (symbol (lib_id "device:R") (at 274.32 200.66 90) (unit 1)
     (in_bom yes) (on_board yes)
@@
     (pin "9")
   )
+  (symbol (lib_id "conn:CONN_COAXIAL") (at 78.74 77.47 0) (unit 1)
+    (in_bom yes) (on_board yes) (fields_autoplaced)
+    (property "Reference" "TP28" (id 0) (at 81.2801 76.8547 0)
+      (effects (font (size 1.27 1.27)) (justify left))
+    )
+    (property "Value" "U.FL" (id 1) (at 81.2801 79.6298 0)
+      (effects (font (size 1.27 1.27)) (justify left))
+    )
+    (property "Footprint" "azonenberg_pcb:CONN_U.FL_TE_1909763-1" (id 2) (at 78.74 77.47 0)
+      (effects (font (size 1.27 1.27)) hide)
+    )
+    (property "Datasheet" "" (id 3) (at 78.74 77.47 0)
+      (effects (font (size 1.27 1.27)) hide)
+    )
+    (pin "1")
+    (pin "2")
+  )
   (sheet (at 314.96 201.93) (size 15.24 25.4) (fields_autoplaced)

Commit message: Finished initial schematic review, added ESD diodes to Ethernet pairs
Connections:
- net I2C_SCL: now also U4.A2 (PB8)
- net I2C_SDA: now also U4.B3 (PB9)
- no-connect marks 100 -> 98
Other:
- note added: "Address = 8'ha0, 8'hb0"
Changed lines of the file:
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@@
   (no_connect (at 214.63 96.52))
   (no_connect (at 214.63 55.88))
-  (no_connect (at 165.1 106.68))
   (no_connect (at 214.63 27.94))
   (no_connect (at 214.63 119.38))
@@
   (no_connect (at 303.53 33.02))
   (no_connect (at 165.1 53.34))
-  (no_connect (at 165.1 104.14))
   (no_connect (at 303.53 60.96))
   (no_connect (at 165.1 114.3))
@@
     (stroke (width 0) (type default) (color 0 0 0 0))
   )
+  (text "Address = 8'ha0, 8'hb0" (at 168.91 179.07 0)
+    (effects (font (size 1.27 1.27)) (justify left bottom))
+  )
   (text "MCU VDD decoupling" (at 35.56 100.33 0)
     (effects (font (size 1.27 1.27)) (justify left bottom))
@@
     (effects (font (size 1.27 1.27)) (justify right bottom))
   )
+  (label "I2C_SDA" (at 165.1 106.68 180)
+    (effects (font (size 1.27 1.27)) (justify right bottom))
+  )
   (label "GND" (at 165.1 135.89 180)
     (effects (font (size 1.27 1.27)) (justify right bottom))
@@
     (effects (font (size 1.27 1.27)) (justify right bottom))
   )
+  (label "I2C_SCL" (at 165.1 104.14 180)
+    (effects (font (size 1.27 1.27)) (justify right bottom))
+  )
   (label "3V3" (at 62.23 105.41 180)
     (effects (font (size 1.27 1.27)) (justify right bottom))
@@
     (pin "R3")
     (pin "R7")
-    (pin "A2")
+    (pin "A2" (alternate "I2C4_SCL"))
     (pin "A5" (alternate "I2C1_SCL"))
     (pin "A6" (alternate "JTDO"))
-    (pin "B3")
+    (pin "B3" (alternate "I2C4_SDA"))
     (pin "B5" (alternate "I2C1_SDA"))
     (pin "B6" (alternate "NJTRST"))
@@
     (pin "R3")
     (pin "R7")
-    (pin "A2")
+    (pin "A2" (alternate "I2C4_SCL"))
     (pin "A5" (alternate "I2C1_SCL"))
     (pin "A6" (alternate "JTDO"))
-    (pin "B3")
+    (pin "B3" (alternate "I2C4_SDA"))
     (pin "B5" (alternate "I2C1_SDA"))
     (pin "B6" (alternate "NJTRST"))
@@
     (pin "R3")
     (pin "R7")
-    (pin "A2")
+    (pin "A2" (alternate "I2C4_SCL"))
     (pin "A5" (alternate "I2C1_SCL"))
     (pin "A6" (alternate "JTDO"))
-    (pin "B3")
+    (pin "B3" (alternate "I2C4_SDA"))
     (pin "B5" (alternate "I2C1_SDA"))
     (pin "B6" (alternate "NJTRST"))
@@
     (pin "R3")
     (pin "R7")
-    (pin "A2")
+    (pin "A2" (alternate "I2C4_SCL"))
     (pin "A5" (alternate "I2C1_SCL"))
     (pin "A6" (alternate "JTDO"))
-    (pin "B3")
+    (pin "B3" (alternate "I2C4_SDA"))
     (pin "B5" (alternate "I2C1_SDA"))
     (pin "B6" (alternate "NJTRST"))
@@
     (pin "R3")
     (pin "R7")
-    (pin "A2")
+    (pin "A2" (alternate "I2C4_SCL"))
     (pin "A5" (alternate "I2C1_SCL"))
     (pin "A6" (alternate "JTDO"))
-    (pin "B3")
+    (pin "B3" (alternate "I2C4_SDA"))
     (pin "B5" (alternate "I2C1_SDA"))
     (pin "B6" (alternate "NJTRST"))
@@
     (pin "R3")
     (pin "R7")
-    (pin "A2")
+    (pin "A2" (alternate "I2C4_SCL"))
     (pin "A5" (alternate "I2C1_SCL"))
     (pin "A6" (alternate "JTDO"))
-    (pin "B3")
+    (pin "B3" (alternate "I2C4_SDA"))
     (pin "B5" (alternate "I2C1_SDA"))
     (pin "B6" (alternate "NJTRST"))
@@
     (pin "R3")
     (pin "R7")
-    (pin "A2")
+    (pin "A2" (alternate "I2C4_SCL"))
     (pin "A5" (alternate "I2C1_SCL"))
     (pin "A6" (alternate "JTDO"))
-    (pin "B3")
+    (pin "B3" (alternate "I2C4_SDA"))
     (pin "B5" (alternate "I2C1_SDA"))
     (pin "B6" (alternate "NJTRST"))
@@
     (pin "R3")
     (pin "R7")
-    (pin "A2")
+    (pin "A2" (alternate "I2C4_SCL"))
     (pin "A5" (alternate "I2C1_SCL"))
     (pin "A6" (alternate "JTDO"))
-    (pin "B3")
+    (pin "B3" (alternate "I2C4_SDA"))
     (pin "B5" (alternate "I2C1_SDA"))
     (pin "B6" (alternate "NJTRST"))
@@
     (pin "R3")
     (pin "R7")
-    (pin "A2")
+    (pin "A2" (alternate "I2C4_SCL"))
     (pin "A5" (alternate "I2C1_SCL"))
     (pin "A6" (alternate "JTDO"))
-    (pin "B3")
+    (pin "B3" (alternate "I2C4_SDA"))
     (pin "B5" (alternate "I2C1_SDA"))
     (pin "B6" (alternate "NJTRST"))
@@
     (pin "R3")
     (pin "R7")
-    (pin "A2")
+    (pin "A2" (alternate "I2C4_SCL"))
     (pin "A5" (alternate "I2C1_SCL"))
     (pin "A6" (alternate "JTDO"))
-    (pin "B3")
+    (pin "B3" (alternate "I2C4_SDA"))
     (pin "B5" (alternate "I2C1_SDA"))
     (pin "B6" (alternate "NJTRST"))

Commit message: Preliminary routing of first four baseT interfaces on VSC8512
Parts:
- U30: symbol osc-azonenberg:OSC_LVDS -> osc-azonenberg:OSC_LVDS_NOPAD
Connections:
- net GND: no longer U30.PAD (GND)
Changed lines of the file:
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@@
   (junction (at 31.75 66.04) (diameter 0) (color 0 0 0 0)
   )
-  (junction (at 241.3 158.75) (diameter 0) (color 0 0 0 0)
-  )
   (junction (at 139.7 55.88) (diameter 0) (color 0 0 0 0)
   )
@@
     (pin "2")
   )
-  (symbol (lib_id "osc-azonenberg:OSC_LVDS") (at 248.92 160.02 0) (unit 1)
+  (symbol (lib_id "osc-azonenberg:OSC_LVDS_NOPAD") (at 248.92 160.02 0) (unit 1)
     (in_bom yes) (on_board yes) (fields_autoplaced)
     (property "Reference" "U30" (id 0) (at 256.54 145.7759 0)
@@
     (pin "5")
     (pin "6")
-    (pin "PAD")
   )
   (symbol (lib_id "device:C") (at 74.93 128.27 0) (unit 1)
