File: latentpink/pcb/phy.kicad_sch (KiCad schematic)
At the start: 149 parts, among them J1 CONN_SFP_HOST, J18 BEL_FUSE_0845-2R1T-E4, J19 BEL_FUSE_0845-2R1T-E4, J2 SFP_CAGE, J20 BEL_FUSE_0845-2R1T-E4, J21 BEL_FUSE_0845-2R1T-E4, J3 XILINX_JTAG, J4 BEL_FUSE_0845-2R1T-E4, J8 BEL_FUSE_0845-2R1T-E4, M1 960-27-12-D-AB-0, U1 VSC8512, U2 XC7K160T-2FBG484C, U24 SIT9121AI-2BF-XXS200.000000G, U25 SIT9121AI-2BF-XXS156.250000G, U31 74LVC1T45, U32 74LVC1T45, U33 74LVC1T45, U34 74LVC1T45, U35 SIT9121AC-2B2-33E125.000000, U4 STM32H735-UFBGA176-25

Commit message: Finished initial schematic, ready for design review
Parts:
- C352, C353, C354: footprint (none) -> azonenberg_pcb:EIA_0402_CAP_NOSILK
- R105, R108, R109, R110, R111: footprint (none) -> azonenberg_pcb:EIA_0402_RES_NOSILK
Connections:
- no-connect marks 44 -> 50
Changed lines of the file:
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@@
   (junction (at 519.43 92.71) (diameter 0) (color 0 0 0 0)
   )
+  (no_connect (at 96.52 24.13))
   (no_connect (at 50.8 147.32))
   (no_connect (at 166.37 237.49))
@@
   (no_connect (at 99.06 104.14))
   (no_connect (at 97.79 137.16))
+  (no_connect (at 96.52 31.75))
   (no_connect (at 97.79 193.04))
   (no_connect (at 97.79 182.88))
@@
   (no_connect (at 50.8 144.78))
   (no_connect (at 50.8 175.26))
+  (no_connect (at 96.52 29.21))
   (no_connect (at 97.79 147.32))
   (no_connect (at 50.8 167.64))
   (no_connect (at 50.8 137.16))
+  (no_connect (at 96.52 26.67))
   (no_connect (at 50.8 139.7))
+  (no_connect (at 96.52 21.59))
   (no_connect (at 97.79 139.7))
   (no_connect (at 99.06 101.6))
+  (no_connect (at 96.52 34.29))
   (no_connect (at 50.8 152.4))
   (no_connect (at 97.79 175.26))
@@
     (effects (font (size 1.27 1.27)) (justify right bottom))
   )
-  (label "1V8_IO" (at 455.93 229.87 180)
-    (effects (font (size 1.27 1.27)) (justify right bottom))
-  )
   (label "VSC_CLKOUT_0" (at 314.96 259.08 0)
     (effects (font (size 1.27 1.27)) (justify left bottom))
@@
     (effects (font (size 1.27 1.27)) (justify left))
   )
+  (hierarchical_label "1V8_IO" (shape input) (at 455.93 229.87 180)
+    (effects (font (size 1.27 1.27)) (justify right))
+  )
   (hierarchical_label "VSC_MDINT_1V8" (shape output) (at 455.93 254 180)
     (effects (font (size 1.27 1.27)) (justify right))
@@
       (effects (font (size 1.27 1.27)) (justify left))
     )
-    (property "Footprint" "" (id 2) (at 213.0552 292.1 0)
+    (property "Footprint" "azonenberg_pcb:EIA_0402_CAP_NOSILK" (id 2) (at 213.0552 292.1 0)
       (effects (font (size 1.27 1.27)) hide)
     )
@@
     (property "Reference" "R110" (id 0) (at 234.95 290.83 90))
     (property "Value" "2K 1%" (id 1) (at 229.87 299.72 90))
-    (property "Footprint" "" (id 2) (at 229.87 293.878 90)
+    (property "Footprint" "azonenberg_pcb:EIA_0402_RES_NOSILK" (id 2) (at 229.87 293.878 90)
       (effects (font (size 1.27 1.27)) hide)
     )
@@
       (effects (font (size 1.27 1.27)) (justify left))
     )
-    (property "Footprint" "" (id 2) (at 202.8952 289.56 0)
+    (property "Footprint" "azonenberg_pcb:EIA_0402_CAP_NOSILK" (id 2) (at 202.8952 289.56 0)
       (effects (font (size 1.27 1.27)) hide)
     )
@@
     (property "Reference" "R111" (id 0) (at 234.95 293.37 90))
     (property "Value" "2K 1%" (id 1) (at 229.87 302.26 90))
-    (property "Footprint" "" (id 2) (at 229.87 296.418 90)
+    (property "Footprint" "azonenberg_pcb:EIA_0402_RES_NOSILK" (id 2) (at 229.87 296.418 90)
       (effects (font (size 1.27 1.27)) hide)
     )
@@
     (property "Reference" "R108" (id 0) (at 218.44 249.2842 90))
     (property "Value" "1K" (id 1) (at 218.44 251.8211 90))
-    (property "Footprint" "" (id 2) (at 218.44 255.778 90)
+    (property "Footprint" "azonenberg_pcb:EIA_0402_RES_NOSILK" (id 2) (at 218.44 255.778 90)
       (effects (font (size 1.27 1.27)) hide)
     )
@@
     (property "Reference" "R105" (id 0) (at 45.72 95.25 90))
     (property "Value" "620 1%" (id 1) (at 40.64 99.06 90))
-    (property "Footprint" "" (id 2) (at 40.64 98.298 90)
+    (property "Footprint" "azonenberg_pcb:EIA_0402_RES_NOSILK" (id 2) (at 40.64 98.298 90)
       (effects (font (size 1.27 1.27)) hide)
     )
@@
       (effects (font (size 1.27 1.27)) (justify left))
     )
-    (property "Footprint" "" (id 2) (at 192.7352 287.02 0)
+    (property "Footprint" "azonenberg_pcb:EIA_0402_CAP_NOSILK" (id 2) (at 192.7352 287.02 0)
       (effects (font (size 1.27 1.27)) hide)
     )
@@
     (property "Reference" "R109" (id 0) (at 234.95 288.29 90))
     (property "Value" "2K 1%" (id 1) (at 229.87 297.18 90))
-    (property "Footprint" "" (id 2) (at 229.87 291.338 90)
+    (property "Footprint" "azonenberg_pcb:EIA_0402_RES_NOSILK" (id 2) (at 229.87 291.338 90)
       (effects (font (size 1.27 1.27)) hide)
     )

Commit message: Finished initial schematic review, added ESD diodes to Ethernet pairs
Parts:
- added U40, U41, U42, U43, U44, U45, U46, U47, U48, U49, U50, U51, U52, U53, U54, U55, U56, U57, U58, U59, U60, U61, U62, U63: RCLAMP0514M, azonenberg_pcb:SOP_10_0.5MM_3MM, symbol special-azonenberg:RCLAMP0514M
Connections:
- net 2V5: now also U40.3 (Vcc), U41.3 (Vcc), U42.3 (Vcc), U43.3 (Vcc), U44.3 (Vcc), U45.3 (Vcc), U46.3 (Vcc), U47.3 (Vcc), U48.3 (Vcc), U49.3 (Vcc), U50.3 (Vcc), U51.3 (Vcc), U52.3 (Vcc), U53.3 (Vcc), U54.3 (Vcc), U55.3 (Vcc), U56.3 (Vcc), U57.3 (Vcc), U58.3 (Vcc), U59.3 (Vcc), U60.3 (Vcc), U61.3 (Vcc), U62.3 (Vcc), U63.3 (Vcc)
- net ETH0_D0_N: now also U48.1 (LINE_1), U48.10 (NC_1)
- net ETH0_D0_P: now also U48.2 (NC_2), U48.9 (LINE_2)
- net ETH0_D1_N: now also U48.4 (LINE_3), U48.7 (NC_3)
- net ETH0_D1_P: now also U48.5 (NC_4), U48.6 (LINE_4)
- net ETH0_D2_N: now also U49.1 (LINE_1), U49.10 (NC_1)
- net ETH0_D2_P: now also U49.2 (NC_2), U49.9 (LINE_2)
- net ETH0_D3_N: now also U49.4 (LINE_3), U49.7 (NC_3)
- net ETH0_D3_P: now also U49.5 (NC_4), U49.6 (LINE_4)
- net ETH10_D0_N: now also U40.1 (LINE_1), U40.10 (NC_1)
- net ETH10_D0_P: now also U40.2 (NC_2), U40.9 (LINE_2)
- net ETH10_D1_N: now also U40.4 (LINE_3), U40.7 (NC_3)
- net ETH10_D1_P: now also U40.5 (NC_4), U40.6 (LINE_4)
- net ETH10_D2_N: now also U43.1 (LINE_1), U43.10 (NC_1)
- net ETH10_D2_P: now also U43.2 (NC_2), U43.9 (LINE_2)
- net ETH10_D3_N: now also U43.4 (LINE_3), U43.7 (NC_3)
- net ETH10_D3_P: now also U43.5 (NC_4), U43.6 (LINE_4)
- net ETH11_D0_N: now also U46.1 (LINE_1), U46.10 (NC_1)
- net ETH11_D0_P: now also U46.2 (NC_2), U46.9 (LINE_2)
- net ETH11_D1_N: now also U46.4 (LINE_3), U46.7 (NC_3)
- net ETH11_D1_P: now also U46.5 (NC_4), U46.6 (LINE_4)
- net ETH11_D2_N: now also U47.1 (LINE_1), U47.10 (NC_1)
- net ETH11_D2_P: now also U47.2 (NC_2), U47.9 (LINE_2)
- net ETH11_D3_N: now also U47.4 (LINE_3), U47.7 (NC_3)
- net ETH11_D3_P: now also U47.5 (NC_4), U47.6 (LINE_4)
- net ETH1_D0_N: now also U52.1 (LINE_1), U52.10 (NC_1)
- net ETH1_D0_P: now also U52.2 (NC_2), U52.9 (LINE_2)
- net ETH1_D1_N: now also U52.4 (LINE_3), U52.7 (NC_3)
- net ETH1_D1_P: now also U52.5 (NC_4), U52.6 (LINE_4)
- net ETH1_D2_N: now also U53.1 (LINE_1), U53.10 (NC_1)
- net ETH1_D2_P: now also U53.2 (NC_2), U53.9 (LINE_2)
- net ETH1_D3_N: now also U53.4 (LINE_3), U53.7 (NC_3)
- net ETH1_D3_P: now also U53.5 (NC_4), U53.6 (LINE_4)
- net ETH2_D0_N: now also U56.1 (LINE_1), U56.10 (NC_1)
- net ETH2_D0_P: now also U56.2 (NC_2), U56.9 (LINE_2)
- net ETH2_D1_N: now also U56.4 (LINE_3), U56.7 (NC_3)
- net ETH2_D1_P: now also U56.5 (NC_4), U56.6 (LINE_4)
- net ETH2_D2_N: now also U57.1 (LINE_1), U57.10 (NC_1)
- net ETH2_D2_P: now also U57.2 (NC_2), U57.9 (LINE_2)
- net ETH2_D3_N: now also U57.4 (LINE_3), U57.7 (NC_3)
- net ETH2_D3_P: now also U57.5 (NC_4), U57.6 (LINE_4)
- net ETH3_D0_N: now also U60.1 (LINE_1), U60.10 (NC_1)
- net ETH3_D0_P: now also U60.2 (NC_2), U60.9 (LINE_2)
- net ETH3_D1_N: now also U60.4 (LINE_3), U60.7 (NC_3)
- net ETH3_D1_P: now also U60.5 (NC_4), U60.6 (LINE_4)
- net ETH3_D2_N: now also U61.1 (LINE_1), U61.10 (NC_1)
- net ETH3_D2_P: now also U61.2 (NC_2), U61.9 (LINE_2)
- net ETH3_D3_N: now also U61.4 (LINE_3), U61.7 (NC_3)
- net ETH3_D3_P: now also U61.5 (NC_4), U61.6 (LINE_4)
- net ETH4_D0_N: now also U41.1 (LINE_1), U41.10 (NC_1)
- net ETH4_D0_P: now also U41.2 (NC_2), U41.9 (LINE_2)
- net ETH4_D1_N: now also U41.4 (LINE_3), U41.7 (NC_3)
- net ETH4_D1_P: now also U41.5 (NC_4), U41.6 (LINE_4)
- net ETH4_D2_N: now also U42.1 (LINE_1), U42.10 (NC_1)
- net ETH4_D2_P: now also U42.2 (NC_2), U42.9 (LINE_2)
- net ETH4_D3_N: now also U42.4 (LINE_3), U42.7 (NC_3)
- net ETH4_D3_P: now also U42.5 (NC_4), U42.6 (LINE_4)
- net ETH5_D0_N: now also U44.1 (LINE_1), U44.10 (NC_1)
- net ETH5_D0_P: now also U44.2 (NC_2), U44.9 (LINE_2)
- net ETH5_D1_N: now also U44.4 (LINE_3), U44.7 (NC_3)
- net ETH5_D1_P: now also U44.5 (NC_4), U44.6 (LINE_4)
- net ETH5_D2_N: now also U45.1 (LINE_1), U45.10 (NC_1)
- net ETH5_D2_P: now also U45.2 (NC_2), U45.9 (LINE_2)
- net ETH5_D3_N: now also U45.4 (LINE_3), U45.7 (NC_3)
- net ETH5_D3_P: now also U45.5 (NC_4), U45.6 (LINE_4)
- net ETH6_D0_N: now also U50.1 (LINE_1), U50.10 (NC_1)
- net ETH6_D0_P: now also U50.2 (NC_2), U50.9 (LINE_2)
- net ETH6_D1_N: now also U50.4 (LINE_3), U50.7 (NC_3)
- net ETH6_D1_P: now also U50.5 (NC_4), U50.6 (LINE_4)
- net ETH6_D2_N: now also U51.1 (LINE_1), U51.10 (NC_1)
- net ETH6_D2_P: now also U51.2 (NC_2), U51.9 (LINE_2)
- net ETH6_D3_N: now also U51.4 (LINE_3), U51.7 (NC_3)
- net ETH6_D3_P: now also U51.5 (NC_4), U51.6 (LINE_4)
- net ETH7_D0_N: now also U54.1 (LINE_1), U54.10 (NC_1)
- net ETH7_D0_P: now also U54.2 (NC_2), U54.9 (LINE_2)
- net ETH7_D1_N: now also U54.4 (LINE_3), U54.7 (NC_3)
- net ETH7_D1_P: now also U54.5 (NC_4), U54.6 (LINE_4)
- net ETH7_D2_N: now also U55.1 (LINE_1), U55.10 (NC_1)
- net ETH7_D2_P: now also U55.2 (NC_2), U55.9 (LINE_2)
- net ETH7_D3_N: now also U55.4 (LINE_3), U55.7 (NC_3)
- net ETH7_D3_P: now also U55.5 (NC_4), U55.6 (LINE_4)
- net ETH8_D0_N: now also U58.1 (LINE_1), U58.10 (NC_1)
- net ETH8_D0_P: now also U58.2 (NC_2), U58.9 (LINE_2)
- net ETH8_D1_N: now also U58.4 (LINE_3), U58.7 (NC_3)
- net ETH8_D1_P: now also U58.5 (NC_4), U58.6 (LINE_4)
- net ETH8_D2_N: now also U59.1 (LINE_1), U59.10 (NC_1)
- net ETH8_D2_P: now also U59.2 (NC_2), U59.9 (LINE_2)
- net ETH8_D3_N: now also U59.4 (LINE_3), U59.7 (NC_3)
- net ETH8_D3_P: now also U59.5 (NC_4), U59.6 (LINE_4)
- net ETH9_D0_N: now also U62.1 (LINE_1), U62.10 (NC_1)
- net ETH9_D0_P: now also U62.2 (NC_2), U62.9 (LINE_2)
- net ETH9_D1_N: now also U62.4 (LINE_3), U62.7 (NC_3)
- net ETH9_D1_P: now also U62.5 (NC_4), U62.6 (LINE_4)
- net ETH9_D2_N: now also U63.1 (LINE_1), U63.10 (NC_1)
- net ETH9_D2_P: now also U63.2 (NC_2), U63.9 (LINE_2)
- net ETH9_D3_N: now also U63.4 (LINE_3), U63.7 (NC_3)
- net ETH9_D3_P: now also U63.5 (NC_4), U63.6 (LINE_4)
- net GND: now also U40.8 (Gnd), U41.8 (Gnd), U42.8 (Gnd), U43.8 (Gnd), U44.8 (Gnd), U45.8 (Gnd), U46.8 (Gnd), U47.8 (Gnd), U48.8 (Gnd), U49.8 (Gnd), U50.8 (Gnd), U51.8 (Gnd), U52.8 (Gnd), U53.8 (Gnd), U54.8 (Gnd), U55.8 (Gnd), U56.8 (Gnd), U57.8 (Gnd), U58.8 (Gnd), U59.8 (Gnd), U60.8 (Gnd), U61.8 (Gnd), U62.8 (Gnd), U63.8 (Gnd)
Other:
- note added: "ESD protection"
- moved on the sheet: C458, C459, C460, C461, C462, C463, C464, C465, C469, C470, C471, C472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

Commit message: Preliminary routing of first four baseT interfaces on VSC8512
Connections:
- net ETH0_D0_N: now also U1.G25 (P1_D0_N), U48.4 (LINE_3), U48.7 (NC_3); no longer U1.L25 (P0_D0_N), U48.1 (LINE_1), U48.10 (NC_1)
- net ETH0_D0_P: now also U1.G26 (P1_D0_P), U48.5 (NC_4), U48.6 (LINE_4); no longer U1.L26 (P0_D0_P), U48.2 (NC_2), U48.9 (LINE_2)
- net ETH0_D1_N: now also U1.H25 (P1_D1_N), U48.1 (LINE_1), U48.10 (NC_1); no longer U1.M25 (P0_D1_N), U48.4 (LINE_3), U48.7 (NC_3)
- net ETH0_D1_P: now also U1.H26 (P1_D1_P), U48.2 (NC_2), U48.9 (LINE_2); no longer U1.M26 (P0_D1_P), U48.5 (NC_4), U48.6 (LINE_4)
- net ETH0_D2_N: now also U1.J25 (P1_D2_N), U49.5 (NC_4), U49.6 (LINE_4); no longer U1.N25 (P0_D2_N), U49.1 (LINE_1), U49.10 (NC_1)
- net ETH0_D2_P: now also U1.J26 (P1_D2_P), U49.4 (LINE_3), U49.7 (NC_3); no longer U1.N26 (P0_D2_P), U49.2 (NC_2), U49.9 (LINE_2)
- net ETH0_D3_N: now also U1.K25 (P1_D3_N), U49.1 (LINE_1), U49.10 (NC_1); no longer U1.P25 (P0_D3_N), U49.4 (LINE_3), U49.7 (NC_3)
- net ETH0_D3_P: now also U1.K26 (P1_D3_P), U49.2 (NC_2), U49.9 (LINE_2); no longer U1.P26 (P0_D3_P), U49.5 (NC_4), U49.6 (LINE_4)
- net ETH1_D0_N: now also U1.M25 (P0_D1_N); no longer U1.G25 (P1_D0_N)
- net ETH1_D0_P: now also U1.M26 (P0_D1_P); no longer U1.G26 (P1_D0_P)
- net ETH1_D1_N: now also U1.L25 (P0_D0_N); no longer U1.H25 (P1_D1_N)
- net ETH1_D1_P: now also U1.L26 (P0_D0_P); no longer U1.H26 (P1_D1_P)
- net ETH1_D2_N: now also U1.P25 (P0_D3_N); no longer U1.J25 (P1_D2_N)
- net ETH1_D2_P: now also U1.P26 (P0_D3_P); no longer U1.J26 (P1_D2_P)
- net ETH1_D3_N: now also U1.N25 (P0_D2_N); no longer U1.K25 (P1_D3_N)
- net ETH1_D3_P: now also U1.N26 (P0_D2_P); no longer U1.K26 (P1_D3_P)
- net ETH2_D0_N: now also U1.B22 (P3_D0_N), U56.4 (LINE_3), U56.7 (NC_3); no longer U1.C25 (P2_D0_N), U56.1 (LINE_1), U56.10 (NC_1)
- net ETH2_D0_P: now also U1.A22 (P3_D0_P), U56.5 (NC_4), U56.6 (LINE_4); no longer U1.C26 (P2_D0_P), U56.2 (NC_2), U56.9 (LINE_2)
- net ETH2_D1_N: now also U1.B23 (P3_D1_N), U56.1 (LINE_1), U56.10 (NC_1); no longer U1.D25 (P2_D1_N), U56.4 (LINE_3), U56.7 (NC_3)
- net ETH2_D1_P: now also U1.A23 (P3_D1_P), U56.2 (NC_2), U56.9 (LINE_2); no longer U1.D26 (P2_D1_P), U56.5 (NC_4), U56.6 (LINE_4)
- net ETH2_D2_N: now also U1.B24 (P3_D2_N), U57.5 (NC_4), U57.6 (LINE_4); no longer U1.E25 (P2_D2_N), U57.1 (LINE_1), U57.10 (NC_1)
- net ETH2_D2_P: now also U1.A24 (P3_D2_P), U57.4 (LINE_3), U57.7 (NC_3); no longer U1.E26 (P2_D2_P), U57.2 (NC_2), U57.9 (LINE_2)
- net ETH2_D3_N: now also U1.B25 (P3_D3_N), U57.1 (LINE_1), U57.10 (NC_1); no longer U1.F25 (P2_D3_N), U57.4 (LINE_3), U57.7 (NC_3)
- net ETH2_D3_P: now also U1.A25 (P3_D3_P), U57.2 (NC_2), U57.9 (LINE_2); no longer U1.F26 (P2_D3_P), U57.5 (NC_4), U57.6 (LINE_4)
- net ETH3_D0_N: now also U1.D25 (P2_D1_N); no longer U1.B22 (P3_D0_N)
- net ETH3_D0_P: now also U1.D26 (P2_D1_P); no longer U1.A22 (P3_D0_P)
- net ETH3_D1_N: now also U1.C25 (P2_D0_N); no longer U1.B23 (P3_D1_N)
- net ETH3_D1_P: now also U1.C26 (P2_D0_P); no longer U1.A23 (P3_D1_P)
- net ETH3_D2_N: now also U1.F25 (P2_D3_N); no longer U1.B24 (P3_D2_N)
- net ETH3_D2_P: now also U1.F26 (P2_D3_P); no longer U1.A24 (P3_D2_P)
- net ETH3_D3_N: now also U1.E25 (P2_D2_N); no longer U1.B25 (P3_D3_N)
- net ETH3_D3_P: now also U1.E26 (P2_D2_P); no longer U1.A25 (P3_D3_P)
Other:
- note added: "Per table 5 (page 23) Can swap A/B pairs Can swap C/D pairs But cannot swap A/B with C/D"
