File: latentpink/pcb/phy.kicad_sch (KiCad schematic)
At the start: 173 parts, among them J1 CONN_SFP_HOST, J18 BEL_FUSE_0845-2R1T-E4, J19 BEL_FUSE_0845-2R1T-E4, J2 SFP_CAGE, J20 BEL_FUSE_0845-2R1T-E4, J21 BEL_FUSE_0845-2R1T-E4, J3 XILINX_JTAG, J4 BEL_FUSE_0845-2R1T-E4, J8 BEL_FUSE_0845-2R1T-E4, M1 960-27-12-D-AB-0, U1 VSC8512, U2 XC7K160T-2FBG484C, U24 SIT9121AI-2BF-XXS200.000000G, U25 SIT9121AI-2BF-XXS156.250000G, U31 74LVC1T45, U32 74LVC1T45, U33 74LVC1T45, U34 74LVC1T45, U35 SIT9121AC-2B2-33E125.000000, U4 STM32H735-UFBGA176-25, U40 RCLAMP0514M, U41 RCLAMP0514M, U42 RCLAMP0514M, U43 RCLAMP0514M, U44 RCLAMP0514M, U45 RCLAMP0514M, U46 RCLAMP0514M, U47 RCLAMP0514M, U48 RCLAMP0514M, U49 RCLAMP0514M, U50 RCLAMP0514M, U51 RCLAMP0514M, U52 RCLAMP0514M, U53 RCLAMP0514M, U54 RCLAMP0514M, U55 RCLAMP0514M, U56 RCLAMP0514M, U57 RCLAMP0514M, U58 RCLAMP0514M, U59 RCLAMP0514M, U60 RCLAMP0514M, U61 RCLAMP0514M, U62 RCLAMP0514M, U63 RCLAMP0514M

Commit message: Lots of layout progress on bottom power/management/supervisor area
Connections:
- net 2V5: now also R106.1; no longer R106.2
- net ETH10_D0_N: now also U1.P2 (P11_D0_N); no longer U1.K2 (P10_D0_N)
- net ETH10_D0_P: now also U1.P1 (P11_D0_P); no longer U1.K1 (P10_D0_P)
- net ETH10_D1_N: now also U1.N2 (P11_D1_N); no longer U1.J2 (P10_D1_N)
- net ETH10_D1_P: now also U1.N1 (P11_D1_P); no longer U1.J1 (P10_D1_P)
- net ETH10_D2_N: now also U1.M2 (P11_D2_N); no longer U1.H2 (P10_D2_N)
- net ETH10_D2_P: now also U1.M1 (P11_D2_P); no longer U1.H1 (P10_D2_P)
- net ETH10_D3_N: now also U1.L2 (P11_D3_N); no longer U1.G2 (P10_D3_N)
- net ETH10_D3_P: now also U1.L1 (P11_D3_P); no longer U1.G1 (P10_D3_P)
- net ETH11_D0_N: now also U1.J2 (P10_D1_N); no longer U1.P2 (P11_D0_N)
- net ETH11_D0_P: now also U1.J1 (P10_D1_P); no longer U1.P1 (P11_D0_P)
- net ETH11_D1_N: now also U1.K2 (P10_D0_N); no longer U1.N2 (P11_D1_N)
- net ETH11_D1_P: now also U1.K1 (P10_D0_P); no longer U1.N1 (P11_D1_P)
- net ETH11_D2_N: now also U1.G2 (P10_D3_N); no longer U1.M2 (P11_D2_N)
- net ETH11_D2_P: now also U1.G1 (P10_D3_P); no longer U1.M1 (P11_D2_P)
- net ETH11_D3_N: now also U1.H2 (P10_D2_N); no longer U1.L2 (P11_D3_N)
- net ETH11_D3_P: now also U1.H1 (P10_D2_P); no longer U1.L1 (P11_D3_P)
- net ETH7_D0_N: now also U1.B11 (P6_D1_N); no longer U1.B10 (P6_D0_N)
- net ETH7_D0_P: now also U1.A11 (P6_D1_P); no longer U1.A10 (P6_D0_P)
- net ETH7_D1_N: now also U1.B10 (P6_D0_N); no longer U1.B11 (P6_D1_N)
- net ETH7_D1_P: now also U1.A10 (P6_D0_P); no longer U1.A11 (P6_D1_P)
- net ETH7_D2_N: now also U1.B13 (P6_D3_N); no longer U1.B12 (P6_D2_N)
- net ETH7_D2_P: now also U1.A13 (P6_D3_P); no longer U1.A12 (P6_D2_P)
- net ETH7_D3_N: now also U1.B12 (P6_D2_N); no longer U1.B13 (P6_D3_N)
- net ETH7_D3_P: now also U1.A12 (P6_D2_P); no longer U1.A13 (P6_D3_P)
- net ETH8_D0_N: now also U1.E2 (P9_D1_N); no longer U1.B2 (P8_D0_N)
- net ETH8_D0_P: now also U1.E1 (P9_D1_P); no longer U1.A2 (P8_D0_P)
- net ETH8_D1_N: now also U1.F2 (P9_D0_N); no longer U1.B3 (P8_D1_N)
- net ETH8_D1_P: now also U1.F1 (P9_D0_P); no longer U1.A3 (P8_D1_P)
- net ETH8_D2_N: now also U1.C2 (P9_D3_N); no longer U1.B4 (B8_D2_N)
- net ETH8_D2_P: now also U1.C1 (P9_D3_P); no longer U1.A4 (P8_D2_P)
- net ETH8_D3_N: now also U1.D2 (P9_D2_N); no longer U1.B5 (P8_D3_N)
- net ETH8_D3_P: now also U1.D1 (P9_D2_P); no longer U1.A5 (P8_D3_P)
- net ETH9_D0_N: now also U1.B3 (P8_D1_N); no longer U1.F2 (P9_D0_N)
- net ETH9_D0_P: now also U1.A3 (P8_D1_P); no longer U1.F1 (P9_D0_P)
- net ETH9_D1_N: now also U1.B2 (P8_D0_N); no longer U1.E2 (P9_D1_N)
- net ETH9_D1_P: now also U1.A2 (P8_D0_P); no longer U1.E1 (P9_D1_P)
- net ETH9_D2_N: now also U1.B5 (P8_D3_N); no longer U1.D2 (P9_D2_N)
- net ETH9_D2_P: now also U1.A5 (P8_D3_P); no longer U1.D1 (P9_D2_P)
- net ETH9_D3_N: now also U1.B4 (B8_D2_N); no longer U1.C2 (P9_D3_N)
- net ETH9_D3_P: now also U1.A4 (P8_D2_P); no longer U1.C1 (P9_D3_P)
- net PHY0_LED0_N: now also R81.1; no longer R82.1
- net PHY0_LED1_N: now also R93.1; no longer R94.1
- net PHY1_LED0_N: now also R82.1; no longer R81.1
- net PHY1_LED1_N: now also R94.1; no longer R93.1
- net PHY2_LED0_N: now also R83.1; no longer R84.1
- net PHY2_LED1_N: now also R95.1; no longer R96.1
- net PHY3_LED0_N: now also R84.1; no longer R83.1
- net PHY3_LED1_N: now also R96.1; no longer R95.1
- net PHY4_LED0_N: now also R85.1; no longer R86.1
- net PHY4_LED1_N: now also R97.1; no longer R98.1
- net PHY5_LED0_N: now also R86.1; no longer R85.1
- net PHY5_LED1_N: now also R98.1; no longer R97.1
- net PHY6_LED0_N: now also R87.1; no longer R88.1
- net PHY6_LED1_N: now also R99.1; no longer R100.1
- net PHY7_LED0_N: now also R88.1; no longer R87.1
- net PHY7_LED1_N: now also R100.1; no longer R99.1
- net VSC_RST_N: now also R106.2; no longer R106.1
- net at R103.2: now also U1.V4 (PHY11_LED1); no longer U1.W1 (PHY10_LED1)
- net at R83.2: now also U1.U4 (PHY3_LED0); no longer U1.V1 (PHY2_LED0)
- net at R90.2: now also U1.T3 (PHY8_LED0); no longer U1.T2 (PHY9_LED0)
- net at R93.2: now also U1.AA2 (PHY1_LED1); no longer U1.AA3 (PHY0_LED1)
- net at R101.2: now also U1.W2 (PHY9_LED1); no longer U1.W3 (PHY8_LED1)
- net at U1.AA1 (PHY2_LED1): now also R96.2; no longer R95.2
- net at R94.2: now also U1.AA3 (PHY0_LED1); no longer U1.AA2 (PHY1_LED1)
- net at U1.R4 (PHY11_LED0): now also R91.2; no longer R92.2
- net at U1.T1 (PHY10_LED0): now also R92.2; no longer R91.2
- net at R89.2: now also U1.T2 (PHY9_LED0); no longer U1.T3 (PHY8_LED0)
- net at U1.T4 (PHY7_LED0): now also R87.2; no longer R88.2
- net at U1.U1 (PHY6_LED0): now also R88.2; no longer R87.2
- net at U1.U2 (PHY5_LED0): now also R85.2; no longer R86.2
- net at U1.U3 (PHY4_LED0): now also R86.2; no longer R85.2
- net at R84.2: now also U1.V1 (PHY2_LED0); no longer U1.U4 (PHY3_LED0)
- net at U1.V2 (PHY1_LED0): now also R81.2; no longer R82.2
- net at U1.V3 (PHY0_LED0): now also R82.2; no longer R81.2
- net at R104.2: now also U1.W1 (PHY10_LED1); no longer U1.V4 (PHY11_LED1)
- net at R102.2: now also U1.W3 (PHY8_LED1); no longer U1.W2 (PHY9_LED1)
- net at U1.W4 (PHY7_LED1): now also R99.2; no longer R100.2
- net at U1.Y1 (PHY6_LED1): now also R100.2; no longer R99.2
- net at U1.Y2 (PHY5_LED1): now also R97.2; no longer R98.2
- net at U1.Y3 (PHY4_LED1): now also R98.2; no longer R97.2
- net at U1.Y4 (PHY3_LED1): now also R95.2; no longer R96.2
Other:
- note added: "!!SIGNOFF REVIEW CHECK!!"
- note added: "Verify LEDs and diffpairs match up to the same port Verify all pin swaps comply with rules for PHY"
- moved on the sheet: R100, R101, R102, R103, R104, R106, R81, R82, R83, R84, R85, R86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
