File: latentpink/pcb/latentpink.kicad_pcb (KiCad board)
At the start: 8 copper layers, 145 x 139 mm, 829 parts, among them J1 CONN_SFP_HOST, J10 XILINX_JTAG, J11 FAN_01, J12 FAN_01, J13 CONN_01X05, J14 CONN_01X03, J15 CONN_01X03, J16 JUMPER_0402_SPDT, J17 JUMPER_0402_SPDT, J18 BEL_FUSE_0845-2R1T-E4, J19 BEL_FUSE_0845-2R1T-E4, J2 SFP_CAGE, J20 BEL_FUSE_0845-2R1T-E4, J21 BEL_FUSE_0845-2R1T-E4, J22 BEL_FUSE_0845-2R1T-E4, J23 PMOD_HOST, J3 XILINX_JTAG, J4 BEL_FUSE_0845-2R1T-E4, J5 0826-1G1T-23-F, J6 BARREL_JACK, J7 RJ45, J8 BEL_FUSE_0845-2R1T-E4, J9 XILINX_JTAG, M1 960-27-12-D-AB-0, M10 WEEE, M2 960-23-23-F-AB-0, M3 SCREWHOLE, M4 SCREWHOLE, M5 SCREWHOLE, M6 SCREWHOLE, M7 LONGTHING, M8 OSHW, M9 POLARITY, U1 VSC8512, U10 MYMGK1R812ERSR, U11 MYMGK00504ERSR, U12 STM32L031-QFN32, U13 MYMGK00504ERSR, U14 MYMGK00504ERSR, U15 MYMGK00504ERSR, U16 NCP45521IMNTWG-H, U17 NCP45521IMNTWG-H, U18 LP2996AMRE, U19 TPS7A2533DRVR, U2 XC7K160T-2FBG484C, U20 AT24MAC402, U21 ECX2-LMV-3CN-125.000-TR, U22 ECS-2016MVQ-250-CN, U23 ADM3101E_QFN, U24 SIT9121AI-2BF-XXS200.000000G, U25 SIT9121AI-2BF-XXS156.250000G, U26 74LVC1T45, U27 74LVC1T45, U28 IS25WP256D-JLLE, U29 DSC1123CI2-150.0000T, U3 CY7C2245KV18-450BZXI, U30 DSC1123CI2-150.0000T, U31 74LVC1T45, U32 74LVC1T45, U33 74LVC1T45, U34 74LVC1T45, U35 SIT9121AC-2B2-33E125.000000, U36 AT30TS74_UDFN, U37 AT30TS74_UDFN, U38 AT30TS74_UDFN, U39 AT30TS74_UDFN, U4 STM32H735-UFBGA176-25, U40 RCLAMP0514M, U41 RCLAMP0514M, U42 RCLAMP0514M, U43 RCLAMP0514M, U44 RCLAMP0514M, U45 RCLAMP0514M, U46 RCLAMP0514M, U47 RCLAMP0514M, U48 RCLAMP0514M, U49 RCLAMP0514M, U5 DP83867, U50 RCLAMP0514M, U51 RCLAMP0514M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

Commit message: Rearranged all unplaced components and grouped by functional subsystem
Parts:
- removed R112: 1.5K, azonenberg_pcb:EIA_0402_RES_NOSILK
- C111, C175, C176, C191, C192, C206, R117, R118, R130, R131, R132, R133, R151, R152, R22, R29, R30, R40, R41, R42, R43, R44, R45, R46, R47, R74, R75, R76, R78, R79: moved to B.Cu
- moved R139 263.3 mm to (221.2, 36.5)
- moved R146 263.0 mm to (219.8, 32.0)
- moved R140 260.7 mm to (209.8, 32.2)
- moved R145 259.6 mm to (214.0, 32.5)
- moved R138 258.0 mm to (214.5, 39.5)
- moved R137 256.4 mm to (209.5, 38.8)
- moved R142 254.8 mm to (209.0, 35.5)
- moved R148 254.7 mm to (217.8, 36.8)
- moved R147 253.5 mm to (214.0, 36.8)
- moved R144 250.0 mm to (203.2, 33.2)
- moved R141 243.3 mm to (203.0, 39.0)
- moved R143 239.9 mm to (201.8, 37.0)
- moved R152 198.5 mm to (150.0, 26.5)
- moved R151 197.8 mm to (150.0, 35.0)
- moved R3 188.4 mm to (101.5, 4.75)
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Connections:
- R44 pad 1: /1V8 -> /1V8_IO
- R76 pad 1: /1V8 -> /1V8_IO
Routing:
- net /QSGMII PHY/ETH11_D3_P: track 16.5 -> 54.6 mm, vias 1 -> 2
- net /QSGMII PHY/ETH11_D3_N: track 16.5 -> 54.6 mm, vias 1 -> 2
- net /QSGMII PHY/ETH11_D2_N: track 15.5 -> 51.1 mm, vias 1 -> 2
- net /QSGMII PHY/ETH11_D2_P: track 15.5 -> 51.0 mm, vias 1 -> 2
- net /QSGMII PHY/ETH11_D1_P: track 15.1 -> 50.1 mm, vias 1 -> 2
- net /QSGMII PHY/ETH11_D1_N: track 15.2 -> 50.2 mm, vias 1 -> 2
- net /GND: track 1676.2 -> 1709.4 mm, vias 678 -> 688
- net /QSGMII PHY/ETH11_D0_N: track 15.0 -> 47.9 mm, vias 1 -> 2
- net /QSGMII PHY/ETH11_D0_P: track 14.9 -> 47.8 mm, vias 1 -> 2
- net /3V3: track 466.1 -> 494.8 mm, vias 35 -> 38
- net /QSGMII PHY/ETH10_D3_N: track 4.00 -> 32.0 mm, vias 0 -> 1
- net /QSGMII PHY/ETH10_D3_P: track 4.00 -> 31.8 mm, vias 0 -> 1
- net /QSGMII PHY/ETH10_D2_P: track 4.00 -> 27.7 mm, vias 0 -> 1
- net /QSGMII PHY/ETH10_D2_N: track 4.00 -> 27.6 mm, vias 0 -> 1
- net /Management/MCU_IRQ: track 11.5 -> 0.00 mm, vias 1 -> 0
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Other:
- board text added: "12V DC"
- board text added: "1V0 supply"
- board text added: "1V2 supply"
- board text added: "1V8 supply"
- board text added: "1V8_IO switch"
- board text added: "Bulk power filtering"
- board text added: "Chassis ground bond"
- board text added: "DP83867 power"
- board text added: "DP83867 straps"
- board text added: "FPGA flash"
- board text added: "GTX 1V0"
- board text added: "GTX 1V2"
- board text added: "GTX 1V8"
- board text added: "Ground clips"
- board text added: "KSZ9031 clocking"
- board text added: "KSZ9031 power"
- board text added: "MAC EEPROM"
- board text added: "Main system clock"
- board text added: "QDR clocking"
- board text added: "QDR decoupling"
- board text added: "QDR termination"
- board text added: "SFP power"
- board text added: "Super level shift"
- board text added: "System clock"
- board text added: "Thermal sensors"
- board text added: "VCCAUX"
- board text added: "VCCINT / VCCBRAM"
- board text added: "VCCO 1V8"
- board text added: "VCCO 3V3"
- board text added: "Vtt / Vref supply"
