File: latentpink/pcb/qdr.kicad_sch (KiCad schematic)
At the start: 69 parts, among them U2 XC7K160T-2FBG484C, U28 IS25WP256D-JLLE, U29 DSC1123CI2-150.0000T, U3 CY7C2245KV18-450BZXI

Commit message: Lots more layout of low speed stuff and power. Partial layout of 1.2V supply. Initial RGMII escape routing.
Connections:
- net I2C_DERP_SCL: now also U2.AA18 (IO_L15P_T2_DQS_13), U2.Y16 (IO_L21N_T3_DQS_13); no longer U2.M17 (IO_L14P_T2_SRCC_14), U2.P17 (IO_L21N_T3_DQS_A06_D22_14)
- net I2C_DERP_SDA: now also U2.AB18 (IO_L15N_T2_DQS_13), U2.W16 (IO_L21P_T3_DQS_13); no longer U2.P21 (IO_L22P_T3_A05_D21_14), U2.R17 (IO_L21P_T3_DQS_14)
Changed lines of the file:
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@@
   (paper "A3")
   (title_block
-    (date "2023-05-31")
+    (date "2023-06-01")
     (rev "0.1")
     (company "Antikernel Labs")
@@
   (no_connect (at 269.24 142.24))
   (no_connect (at 198.12 25.4))
+  (no_connect (at 269.24 132.08))
   (no_connect (at 346.71 132.08))
   (no_connect (at 346.71 99.06))
   (no_connect (at 33.02 181.61))
+  (no_connect (at 269.24 134.62))
   (no_connect (at 346.71 129.54))
   (no_connect (at 346.71 25.4))
@@
   (no_connect (at 269.24 149.86))
   (no_connect (at 269.24 48.26))
-  (no_connect (at 198.12 132.08))
   (no_connect (at 346.71 101.6))
   (no_connect (at 269.24 55.88))
@@
   (no_connect (at 346.71 116.84))
   (no_connect (at 200.66 261.62))
-  (no_connect (at 198.12 99.06))
   (no_connect (at 33.02 176.53))
   (no_connect (at 346.71 149.86))
   (no_connect (at 200.66 264.16))
+  (no_connect (at 269.24 129.54))
   (no_connect (at 33.02 179.07))
   (no_connect (at 269.24 91.44))
   (no_connect (at 346.71 71.12))
   (no_connect (at 269.24 139.7))
-  (no_connect (at 198.12 101.6))
   (no_connect (at 198.12 38.1))
-  (no_connect (at 198.12 129.54))
   (no_connect (at 198.12 149.86))
   (no_connect (at 346.71 86.36))
   (no_connect (at 269.24 119.38))
+  (no_connect (at 269.24 93.98))
   (wire (pts (xy 88.9 209.55) (xy 101.6 209.55))
     (stroke (width 0) (type default) (color 0 0 0 0))
@@
     (effects (font (size 1.27 1.27)) (justify right bottom))
   )
-  (label "I2C_DERP_SCL" (at 269.24 132.08 180)
+  (label "I2C_DERP_SCL" (at 198.12 132.08 180)
     (effects (font (size 1.27 1.27)) (justify right bottom))
   )
@@
     (effects (font (size 1.27 1.27)) (justify right bottom))
   )
-  (label "I2C_DERP_SDA" (at 269.24 134.62 180)
+  (label "I2C_DERP_SDA" (at 198.12 101.6 180)
     (effects (font (size 1.27 1.27)) (justify right bottom))
   )
@@
     (effects (font (size 1.27 1.27)) (justify right bottom))
   )
-  (label "I2C_DERP_SDA" (at 269.24 129.54 180)
+  (label "I2C_DERP_SDA" (at 198.12 129.54 180)
     (effects (font (size 1.27 1.27)) (justify right bottom))
   )
@@
     (effects (font (size 1.27 1.27)) (justify right bottom))
   )
-  (label "I2C_DERP_SCL" (at 269.24 93.98 180)
-    (effects (font (size 1.27 1.27)) (justify right bottom))
-  )
+  (label "I2C_DERP_SCL" (at 198.12 99.06 180)
+    (effects (font (size 1.27 1.27)) (justify right bottom))
+  )

Commit message: Partial routing of QDR D/Q bus, but it's a huge nightmare that might not be doable using MIG pinout
Parts:
- added R167: 1K, azonenberg_pcb:EIA_0402_RES_NOSILK, symbol device:R
- added R168: DNP, azonenberg_pcb:EIA_0402_RES_NOSILK, symbol device:R
Connections:
- net 1V8_IO: now also R168.2
- net GND: now also R167.2
- net QDR_BWS_0_N: now also U2.W21 (IO_L4P_T0_13); no longer U2.AA15 (IO_L18N_T2_13)
- net QDR_BWS_1_N: now also U2.Y22 (IO_L7N_T1_13); no longer U2.W19 (IO_12N_T1_MRCC_13)
- net QDR_BWS_2_N: now also U2.AA15 (IO_L18N_T2_13); no longer U2.T20 (IO_L6P_T0_13)
- net QDR_D0: now also U2.T20 (IO_L6P_T0_13); no longer U2.Y18 (IO_L13P_T2_MRCC_13)
- net QDR_D1: now also U2.U17 (IO_L5P_T0_13); no longer U2.Y19 (IO_L13N_T2_MRCC_13)
- net QDR_D10: now also U2.W19 (IO_12N_T1_MRCC_13); no longer U2.Y22 (IO_L7N_T1_13)
- net QDR_D11: now also U2.Y21 (IO_L7P_T1_13); no longer U2.AA20 (IO_L8P_T1_13)
- net QDR_D12: now also U2.V19 (IO_L12P_T1_MRCC_13); no longer U2.AB21 (IO_L8N_T1_13)
- net QDR_D13: now also U2.V20 (IO_L11P_T1_SRCC_13); no longer U2.AA19 (IO_L10_PT1_13)
- net QDR_D15: now also U2.W20 (IO_L11N_T1_SRCC_13); no longer U2.V20 (IO_L11P_T1_SRCC_13)
- net QDR_D16: now also U2.AA20 (IO_L8P_T1_13); no longer U2.W20 (IO_L11N_T1_SRCC_13)
- net QDR_D17: now also U2.AB21 (IO_L8N_T1_13); no longer U2.V19 (IO_L12P_T1_MRCC_13)
- net QDR_D18: now also U2.Y17 (IO_L14N_T2_SRCC_13); no longer U2.T21 (IO_L1P_T0_13)
- net QDR_D19: now also U2.Y18 (IO_L13P_T2_MRCC_13); no longer U2.U22 (IO_L2P_T0_13)
- net QDR_D2: now also U2.U20 (IO_L6N_T0_VREF_13); no longer U2.W17 (IO_L14P_T2_SRCC_13)
- net QDR_D20: now also U2.W17 (IO_L14P_T2_SRCC_13); no longer U2.U21 (IO_L1N_T0_13)
- net QDR_D21: now also U2.Y19 (IO_L13N_T2_MRCC_13); no longer U2.V22 (IO_L2N_T0_13)
- net QDR_D22: now also U2.AB16 (IO_L16N_T2_13); no longer U2.W21 (IO_L4P_T0_13)
- net QDR_D23: now also U2.AA16 (IO_L17P_T2_13); no longer U2.W22 (IO_L4N_T0_13)
- net QDR_D24: now also U2.AB15 (IO_L16P_T2_13); no longer U2.U20 (IO_L6N_T0_VREF_13)
- net QDR_D25: now also U2.AB17 (IO_L17N_T2_13); no longer U2.U17 (IO_L5P_T0_13)
- net QDR_D26: now also U2.AA14 (IO_L18P_T2_13); no longer U2.V18 (IO_L5N_T0_13)
- net QDR_D3: now also U2.U21 (IO_L1N_T0_13); no longer U2.Y17 (IO_L14N_T2_SRCC_13)
- net QDR_D4: now also U2.T21 (IO_L1P_T0_13); no longer U2.AB15 (IO_L16P_T2_13)
- net QDR_D5: now also U2.U22 (IO_L2P_T0_13); no longer U2.AB16 (IO_L16N_T2_13)
- net QDR_D6: now also U2.V22 (IO_L2N_T0_13); no longer U2.AA16 (IO_L17P_T2_13)
- net QDR_D7: now also U2.W22 (IO_L4N_T0_13); no longer U2.AB17 (IO_L17N_T2_13)
- net QDR_D8: now also U2.V18 (IO_L5N_T0_13); no longer U2.AA14 (IO_L18P_T2_13)
- net QDR_D9: now also U2.AA19 (IO_L10_PT1_13); no longer U2.Y21 (IO_L7P_T1_13)
- net QDR_ODT: now also R167.1, R168.1; no longer U2.R21 (IO_L24P_T3_A01_D17_14)
- net QDR_Q0: now also U2.B18 (IO_L20P_T3_A20_15); no longer U2.A19 (IO_L20N_T3_A19_15)
- net QDR_Q1: now also U2.A19 (IO_L20N_T3_A19_15); no longer U2.B18 (IO_L20P_T3_A20_15)
- no-connect marks 36 -> 37
Changed lines of the file:
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@@
   (no_connect (at 269.24 55.88))
   (no_connect (at 269.24 25.4))
+  (no_connect (at 198.12 38.1))
   (no_connect (at 269.24 96.52))
   (no_connect (at 269.24 121.92))
-  (no_connect (at 198.12 40.64))
   (no_connect (at 269.24 124.46))
   (no_connect (at 346.71 116.84))
@@
   (no_connect (at 33.02 179.07))
   (no_connect (at 269.24 91.44))
+  (no_connect (at 269.24 144.78))
   (no_connect (at 346.71 71.12))
   (no_connect (at 269.24 139.7))
-  (no_connect (at 198.12 38.1))
+  (no_connect (at 198.12 40.64))
   (no_connect (at 198.12 149.86))
   (no_connect (at 346.71 86.36))
@@
     (stroke (width 0) (type default) (color 0 0 0 0))
   )
+  (wire (pts (xy 38.1 146.05) (xy 38.1 151.13))
+    (stroke (width 0) (type default) (color 0 0 0 0))
+  )
   (wire (pts (xy 210.82 274.32) (xy 209.55 274.32))
     (stroke (width 0) (type default) (color 0 0 0 0))
@@
     (effects (font (size 1.27 1.27)) (justify right bottom))
   )
-  (label "QDR_D12" (at 198.12 66.04 180)
+  (label "QDR_D12" (at 198.12 83.82 180)
     (effects (font (size 1.27 1.27)) (justify right bottom))
   )
@@
     (effects (font (size 1.27 1.27)) (justify right bottom))
   )
-  (label "QDR_D20" (at 198.12 30.48 180)
+  (label "QDR_D20" (at 198.12 93.98 180)
     (effects (font (size 1.27 1.27)) (justify right bottom))
   )
@@
     (effects (font (size 1.27 1.27)) (justify right bottom))
   )
+  (label "1V8_IO" (at 45.72 151.13 0)
+    (effects (font (size 1.27 1.27)) (justify left bottom))
+  )
   (label "QDR_A11" (at 132.08 115.57 180)
     (effects (font (size 1.27 1.27)) (justify right bottom))
@@
     (effects (font (size 1.27 1.27)) (justify right bottom))
   )
-  (label "QDR_Q1" (at 346.71 124.46 180)
+  (label "QDR_Q1" (at 346.71 127 180)
     (effects (font (size 1.27 1.27)) (justify right bottom))
   )
@@
     (effects (font (size 1.27 1.27)) (justify right bottom))
   )
-  (label "QDR_BWS_0_N" (at 198.12 116.84 180)
+  (label "QDR_BWS_0_N" (at 198.12 43.18 180)
     (effects (font (size 1.27 1.27)) (justify right bottom))
   )
@@
     (effects (font (size 1.27 1.27)) (justify right bottom))
   )
-  (label "QDR_D17" (at 198.12 83.82 180)
+  (label "QDR_D17" (at 198.12 66.04 180)
     (effects (font (size 1.27 1.27)) (justify right bottom))
   )
@@
     (effects (font (size 1.27 1.27)) (justify right bottom))
   )
-  (label "QDR_D2" (at 198.12 93.98 180)
+  (label "QDR_D2" (at 198.12 55.88 180)
     (effects (font (size 1.27 1.27)) (justify right bottom))
   )
@@
     (effects (font (size 1.27 1.27)) (justify right bottom))
   )
-  (label "QDR_D8" (at 198.12 114.3 180)
+  (label "QDR_D8" (at 198.12 50.8 180)
     (effects (font (size 1.27 1.27)) (justify right bottom))
   )
@@
     (effects (font (size 1.27 1.27)) (justify right bottom))
   )
-  (label "QDR_D10" (at 198.12 60.96 180)
+  (label "QDR_D10" (at 198.12 86.36 180)
     (effects (font (size 1.27 1.27)) (justify right bottom))
   )
@@
     (effects (font (size 1.27 1.27)) (justify right bottom))
   )
-  (label "QDR_D19" (at 198.12 33.02 180)
+  (label "QDR_D19" (at 198.12 88.9 180)
     (effects (font (size 1.27 1.27)) (justify right bottom))
   )
@@
     (effects (font (size 1.27 1.27)) (justify right bottom))
   )
-  (label "QDR_BWS_1_N" (at 198.12 86.36 180)
+  (label "QDR_BWS_1_N" (at 198.12 60.96 180)
     (effects (font (size 1.27 1.27)) (justify right bottom))
   )
@@
     (effects (font (size 1.27 1.27)) (justify right bottom))
   )
-  (label "QDR_D18" (at 198.12 27.94 180)
+  (label "QDR_D18" (at 198.12 96.52 180)
     (effects (font (size 1.27 1.27)) (justify right bottom))
   )
-  (label "QDR_D3" (at 198.12 96.52 180)
+  (label "QDR_D3" (at 198.12 30.48 180)
     (effects (font (size 1.27 1.27)) (justify right bottom))
   )
@@
     (effects (font (size 1.27 1.27)) (justify right bottom))
   )
-  (label "QDR_D26" (at 198.12 50.8 180)
+  (label "QDR_D26" (at 198.12 114.3 180)
+    (effects (font (size 1.27 1.27)) (justify right bottom))
+  )
+  (label "QDR_ODT" (at 38.1 146.05 180)
     (effects (font (size 1.27 1.27)) (justify right bottom))
   )
@@
     (effects (font (size 1.27 1.27)) (justify right bottom))
   )
-  (label "QDR_D21" (at 198.12 35.56 180)
+  (label "QDR_D21" (at 198.12 91.44 180)
     (effects (font (size 1.27 1.27)) (justify right bottom))
   )
@@
     (effects (font (size 1.27 1.27)) (justify right bottom))
   )
-  (label "QDR_D15" (at 198.12 78.74 180)
+  (label "QDR_D15" (at 198.12 81.28 180)
     (effects (font (size 1.27 1.27)) (justify right bottom))
   )
-  (label "QDR_D24" (at 198.12 55.88 180)
+  (label "QDR_D24" (at 198.12 104.14 180)
     (effects (font (size 1.27 1.27)) (justify right bottom))
   )
@@
     (effects (font (size 1.27 1.27)) (justify right bottom))
   )
-  (label "QDR_D0" (at 198.12 88.9 180)
+  (label "QDR_D0" (at 198.12 53.34 180)
     (effects (font (size 1.27 1.27)) (justify right bottom))
   )
@@
     (effects (font (size 1.27 1.27)) (justify right bottom))
   )
-  (label "QDR_D23" (at 198.12 45.72 180)
+  (label "QDR_D23" (at 198.12 109.22 180)
     (effects (font (size 1.27 1.27)) (justify right bottom))
   )
@@
     (effects (font (size 1.27 1.27)) (justify right bottom))
   )
-  (label "QDR_D1" (at 198.12 91.44 180)
+  (label "QDR_D1" (at 198.12 48.26 180)
     (effects (font (size 1.27 1.27)) (justify right bottom))
   )
@@
     (effects (font (size 1.27 1.27)) (justify right bottom))
   )
-  (label "QDR_D6" (at 198.12 109.22 180)
+  (label "QDR_D6" (at 198.12 35.56 180)
     (effects (font (size 1.27 1.27)) (justify right bottom))
   )
@@
     (effects (font (size 1.27 1.27)) (justify right bottom))
   )
-  (label "QDR_D9" (at 198.12 58.42 180)
+  (label "QDR_D9" (at 198.12 73.66 180)
     (effects (font (size 1.27 1.27)) (justify right bottom))
   )
-  (label "QDR_D4" (at 198.12 104.14 180)
+  (label "QDR_D4" (at 198.12 27.94 180)
     (effects (font (size 1.27 1.27)) (justify right bottom))
   )
@@
     (effects (font (size 1.27 1.27)) (justify right bottom))
   )
-  (label "QDR_D16" (at 198.12 81.28 180)
+  (label "QDR_D16" (at 198.12 63.5 180)
     (effects (font (size 1.27 1.27)) (justify right bottom))
   )
@@
     (effects (font (size 1.27 1.27)) (justify right bottom))
   )
-  (label "QDR_D22" (at 198.12 43.18 180)
+  (label "QDR_D22" (at 198.12 106.68 180)
     (effects (font (size 1.27 1.27)) (justify right bottom))
   )
@@
     (effects (font (size 1.27 1.27)) (justify right bottom))
   )
+  (label "GND" (at 45.72 146.05 0)
+    (effects (font (size 1.27 1.27)) (justify left bottom))
+  )
   (label "QDR_Q26" (at 346.71 114.3 180)
     (effects (font (size 1.27 1.27)) (justify right bottom))
@@
     (effects (font (size 1.27 1.27)) (justify right bottom))
   )
-  (label "QDR_D13" (at 198.12 73.66 180)
+  (label "QDR_D13" (at 198.12 78.74 180)
     (effects (font (size 1.27 1.27)) (justify right bottom))
   )
@@
     (effects (font (size 1.27 1.27)) (justify right bottom))
   )
-  (label "QDR_ODT" (at 269.24 144.78 180)
-    (effects (font (size 1.27 1.27)) (justify right bottom))
-  )
-  (label "QDR_BWS_2_N" (at 198.12 53.34 180)
+  (label "QDR_BWS_2_N" (at 198.12 116.84 180)
     (effects (font (size 1.27 1.27)) (justify right bottom))
   )
@@
     (effects (font (size 1.27 1.27)) (justify right bottom))
   )
-  (label "QDR_D25" (at 198.12 48.26 180)
+  (label "QDR_D25" (at 198.12 111.76 180)
     (effects (font (size 1.27 1.27)) (justify right bottom))
   )
@@
     (effects (font (size 1.27 1.27)) (justify right bottom))
   )
-  (label "QDR_Q0" (at 346.71 127 180)
+  (label "QDR_Q0" (at 346.71 124.46 180)
     (effects (font (size 1.27 1.27)) (justify right bottom))
   )
@@
     (effects (font (size 1.27 1.27)) (justify right bottom))
   )
-  (label "QDR_D7" (at 198.12 111.76 180)
+  (label "QDR_D7" (at 198.12 45.72 180)
     (effects (font (size 1.27 1.27)) (justify right bottom))
   )
@@
     (effects (font (size 1.27 1.27)) (justify right bottom))
   )
-  (label "QDR_D11" (at 198.12 63.5 180)
+  (label "QDR_D11" (at 198.12 58.42 180)
     (effects (font (size 1.27 1.27)) (justify right bottom))
   )
@@
     (effects (font (size 1.27 1.27)) (justify right bottom))
   )
-  (label "QDR_D5" (at 198.12 106.68 180)
+  (label "QDR_D5" (at 198.12 33.02 180)
     (effects (font (size 1.27 1.27)) (justify right bottom))
   )
@@
     (pin "8")
   )
+  (symbol (lib_id "device:R") (at 41.91 146.05 90) (unit 1)
+    (in_bom yes) (on_board yes)
+    (property "Reference" "R167" (id 0) (at 41.91 143.51 90))
+    (property "Value" "1K" (id 1) (at 41.91 146.05 90))
+    (property "Footprint" "azonenberg_pcb:EIA_0402_RES_NOSILK" (id 2) (at 41.91 147.828 90)
+      (effects (font (size 1.27 1.27)) hide)
+    )
+    (property "Datasheet" "" (id 3) (at 41.91 146.05 0)
+      (effects (font (size 1.27 1.27)) hide)
+    )
+    (pin "1")
+    (pin "2")
+  )
   (symbol (lib_id "device:C") (at 143.51 243.84 0) (unit 1)
     (in_bom yes) (on_board yes) (fields_autoplaced)
@@
       (effects (font (size 1.27 1.27)) hide)
     )
+    (pin "1")
+    (pin "2")
+  )
+  (symbol (lib_id "device:R") (at 41.91 151.13 90) (unit 1)
+    (in_bom yes) (on_board yes)
+    (property "Reference" "R168" (id 0) (at 41.91 148.59 90))
+    (property "Value" "DNP" (id 1) (at 41.91 151.13 90))
+    (property "Footprint" "azonenberg_pcb:EIA_0402_RES_NOSILK" (id 2) (at 41.91 152.908 90)
+      (effects (font (size 1.27 1.27)) hide)
+    )
+    (property "Datasheet" "" (id 3) (at 41.91 151.13 0)
+      (effects (font (size 1.27 1.27)) hide)
+    )
