File: latentpink/pcb/qsgmii-power.kicad_sch (KiCad schematic)
At the start: 165 parts, among them U1 VSC8512

Commit message: Continued layout of VSC8512
Parts:
- added TP36, TP37, TP38, TP39: U.FL, azonenberg_pcb:CONN_U.FL_TE_1909763-1, symbol conn:CONN_COAXIAL
Connections:
- net A1V0_VSC: now also TP37.1 (In)
- net A1V0_VSC_SERDES1: now also TP36.1 (In)
- net A1V0_VSC_SERDES2: now also TP39.1 (In)
- net A2V5_VSC: now also TP38.1 (In)
- net GND: now also TP36.2 (Ext), TP37.2 (Ext), TP38.2 (Ext), TP39.2 (Ext)
Changed lines of the file:
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@@
   (paper "A3")
   (title_block
-    (date "2023-05-21")
+    (date "2023-05-23")
     (rev "0.1")
     (company "Antikernel Labs")
@@
   (junction (at 99.06 78.74) (diameter 0) (color 0 0 0 0)
   )
+  (junction (at 213.36 270.51) (diameter 0) (color 0 0 0 0)
+  )
   (junction (at 67.31 231.14) (diameter 0) (color 0 0 0 0)
   )
@@
   (junction (at 295.91 30.48) (diameter 0) (color 0 0 0 0)
   )
+  (junction (at 162.56 231.14) (diameter 0) (color 0 0 0 0)
+  )
   (junction (at 295.91 48.26) (diameter 0) (color 0 0 0 0)
   )
@@
   (junction (at 53.34 262.89) (diameter 0) (color 0 0 0 0)
   )
+  (junction (at 281.94 182.88) (diameter 0) (color 0 0 0 0)
+  )
   (junction (at 130.81 48.26) (diameter 0) (color 0 0 0 0)
   )
@@
   (junction (at 193.04 201.93) (diameter 0) (color 0 0 0 0)
   )
+  (junction (at 342.9 223.52) (diameter 0) (color 0 0 0 0)
+  )
   (junction (at 243.84 182.88) (diameter 0) (color 0 0 0 0)
   )
@@
   (junction (at 68.58 270.51) (diameter 0) (color 0 0 0 0)
   )
+  (junction (at 342.9 231.14) (diameter 0) (color 0 0 0 0)
+  )
   (junction (at 208.28 88.9) (diameter 0) (color 0 0 0 0)
   )
@@
   (junction (at 99.06 38.1) (diameter 0) (color 0 0 0 0)
   )
+  (junction (at 162.56 223.52) (diameter 0) (color 0 0 0 0)
+  )
   (junction (at 287.02 110.49) (diameter 0) (color 0 0 0 0)
   )
@@
   (junction (at 110.49 270.51) (diameter 0) (color 0 0 0 0)
   )
+  (junction (at 213.36 262.89) (diameter 0) (color 0 0 0 0)
+  )
   (junction (at 269.24 217.17) (diameter 0) (color 0 0 0 0)
   )
@@
   (junction (at 167.64 83.82) (diameter 0) (color 0 0 0 0)
   )
+  (junction (at 281.94 190.5) (diameter 0) (color 0 0 0 0)
+  )
   (junction (at 167.64 147.32) (diameter 0) (color 0 0 0 0)
   )
@@
     (stroke (width 0) (type default) (color 0 0 0 0))
   )
+  (wire (pts (xy 177.8 231.14) (xy 177.8 228.6))
+    (stroke (width 0) (type default) (color 0 0 0 0))
+  )
   (wire (pts (xy 295.91 20.32) (xy 295.91 22.86))
     (stroke (width 0) (type default) (color 0 0 0 0))
@@
     (stroke (width 0) (type default) (color 0 0 0 0))
   )
+  (wire (pts (xy 162.56 223.52) (xy 173.99 223.52))
+    (stroke (width 0) (type default) (color 0 0 0 0))
+  )
   (wire (pts (xy 273.05 142.24) (xy 287.02 142.24))
     (stroke (width 0) (type default) (color 0 0 0 0))
@@
     (stroke (width 0) (type default) (color 0 0 0 0))
   )
+  (wire (pts (xy 213.36 270.51) (xy 231.14 270.51))
+    (stroke (width 0) (type default) (color 0 0 0 0))
+  )
   (wire (pts (xy 99.06 71.12) (xy 99.06 73.66))
     (stroke (width 0) (type default) (color 0 0 0 0))
@@
     (stroke (width 0) (type default) (color 0 0 0 0))
   )
+  (wire (pts (xy 342.9 231.14) (xy 359.41 231.14))
+    (stroke (width 0) (type default) (color 0 0 0 0))
+  )
   (wire (pts (xy 208.28 109.22) (xy 208.28 111.76))
     (stroke (width 0) (type default) (color 0 0 0 0))
@@
     (stroke (width 0) (type default) (color 0 0 0 0))
   )
+  (wire (pts (xy 295.91 190.5) (xy 295.91 187.96))
+    (stroke (width 0) (type default) (color 0 0 0 0))
+  )
   (wire (pts (xy 267.97 81.28) (xy 267.97 83.82))
     (stroke (width 0) (type default) (color 0 0 0 0))
@@
     (stroke (width 0) (type default) (color 0 0 0 0))
   )
+  (wire (pts (xy 281.94 190.5) (xy 295.91 190.5))
+    (stroke (width 0) (type default) (color 0 0 0 0))
+  )
   (wire (pts (xy 64.77 200.66) (xy 77.47 200.66))
     (stroke (width 0) (type default) (color 0 0 0 0))
@@
     (stroke (width 0) (type default) (color 0 0 0 0))
   )
+  (wire (pts (xy 231.14 270.51) (xy 231.14 267.97))
+    (stroke (width 0) (type default) (color 0 0 0 0))
+  )
   (wire (pts (xy 269.24 182.88) (xy 281.94 182.88))
     (stroke (width 0) (type default) (color 0 0 0 0))
@@
     (stroke (width 0) (type default) (color 0 0 0 0))
   )
+  (wire (pts (xy 359.41 228.6) (xy 359.41 231.14))
+    (stroke (width 0) (type default) (color 0 0 0 0))
+  )
   (wire (pts (xy 302.26 118.11) (xy 314.96 118.11))
     (stroke (width 0) (type default) (color 0 0 0 0))
@@
     (stroke (width 0) (type default) (color 0 0 0 0))
   )
+  (wire (pts (xy 162.56 231.14) (xy 177.8 231.14))
+    (stroke (width 0) (type default) (color 0 0 0 0))
+  )
   (wire (pts (xy 208.28 50.8) (xy 208.28 53.34))
     (stroke (width 0) (type default) (color 0 0 0 0))
@@
     (stroke (width 0) (type default) (color 0 0 0 0))
   )
+  (wire (pts (xy 342.9 223.52) (xy 355.6 223.52))
+    (stroke (width 0) (type default) (color 0 0 0 0))
+  )
   (wire (pts (xy 269.24 194.31) (xy 281.94 194.31))
     (stroke (width 0) (type default) (color 0 0 0 0))
@@
     (stroke (width 0) (type default) (color 0 0 0 0))
   )
+  (wire (pts (xy 281.94 182.88) (xy 292.1 182.88))
+    (stroke (width 0) (type default) (color 0 0 0 0))
+  )
   (wire (pts (xy 208.28 30.48) (xy 208.28 33.02))
     (stroke (width 0) (type default) (color 0 0 0 0))
@@
     (stroke (width 0) (type default) (color 0 0 0 0))
   )
+  (wire (pts (xy 213.36 262.89) (xy 227.33 262.89))
+    (stroke (width 0) (type default) (color 0 0 0 0))
+  )
   (wire (pts (xy 248.92 157.48) (xy 248.92 160.02))
     (stroke (width 0) (type default) (color 0 0 0 0))
@@
     (pin "2")
   )
+  (symbol (lib_id "conn:CONN_COAXIAL") (at 295.91 182.88 0) (unit 1)
+    (in_bom yes) (on_board yes) (fields_autoplaced)
+    (property "Reference" "TP38" (id 0) (at 298.4501 182.3385 0)
+      (effects (font (size 1.27 1.27)) (justify left))
+    )
+    (property "Value" "U.FL" (id 1) (at 298.4501 184.8754 0)
+      (effects (font (size 1.27 1.27)) (justify left))
+    )
+    (property "Footprint" "azonenberg_pcb:CONN_U.FL_TE_1909763-1" (id 2) (at 295.91 182.88 0)
+      (effects (font (size 1.27 1.27)) hide)
+    )
+    (property "Datasheet" "" (id 3) (at 295.91 182.88 0)
+      (effects (font (size 1.27 1.27)) hide)
+    )
+    (pin "1")
+    (pin "2")
+  )
   (symbol (lib_id "device:C") (at 25.4 175.26 0) (unit 1)
     (in_bom yes) (on_board yes)
@@
     (pin "2")
   )
+  (symbol (lib_id "conn:CONN_COAXIAL") (at 177.8 223.52 0) (unit 1)
+    (in_bom yes) (on_board yes) (fields_autoplaced)
+    (property "Reference" "TP36" (id 0) (at 180.3401 222.9785 0)
+      (effects (font (size 1.27 1.27)) (justify left))
+    )
+    (property "Value" "U.FL" (id 1) (at 180.3401 225.5154 0)
+      (effects (font (size 1.27 1.27)) (justify left))
+    )
+    (property "Footprint" "azonenberg_pcb:CONN_U.FL_TE_1909763-1" (id 2) (at 177.8 223.52 0)
+      (effects (font (size 1.27 1.27)) hide)
+    )
+    (property "Datasheet" "" (id 3) (at 177.8 223.52 0)
+      (effects (font (size 1.27 1.27)) hide)
+    )
+    (pin "1")
+    (pin "2")
+  )
   (symbol (lib_id "device:C") (at 213.36 266.7 0) (unit 1)
     (in_bom yes) (on_board yes)
@@
     (pin "2")
   )
+  (symbol (lib_id "conn:CONN_COAXIAL") (at 359.41 223.52 0) (unit 1)
+    (in_bom yes) (on_board yes) (fields_autoplaced)
+    (property "Reference" "TP39" (id 0) (at 361.9501 222.9785 0)
+      (effects (font (size 1.27 1.27)) (justify left))
+    )
+    (property "Value" "U.FL" (id 1) (at 361.9501 225.5154 0)
+      (effects (font (size 1.27 1.27)) (justify left))
+    )
+    (property "Footprint" "azonenberg_pcb:CONN_U.FL_TE_1909763-1" (id 2) (at 359.41 223.52 0)
+      (effects (font (size 1.27 1.27)) hide)
+    )
+    (property "Datasheet" "" (id 3) (at 359.41 223.52 0)
+      (effects (font (size 1.27 1.27)) hide)
+    )
+    (pin "1")
+    (pin "2")
+  )
   (symbol (lib_id "device:C") (at 82.55 266.7 0) (unit 1)
     (in_bom yes) (on_board yes)
@@
       (effects (font (size 1.27 1.27)) hide)
     )
+    (pin "1")
+    (pin "2")
+  )
+  (symbol (lib_id "conn:CONN_COAXIAL") (at 231.14 262.89 0) (unit 1)
+    (in_bom yes) (on_board yes) (fields_autoplaced)
+    (property "Reference" "TP37" (id 0) (at 233.6801 262.3485 0)
+      (effects (font (size 1.27 1.27)) (justify left))
+    )
+    (property "Value" "U.FL" (id 1) (at 233.6801 264.8854 0)
+      (effects (font (size 1.27 1.27)) (justify left))
+    )
+    (property "Footprint" "azonenberg_pcb:CONN_U.FL_TE_1909763-1" (id 2) (at 231.14 262.89 0)
+      (effects (font (size 1.27 1.27)) hide)
+    )
+    (property "Datasheet" "" (id 3) (at 231.14 262.89 0)
+      (effects (font (size 1.27 1.27)) hide)
+    )

Commit message: Continued initial layout. Working on PHY decoupling caps and fanout
Other:
- note added: "TODO: can we shove more caps on A2V5?"
Changed lines of the file:
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@@
+    (effects (font (size 1.27 1.27)) (justify left bottom))
+  )
+  (text "TODO: can we shove more caps on A2V5?" (at 306.07 193.04 0)
     (effects (font (size 1.27 1.27)) (justify left bottom))
   )
